Commit message: add piper joint position controller for test

File: robot_description/piper_description/xacro/ros2_control.xacro (robot description, xacro)
@@ -5,142 +5,60 @@
             <plugin>hardware_mujoco_piper/HardwareMujocoPiper</plugin>
         </hardware>
-        <joint name="FR_hip_joint">
+        <joint name="joint1">
             <command_interface name="position"/>
             <command_interface name="velocity"/>
-            <command_interface name="effort"/>
-            <command_interface name="kp"/>
-            <command_interface name="kd"/>
             <state_interface name="position"/>
             <state_interface name="velocity"/>
             <state_interface name="effort"/>
         </joint>
-        <joint name="FR_thigh_joint">
+        <joint name="joint2">
             <command_interface name="position"/>
             <command_interface name="velocity"/>
-            <command_interface name="effort"/>
-            <command_interface name="kp"/>
-            <command_interface name="kd"/>
             <state_interface name="position"/>
             <state_interface name="velocity"/>
             <state_interface name="effort"/>
         </joint>
-        <joint name="FR_calf_joint">
+        <joint name="joint3">
             <command_interface name="position"/>
             <command_interface name="velocity"/>
-            <command_interface name="effort"/>
-            <command_interface name="kp"/>
-            <command_interface name="kd"/>
             <state_interface name="position"/>
             <state_interface name="velocity"/>
             <state_interface name="effort"/>
         </joint>
-        <joint name="FL_hip_joint">
+        <joint name="joint4">
             <command_interface name="position"/>
             <command_interface name="velocity"/>
-            <command_interface name="effort"/>
-            <command_interface name="kp"/>
-            <command_interface name="kd"/>
             <state_interface name="position"/>
             <state_interface name="velocity"/>
             <state_interface name="effort"/>
         </joint>
-        <joint name="FL_thigh_joint">
+        <joint name="joint5">
             <command_interface name="position"/>
             <command_interface name="velocity"/>
-            <command_interface name="effort"/>
-            <command_interface name="kp"/>
-            <command_interface name="kd"/>
             <state_interface name="position"/>
             <state_interface name="velocity"/>
             <state_interface name="effort"/>
         </joint>
-        <joint name="FL_calf_joint">
+        <joint name="joint6">
             <command_interface name="position"/>
             <command_interface name="velocity"/>
-            <command_interface name="effort"/>
-            <command_interface name="kp"/>
-            <command_interface name="kd"/>
             <state_interface name="position"/>
             <state_interface name="velocity"/>
             <state_interface name="effort"/>
         </joint>
-        <joint name="RR_hip_joint">
+        <joint name="joint7">
             <command_interface name="position"/>
             <command_interface name="velocity"/>
-            <command_interface name="effort"/>
-            <command_interface name="kp"/>
-            <command_interface name="kd"/>
             <state_interface name="position"/>
             <state_interface name="velocity"/>
             <state_interface name="effort"/>
         </joint>
-        <joint name="RR_thigh_joint">
+        <joint name="joint8">
             <command_interface name="position"/>
             <command_interface name="velocity"/>
-            <command_interface name="effort"/>
-            <command_interface name="kp"/>
-            <command_interface name="kd"/>
             <state_interface name="position"/>
             <state_interface name="velocity"/>
             <state_interface name="effort"/>
         </joint>
-        <joint name="RR_calf_joint">
-            <command_interface name="position"/>
-            <command_interface name="velocity"/>
-            <command_interface name="effort"/>
-            <command_interface name="kp"/>
-            <command_interface name="kd"/>
-            <state_interface name="position"/>
-            <state_interface name="velocity"/>
-            <state_interface name="effort"/>
-        </joint>
-        <joint name="RL_hip_joint">
-            <command_interface name="position"/>
-            <command_interface name="velocity"/>
-            <command_interface name="effort"/>
-            <command_interface name="kp"/>
-            <command_interface name="kd"/>
-            <state_interface name="position"/>
-            <state_interface name="velocity"/>
-            <state_interface name="effort"/>
-        </joint>
-        <joint name="RL_thigh_joint">
-            <command_interface name="position"/>
-            <command_interface name="velocity"/>
-            <command_interface name="effort"/>
-            <command_interface name="kp"/>
-            <command_interface name="kd"/>
-            <state_interface name="position"/>
-            <state_interface name="velocity"/>
-            <state_interface name="effort"/>
-        </joint>
-        <joint name="RL_calf_joint">
-            <command_interface name="position"/>
-            <command_interface name="velocity"/>
-            <command_interface name="effort"/>
-            <command_interface name="kp"/>
-            <command_interface name="kd"/>
-            <state_interface name="position"/>
-            <state_interface name="velocity"/>
-            <state_interface name="effort"/>
-        </joint>
-        <sensor name="imu_sensor">
-            <state_interface name="orientation.w"/>
-            <state_interface name="orientation.x"/>
-            <state_interface name="orientation.y"/>
-            <state_interface name="orientation.z"/>
-            <state_interface name="angular_velocity.x"/>
-            <state_interface name="angular_velocity.y"/>
-            <state_interface name="angular_velocity.z"/>
-            <state_interface name="linear_acceleration.x"/>
-            <state_interface name="linear_acceleration.y"/>
-            <state_interface name="linear_acceleration.z"/>
-        </sensor>
-        <!-- <sensor name="foot_contact_sensor">
-            <state_interface name="FR_foot"/>
-            <state_interface name="FL_foot"/>
-            <state_interface name="RR_foot"/>
-            <state_interface name="RL_foot"/>
-        </sensor> -->
     </ros2_control>
 </robot>
