Commit message: Sirius rl_controller bug fix
Update .pt [OBS NAME]/[ACTION NAME]. Update Sirius`s config. Fix urdf error.

File: robot_description/sirius_description/urdf/robot.urdf (robot description, URDF)
Before this commit: robot sirius, 19 links, 18 joints
Links:
- link trunk: geometry collision box size=0.047 0.047 0.047; collision box size=0.1881 0.04675 0.057

File: robot_description/sirius_description/xacro/robot.urdf (robot description, URDF)
Before this commit: robot sirius, 19 links, 18 joints
Links:
- link trunk: geometry collision box size=0.047 0.047 0.047; collision box size=0.1881 0.04675 0.057
