Commit message: update model for sirius with piper

File: robot_description/quadruped_manipulator_description/urdf/robot.urdf (robot description, URDF)
Before this commit: robot arcdog, 19 links, 18 joints
Links:
- added link base_link, mass 1.02; collision mesh filename=package://piper_description/meshes/base_link.STL; visual mesh filename=package://piper_description/meshes/base_link.STL
- added link gripper_base, mass 0.45; collision mesh filename=package://piper_description/meshes/gripper_base.STL; visual mesh filename=package://piper_description/meshes/gripper_base.STL
- added link link1, mass 0.71; collision mesh filename=package://piper_description/meshes/link1.STL; visual mesh filename=package://piper_description/meshes/link1.STL
- added link link2, mass 1.17; collision mesh filename=package://piper_description/meshes/link2.STL; visual mesh filename=package://piper_description/meshes/link2.STL
- added link link3, mass 0.5; collision mesh filename=package://piper_description/meshes/link3.STL; visual mesh filename=package://piper_description/meshes/link3.STL
- added link link4, mass 0.38; collision mesh filename=package://piper_description/meshes/link4.STL; visual mesh filename=package://piper_description/meshes/link4.STL
- added link link5, mass 0.383; collision mesh filename=package://piper_description/meshes/link5.STL; visual mesh filename=package://piper_description/meshes/link5.STL
- added link link6, mass 0.00699089613564366; collision mesh filename=package://piper_description/meshes/link6.STL; visual mesh filename=package://piper_description/meshes/link6.STL
- added link link7, mass 0.025; collision mesh filename=package://piper_description/meshes/link7.STL; visual mesh filename=package://piper_description/meshes/link7.STL
- added link link8, mass 0.025; collision mesh filename=package://piper_description/meshes/link8.STL; visual mesh filename=package://piper_description/meshes/link8.STL
- link FL_calf: mass 0.213 -> 0.46394589686281; geometry collision mesh filename=package://sirius_mid_v3_description/meshes/shank_fr.STL scale=1 1 1; visual mesh filename=package://sirius_mid_v3_description/meshes/shank_fr.STL scale=1 1 1
- link FL_foot: geometry collision sphere radius=0.03; visual sphere radius=0.03
- link FL_hip: mass 0.8365 -> 1.83991949808533; geometry collision cylinder length=0.09 radius=0.055; visual mesh filename=package://sirius_mid_v3_description/meshes/difference_fr.STL scale=1 1 1
- link FL_thigh: mass 1.987 -> 1.84491872524247; geometry collision box size=0.270122814075178 0.05 0.05; collision cylinder length=0.0985 radius=0.044
- link FR_calf: mass 0.213 -> 0.46394589686281; geometry collision mesh filename=package://sirius_mid_v3_description/meshes/shank_fl.STL scale=1 1 1; visual mesh filename=package://sirius_mid_v3_description/meshes/shank_fl.STL scale=1 1 1
- link FR_foot: geometry collision sphere radius=0.03; visual sphere radius=0.03
- link FR_hip: mass 0.8365 -> 1.83991949808533; geometry collision cylinder length=0.09 radius=0.055; visual mesh filename=package://sirius_mid_v3_description/meshes/difference_fl.STL scale=1 1 1
- link FR_thigh: mass 1.987 -> 1.84491872524247; geometry collision box size=0.270122814075178 0.05 0.05; collision cylinder length=0.0985 radius=0.044
- link RL_calf: mass 0.213 -> 0.46394589686281; geometry collision mesh filename=package://sirius_mid_v3_description/meshes/shank_br.STL scale=1 1 1; visual mesh filename=package://sirius_mid_v3_description/meshes/shank_br.STL scale=1 1 1
- link RL_foot: geometry collision sphere radius=0.03; visual sphere radius=0.03
- link RL_hip: mass 0.8365 -> 1.83991949808533; geometry collision cylinder length=0.09 radius=0.055; visual mesh filename=package://sirius_mid_v3_description/meshes/difference_br.STL scale=1 1 1
- link RL_thigh: mass 1.987 -> 1.84491872524247; geometry collision box size=0.270122814075178 0.05 0.05; collision cylinder length=0.0985 radius=0.044
- link RR_calf: mass 0.213 -> 0.46394589686281; geometry collision mesh filename=package://sirius_mid_v3_description/meshes/shank_bl.STL scale=1 1 1; visual mesh filename=package://sirius_mid_v3_description/meshes/shank_bl.STL scale=1 1 1
- link RR_foot: geometry collision sphere radius=0.03; visual sphere radius=0.03
- link RR_hip: mass 0.8365 -> 1.83991949808533; geometry collision cylinder length=0.09 radius=0.055; visual mesh filename=package://sirius_mid_v3_description/meshes/difference_bl.STL scale=1 1 1
- link RR_thigh: mass 1.987 -> 1.84491872524247; geometry collision box size=0.270122814075178 0.05 0.05; collision cylinder length=0.0985 radius=0.044
- link trunk: mass 8.4845 -> 12.149; geometry collision box size=0.48200 0.21200 0.11200; visual mesh filename=package://sirius_mid_v3_description/meshes/base_link.STL scale=1 1 1
Joints:
- added joint arm_mount_joint: type fixed, parent trunk, child base_link, origin xyz=0.10 0 0.065 rpy=0 0 0
- added joint joint1: type revolute, parent base_link, child link1, origin xyz=0 0 0.123 rpy=0 0 0, axis 0 0 1, limit lower=-2.618 upper=2.168 effort=100 velocity=5
- added joint joint2: type revolute, parent link1, child link2, origin xyz=0 0 0 rpy=1.5708 -0.1359 -3.1416, axis 0 0 1, limit lower=0 upper=3.14 effort=100 velocity=5
- added joint joint3: type revolute, parent link2, child link3, origin xyz=0.28503 0 0 rpy=0 0 -1.7939, axis 0 0 1, limit lower=-2.967 upper=0 effort=100 velocity=5
- added joint joint4: type revolute, parent link3, child link4, origin xyz=-0.021984 -0.25075 0 rpy=1.5708 0 0, axis 0 0 1, limit lower=-1.745 upper=1.745 effort=100 velocity=5
- added joint joint5: type revolute, parent link4, child link5, origin xyz=0 0 0 rpy=-1.5708 0 0, axis 0 0 1, limit lower=-1.22 upper=1.22 effort=100 velocity=5
- added joint joint6: type revolute, parent link5, child link6, origin xyz=8.8259E-05 -0.091 0 rpy=1.5708 0 0, axis 0 0 1, limit lower=-2.0944 upper=2.0944 effort=100 velocity=3
- added joint joint6_to_gripper_base: type fixed, parent link6, child gripper_base, origin xyz=0 0 0 rpy=0 0 0
- added joint joint7: type prismatic, parent gripper_base, child link7, origin xyz=0 0 0.1358 rpy=1.5708 0 0, axis 0 0 1, limit lower=0 upper=0.035 effort=10 velocity=1
- added joint joint8: type prismatic, parent gripper_base, child link8, origin xyz=0 0 0.1358 rpy=1.5708 0 -3.1416, axis 0 0 -1, limit lower=-0.035 upper=0 effort=10 velocity=1
- joint FL_calf_joint: limit lower=-2.775073510670984 upper=-0.6457718232379019 effort=44.4 velocity=15.89 -> lower=-3.141592653589793 upper=1.174532925199433 effort=45 velocity=45; origin xyz=0 0 -0.2445 rpy=0 0 0 -> xyz=0 0.0931000000000018 -0.270122814075178 rpy=0 0 0
- joint FL_foot_fixed: origin xyz=0 0 -0.23704 rpy=0 0 0 -> xyz=-0.07 0 -0.252 rpy=0 0 0
- joint FL_hip_joint: limit lower=-1.2217304763960306 upper=1.2217304763960306 effort=35.278 velocity=20 -> lower=-0.7853981633974483 upper=0.7853981633974483 effort=35.0 velocity=45; origin xyz=0.274 0.0605 0 rpy=0 0 0 -> xyz=0.31 0.05 0 rpy=0 0 0
- joint FL_thigh_joint: limit lower=-1.5708 upper=3.4907 effort=35.278 velocity=20 -> lower=-1.57 upper=1.57 effort=35.0 velocity=45; origin xyz=0 0.1095 0 rpy=0 0 0 -> xyz=0 0.0415 0 rpy=0 0 0
- joint FR_calf_joint: limit lower=-2.775073510670984 upper=-0.6457718232379019 effort=44.4 velocity=15.89 -> lower=-3.141592653589793 upper=1.174532925199433 effort=45 velocity=45; origin xyz=0 0 -0.2445 rpy=0 0 0 -> xyz=0 -0.0931000000000018 -0.270122814075178 rpy=0 0 0
- joint FR_foot_fixed: origin xyz=0 0 -0.23704 rpy=0 0 0 -> xyz=-0.07 0 -0.252 rpy=0 0 0
- joint FR_hip_joint: limit lower=-1.2217304763960306 upper=1.2217304763960306 effort=35.278 velocity=20 -> lower=-0.7853981633974483 upper=0.7853981633974483 effort=35.0 velocity=45; origin xyz=0.274 -0.0605 0 rpy=0 0 0 -> xyz=0.31 -0.05 0 rpy=0 0 0
- joint FR_thigh_joint: limit lower=-1.5708 upper=3.4907 effort=35.278 velocity=20 -> lower=-1.57 upper=1.57 effort=35.0 velocity=45; origin xyz=0 -0.1095 0 rpy=0 0 0 -> xyz=0 -0.0415 0 rpy=0 0 0
- joint RL_calf_joint: limit lower=-2.775073510670984 upper=-0.6457718232379019 effort=44.4 velocity=15.89 -> lower=-1.174532925199433 upper=3.141592653589793 effort=45 velocity=45; origin xyz=0 0 -0.2445 rpy=0 0 0 -> xyz=0 0.0931000000000018 -0.270122814075178 rpy=0 0 0
- joint RL_foot_fixed: origin xyz=0 0 -0.23704 rpy=0 0 0 -> xyz=0.07 0 -0.252 rpy=0 0 0
- joint RL_hip_joint: limit lower=-1.2217304763960306 upper=1.2217304763960306 effort=35.278 velocity=20 -> lower=-0.7853981633974483 upper=0.7853981633974483 effort=35.0 velocity=45; origin xyz=-0.274 0.0605 0 rpy=0 0 0 -> xyz=-0.31 0.05 0 rpy=0 0 0
- joint RL_thigh_joint: limit lower=-1.5708 upper=3.4907 effort=35.278 velocity=20 -> lower=-1.57 upper=1.57 effort=35.0 velocity=45; origin xyz=0 0.1095 0 rpy=0 0 0 -> xyz=0 0.0415 0 rpy=0 0 0
- joint RR_calf_joint: limit lower=-2.775073510670984 upper=-0.6457718232379019 effort=44.4 velocity=15.89 -> lower=-1.174532925199433 upper=3.141592653589793 effort=45 velocity=45; origin xyz=0 0 -0.2445 rpy=0 0 0 -> xyz=0 -0.0931000000000018 -0.270122814075178 rpy=0 0 0
- joint RR_foot_fixed: origin xyz=0 0 -0.23704 rpy=0 0 0 -> xyz=0.07 0 -0.252 rpy=0 0 0
- joint RR_hip_joint: limit lower=-1.2217304763960306 upper=1.2217304763960306 effort=35.278 velocity=20 -> lower=-0.7853981633974483 upper=0.7853981633974483 effort=35.0 velocity=45; origin xyz=-0.274 -0.0605 0 rpy=0 0 0 -> xyz=-0.31 -0.05 0 rpy=0 0 0
- joint RR_thigh_joint: limit lower=-1.5708 upper=3.4907 effort=35.278 velocity=20 -> lower=-1.57 upper=1.57 effort=35.0 velocity=45; origin xyz=0 -0.1095 0 rpy=0 0 0 -> xyz=0 -0.0415 0 rpy=0 0 0

File: robot_description/quadruped_manipulator_description/xacro/robot.xacro (robot description, xacro)
@@ -1,5 +1,4 @@
 <?xml version="1.0"?>
-<robot name="arcdog_with_arm" xmlns:xacro="http://www.ros.org/wiki/xacro">
-    <!-- 1. 定义arcdog需要的参数（与arcdog文件中的参数一致） -->
+<robot name="sirius_piper" xmlns:xacro="http://www.ros.org/wiki/xacro">
     <xacro:arg name="DEBUG" default="false"/>
     <xacro:arg name="GAZEBO" default="false"/>
@@ -7,19 +6,11 @@
     <xacro:arg name="robot_type" default="arcdog"/>
     <xacro:arg name="simulator" default="test"/>
-    <!-- 2. 包含arcdog的xacro文件 -->
-    <!-- 注意：这里直接包含原始arcdog文件，它会使用上面定义的参数 -->
-    <xacro:include filename="$(find arcdog_description)/xacro/arcdog.xacro" />
-    <!-- 3. 包含机械臂描述文件 -->
+    <xacro:include filename="$(find sirius_mid_v3_description)/xacro/sirius_mid_v3.xacro" />
     <xacro:include filename="$(find piper_description)/urdf/piper_arm.xacro"/>
-<!--    &lt;!&ndash; 4. 实例化机械臂（添加前缀） &ndash;&gt;-->
-<!--    <xacro:piper_arm prefix="arm_"/>-->
-    <!-- 5. 创建连接关节（安装在躯干上） -->
     <joint name="arm_mount_joint" type="fixed">
         <parent link="trunk"/>
         <child link="base_link"/>
-        <!-- 安装位姿：躯干中心前方0.2m，高度0.15m -->
-        <origin xyz="0.10 0 0.05" rpy="0 0 0"/>
+        <origin xyz="0.10 0 0.065" rpy="0 0 0"/>
     </joint>
-    <!-- 6. Gazebo插件集成（如果GAZEBO参数为true） -->
     <xacro:if value="$(arg GAZEBO)">
         <gazebo>
@@ -30,3 +21,6 @@
         </gazebo>
     </xacro:if>
+    <xacro:unless value="$(arg GAZEBO)">
+    	<xacro:include filename="$(find quadruped_manipulator_description)/xacro/ros2_control.xacro"/>
+    </xacro:unless>
 </robot>

File: robot_description/sirius_mid_v3_description/urdf/robot.urdf (robot description, URDF)
Before this commit: robot sirius_mid_v3, 18 links, 17 joints
Links:
- removed link LF_FOOT
- removed link LH_FOOT
- removed link RF_FOOT
- removed link RH_FOOT
- removed link difference_bl
- removed link difference_br
- removed link difference_fl
- removed link difference_fr
- removed link shank_bl
- removed link shank_br
- removed link shank_fl
- removed link shank_fr
- removed link thigh_bl
- removed link thigh_br
- removed link thigh_fl
- removed link thigh_fr
- removed link unitree_imu
- added link FL_calf, mass 0.46394589686281; collision mesh filename=package://sirius_mid_v3_description/meshes/shank_fr.STL scale=1 1 1; visual mesh filename=package://sirius_mid_v3_description/meshes/shank_fr.STL scale=1 1 1
- added link FL_foot, mass 0.06; collision sphere radius=0.03; visual sphere radius=0.03
- added link FL_hip, mass 1.83991949808533; collision cylinder length=0.09 radius=0.055; visual mesh filename=package://sirius_mid_v3_description/meshes/difference_fr.STL scale=1 1 1
- added link FL_thigh, mass 1.84491872524247; collision box size=0.270122814075178 0.05 0.05; collision cylinder length=0.0985 radius=0.044
- added link FR_calf, mass 0.46394589686281; collision mesh filename=package://sirius_mid_v3_description/meshes/shank_fl.STL scale=1 1 1; visual mesh filename=package://sirius_mid_v3_description/meshes/shank_fl.STL scale=1 1 1
- added link FR_foot, mass 0.06; collision sphere radius=0.03; visual sphere radius=0.03
- added link FR_hip, mass 1.83991949808533; collision cylinder length=0.09 radius=0.055; visual mesh filename=package://sirius_mid_v3_description/meshes/difference_fl.STL scale=1 1 1
- added link FR_thigh, mass 1.84491872524247; collision box size=0.270122814075178 0.05 0.05; collision cylinder length=0.0985 radius=0.044
- added link RL_calf, mass 0.46394589686281; collision mesh filename=package://sirius_mid_v3_description/meshes/shank_br.STL scale=1 1 1; visual mesh filename=package://sirius_mid_v3_description/meshes/shank_br.STL scale=1 1 1
- added link RL_foot, mass 0.06; collision sphere radius=0.03; visual sphere radius=0.03
- added link RL_hip, mass 1.83991949808533; collision cylinder length=0.09 radius=0.055; visual mesh filename=package://sirius_mid_v3_description/meshes/difference_br.STL scale=1 1 1
- added link RL_thigh, mass 1.84491872524247; collision box size=0.270122814075178 0.05 0.05; collision cylinder length=0.0985 radius=0.044
- added link RR_calf, mass 0.46394589686281; collision mesh filename=package://sirius_mid_v3_description/meshes/shank_bl.STL scale=1 1 1; visual mesh filename=package://sirius_mid_v3_description/meshes/shank_bl.STL scale=1 1 1
- added link RR_foot, mass 0.06; collision sphere radius=0.03; visual sphere radius=0.03
- added link RR_hip, mass 1.83991949808533; collision cylinder length=0.09 radius=0.055; visual mesh filename=package://sirius_mid_v3_description/meshes/difference_bl.STL scale=1 1 1
- added link RR_thigh, mass 1.84491872524247; collision box size=0.270122814075178 0.05 0.05; collision cylinder length=0.0985 radius=0.044
- added link imu_link, mass 0.001; collision box size=.001 .001 .001; visual box size=0.001 0.001 0.001
- added link trunk, mass 12.149; collision box size=0.48200 0.21200 0.11200; visual mesh filename=package://sirius_mid_v3_description/meshes/base_link.STL scale=1 1 1
- link base: mass 12.149 -> None; geometry visual box size=0.001 0.001 0.001
Joints:
- removed joint LF_FOOT_fixed_joint
- removed joint LF_HAA
- removed joint LF_HFE
- removed joint LF_KFE
- removed joint LH_FOOT_fixed_joint
- removed joint LH_HAA
- removed joint LH_HFE
- removed joint LH_KFE
- removed joint RF_FOOT_fixed_joint
- removed joint RF_HAA
- removed joint RF_HFE
- removed joint RF_KFE
- removed joint RH_FOOT_fixed_joint
- removed joint RH_HAA
- removed joint RH_HFE
- removed joint RH_KFE
- removed joint unitree_imu_joint
- added joint FL_calf_joint: type revolute, parent FL_thigh, child FL_calf, origin xyz=0 0.0931000000000018 -0.270122814075178 rpy=0 0 0, axis 0 1 0, limit lower=-3.141592653589793 upper=1.174532925199433 effort=45 velocity=45
- added joint FL_foot_fixed: type fixed, parent FL_calf, child FL_foot, origin xyz=-0.07 0 -0.252 rpy=0 0 0
- added joint FL_hip_joint: type revolute, parent trunk, child FL_hip, origin xyz=0.31 0.05 0 rpy=0 0 0, axis 1 0 0, limit lower=-0.7853981633974483 upper=0.7853981633974483 effort=35.0 velocity=45
- added joint FL_thigh_joint: type revolute, parent FL_hip, child FL_thigh, origin xyz=0 0.0415 0 rpy=0 0 0, axis 0 1 0, limit lower=-1.57 upper=1.57 effort=35.0 velocity=45
- added joint FR_calf_joint: type revolute, parent FR_thigh, child FR_calf, origin xyz=0 -0.0931000000000018 -0.270122814075178 rpy=0 0 0, axis 0 1 0, limit lower=-3.141592653589793 upper=1.174532925199433 effort=45 velocity=45
- added joint FR_foot_fixed: type fixed, parent FR_calf, child FR_foot, origin xyz=-0.07 0 -0.252 rpy=0 0 0
- added joint FR_hip_joint: type revolute, parent trunk, child FR_hip, origin xyz=0.31 -0.05 0 rpy=0 0 0, axis 1 0 0, limit lower=-0.7853981633974483 upper=0.7853981633974483 effort=35.0 velocity=45
- added joint FR_thigh_joint: type revolute, parent FR_hip, child FR_thigh, origin xyz=0 -0.0415 0 rpy=0 0 0, axis 0 1 0, limit lower=-1.57 upper=1.57 effort=35.0 velocity=45
- added joint RL_calf_joint: type revolute, parent RL_thigh, child RL_calf, origin xyz=0 0.0931000000000018 -0.270122814075178 rpy=0 0 0, axis 0 1 0, limit lower=-1.174532925199433 upper=3.141592653589793 effort=45 velocity=45
- added joint RL_foot_fixed: type fixed, parent RL_calf, child RL_foot, origin xyz=0.07 0 -0.252 rpy=0 0 0
- added joint RL_hip_joint: type revolute, parent trunk, child RL_hip, origin xyz=-0.31 0.05 0 rpy=0 0 0, axis 1 0 0, limit lower=-0.7853981633974483 upper=0.7853981633974483 effort=35.0 velocity=45
- added joint RL_thigh_joint: type revolute, parent RL_hip, child RL_thigh, origin xyz=0 0.0415 0 rpy=0 0 0, axis 0 1 0, limit lower=-1.57 upper=1.57 effort=35.0 velocity=45
- added joint RR_calf_joint: type revolute, parent RR_thigh, child RR_calf, origin xyz=0 -0.0931000000000018 -0.270122814075178 rpy=0 0 0, axis 0 1 0, limit lower=-1.174532925199433 upper=3.141592653589793 effort=45 velocity=45
- added joint RR_foot_fixed: type fixed, parent RR_calf, child RR_foot, origin xyz=0.07 0 -0.252 rpy=0 0 0
- added joint RR_hip_joint: type revolute, parent trunk, child RR_hip, origin xyz=-0.31 -0.05 0 rpy=0 0 0, axis 1 0 0, limit lower=-0.7853981633974483 upper=0.7853981633974483 effort=35.0 velocity=45
- added joint RR_thigh_joint: type revolute, parent RR_hip, child RR_thigh, origin xyz=0 -0.0415 0 rpy=0 0 0, axis 0 1 0, limit lower=-1.57 upper=1.57 effort=35.0 velocity=45
- added joint floating_base: type fixed, parent base, child trunk, origin xyz=0 0 0 rpy=0 0 0
- added joint imu_joint: type fixed, parent trunk, child imu_link, origin xyz=0 0 0 rpy=0 0 0

File: robot_description/sirius_mid_v3_description/xacro/const.xacro (robot description, xacro)
@@ -43,18 +43,18 @@
     <xacro:property name="damping" value="0.05"/>
     <xacro:property name="friction" value="0.01"/>
-    <xacro:property name="hip_max" value="0.8028514559173915"/>
-    <xacro:property name="hip_min" value="-0.8028514559173915"/>
-    <xacro:property name="hip_velocity_max" value="21"/>
-    <xacro:property name="hip_torque_max" value="45.0"/>
-    <xacro:property name="thigh_max" value="4.1887902047863905"/>
-    <xacro:property name="thigh_min" value="-4.1887902047863905"/>
-    <xacro:property name="thigh_velocity_max" value="21"/>
-    <xacro:property name="thigh_torque_max" value="45.0"/>
-    <xacro:property name="calf_max_f" value="-0.9162978572970231"/>
-    <xacro:property name="calf_min_f" value="-2.6965336943312392"/>
-    <xacro:property name="calf_min_r" value="0.9162978572970231"/>
-    <xacro:property name="calf_max_r" value="2.6965336943312392"/>
-    <xacro:property name="calf_velocity_max" value="21"/>
-    <xacro:property name="calf_torque_max" value="80"/>
+    <xacro:property name="hip_max" value="0.7853981633974483"/>
+    <xacro:property name="hip_min" value="-0.7853981633974483"/>
+    <xacro:property name="hip_velocity_max" value="45"/>
+    <xacro:property name="hip_torque_max" value="35.0"/>
+    <xacro:property name="thigh_max" value="1.57"/>
+    <xacro:property name="thigh_min" value="-1.57"/>
+    <xacro:property name="thigh_velocity_max" value="45"/>
+    <xacro:property name="thigh_torque_max" value="35.0"/>
+    <xacro:property name="calf_max_f" value="1.17453292519943295"/>
+    <xacro:property name="calf_min_f" value="-3.141592653589793"/>
+    <xacro:property name="calf_min_r" value="-1.17453292519943295"/>
+    <xacro:property name="calf_max_r" value="3.141592653589793"/>
+    <xacro:property name="calf_velocity_max" value="45"/>
+    <xacro:property name="calf_torque_max" value="45"/>
     <!-- dynamics inertial value    total 22.0kg-->
     <!-- trunk -->

File: robot_description/sirius_mid_v3_description/xacro/robot.xacro (robot description, xacro)
@@ -51,5 +51,5 @@
 			<origin rpy="0 0 0" xyz="0 0 0"/>
 			<geometry>
-				<mesh filename="file://$(find sirius_mid_v3_description)/meshes/base_link.STL" scale="1 1 1"/>
+				<mesh filename="package://sirius_mid_v3_description/meshes/base_link.STL" scale="1 1 1"/>
 			</geometry>
 			<!-- <material name="orange"/> -->
