Commit message: update for sirius real robot

File: robot_description/sirius_description/xacro/real_robot.xacro (robot description, xacro)
@@ -1,4 +1,4 @@
 <?xml version="1.0"?>
-<robot name="arcdog" xmlns:xacro="http://www.ros.org/wiki/xacro">
+<robot name="sirius" xmlns:xacro="http://www.ros.org/wiki/xacro">
 	<xacro:arg name="DEBUG" default="false"/>
 	<xacro:arg name="GAZEBO" default="false"/>
@@ -8,17 +8,17 @@
 	<xacro:arg name="simulator" default="test"/>
     <xacro:property name="simulator" value="$(arg simulator)"/>
-	<xacro:include filename="$(find arcdog_description)/xacro/const.xacro"/>
-	<xacro:include filename="$(find arcdog_description)/xacro/materials.xacro"/>
-	<xacro:include filename="$(find arcdog_description)/xacro/leg.xacro"/>
+	<xacro:include filename="$(find sirius_description)/xacro/const.xacro"/>
+	<xacro:include filename="$(find sirius_description)/xacro/materials.xacro"/>
+	<xacro:include filename="$(find sirius_description)/xacro/leg.xacro"/>
 	<xacro:if value="$(arg GAZEBO)">
 		<xacro:if value="$(arg CLASSIC)">
-			<xacro:include filename="$(find arcdog_description)/xacro/gazebo_classic.xacro"/>
+			<xacro:include filename="$(find sirius_description)/xacro/gazebo_classic.xacro"/>
 		</xacro:if>
 		<xacro:unless value="$(arg CLASSIC)">
-			<xacro:include filename="$(find arcdog_description)/xacro/gazebo.xacro"/>
+			<xacro:include filename="$(find sirius_description)/xacro/gazebo.xacro"/>
 		</xacro:unless>
 	</xacro:if>
 	<xacro:unless value="$(arg GAZEBO)">
-		<xacro:include filename="$(find arcdog_description)/xacro/ros2_control_real_robot.xacro"/>
+		<xacro:include filename="$(find sirius_description)/xacro/ros2_control_real_robot.xacro"/>
 	</xacro:unless>
 	<!-- <xacro:stairs stairs="15" xpos="0" ypos="0" zpos="0" /> -->
@@ -51,5 +51,5 @@
 			<origin rpy="0 0 0" xyz="0 0 0"/>
 			<geometry>
-				<mesh filename="file://$(find arcdog_description)/meshes/trunk.dae" scale="1 1 1"/>
+				<mesh filename="file://$(find sirius_description)/meshes/base_link.dae" scale="1 1 1"/>
 			</geometry>
 			<!-- <material name="orange"/> -->

File: robot_description/sirius_description/xacro/ros2_control_real_robot.xacro (robot description, xacro)
@@ -3,5 +3,5 @@
 	<ros2_control name="SiriusSystem" type="system">
 		<hardware>
-			<plugin>hardware_arcdog/HardwareArcdog</plugin>
+			<plugin>hardware_sirius/HardwareSirius</plugin>
 		</hardware>
 		<joint name="FR_hip_joint">
