Commit message: bug hunting, save version

File: robot_description/piper_description/urdf/piper_arm_joint1_fixed.xacro (robot description, xacro)
@@ -11,5 +11,5 @@
 <!-- arm -->
 <link
-    name="base_link">
+    name="arm_base_link">
     <inertial>
             <origin xyz="-0.00473641164191482 2.56829134630247E-05 0.041451518036016" rpy="0 0 0" />
@@ -74,10 +74,10 @@
   <joint
     name="joint1"
-    type="revolute">
+    type="fixed">
     <origin
       xyz="0 0 0.123"
       rpy="0 0 0" />
     <parent
-      link="base_link" />
+      link="arm_base_link" />
     <child
       link="link1" />
@@ -505,4 +505,21 @@
   </joint>
 <!-- controller -->
+  <xacro:macro name="transmission_block" params="tran_name joint_name motor_name">
+    <transmission name="${tran_name}">
+        <type>transmission_interface/SimpleTransmission</type>
+        <joint name="${joint_name}">
+            <hardwareInterface>hardware_interface/PositionJointInterface</hardwareInterface>
+        </joint>
+        <actuator name="$motor_name">
+            <hardwareInterface>hardware_interface/PositionJointInterface</hardwareInterface>
+            <mechanicalReduction>1</mechanicalReduction>
+        </actuator>
+    </transmission>
+  </xacro:macro>
+  <xacro:transmission_block tran_name="tran2" joint_name="joint2" motor_name="motor2"/>
+  <xacro:transmission_block tran_name="tran3" joint_name="joint3" motor_name="motor3"/>
+  <xacro:transmission_block tran_name="tran4" joint_name="joint4" motor_name="motor4"/>
+  <xacro:transmission_block tran_name="tran5" joint_name="joint5" motor_name="motor5"/>
+  <xacro:transmission_block tran_name="tran6" joint_name="joint6" motor_name="motor6"/>
 <!-- gazebo -->
 <!--  <gazebo>-->

File: robot_description/quadruped_manipulator_description/xacro/robot.urdf (robot description, URDF)
Before this commit: robot sirius_piper, 29 links, 28 joints
Joints:
- joint joint7: type prismatic -> fixed
- joint joint8: type prismatic -> fixed

File: robot_description/quadruped_manipulator_description/xacro/robot.xacro (robot description, xacro)
@@ -8,5 +8,4 @@
 	<xacro:arg name="simulator" default="arclab_rl"/>
     <xacro:include filename="$(find sirius_description)/xacro/sirius.xacro" />
-    <xacro:include filename="$(find piper_description)/urdf/piper_arm.xacro"/>
     <joint name="arm_mount_joint" type="fixed">
         <parent link="trunk"/>
@@ -14,4 +13,5 @@
         <origin xyz="0.2 0 0.085" rpy="0 0 0"/>
     </joint>
+    <xacro:include filename="$(find piper_description)/urdf/piper_arm.xacro"/>
     <xacro:include filename="$(find quadruped_manipulator_description)/xacro/ros2_control.xacro"/>
 </robot>

File: robot_description/quadruped_manipulator_description/xacro/ros2_control.xacro (robot description, xacro)
@@ -1,5 +1,5 @@
 <?xml version="1.0"?>
 <robot xmlns:xacro="http://www.ros.org/wiki/xacro">
-	<ros2_control name="ArcdogSystem" type="system">
+	<ros2_control name="QuadrupedManipulatorSystem" type="system">
 		<hardware>
 			<plugin>hardware_mujoco_quadruped_manipulator/HardwareMujocoQuadrupedManipulator</plugin>

File: robot_description/sirius_description/xacro/sirius.xacro (robot description, xacro)
@@ -9,5 +9,4 @@
 	<xacro:include filename="$(find sirius_description)/xacro/materials.xacro"/>
 	<xacro:include filename="$(find sirius_description)/xacro/leg.xacro"/>
-	<xacro:include filename="$(find sirius_description)/xacro/ros2_control.xacro"/>
 	<!-- <xacro:stairs stairs="15" xpos="0" ypos="0" zpos="0" /> -->
 	<!-- Rotor related joint and link is only for demonstrate location. -->
