Commit message: add arcdog adjustable leg model

File: robot_description/arcdog_adjustable_leg_description/xacro/const.xacro (robot description, xacro)
@@ -22,10 +22,10 @@
 	<xacro:property name="stick_radius" value="0.01"/>
 	<xacro:property name="stick_length" value="0.2"/>
-	<!-- kinematic value -->
-	<xacro:property name="thigh_offset" value="0.0955"/>
-	<xacro:property name="thigh_length" value="0.213"/>
-	<xacro:property name="calf_length" value="0.213"/>
+    <!-- kinematic value -->
+    <xacro:property name="thigh_offset" value="0.09426"/>
+    <xacro:property name="thigh_length" value="0.2445"/>
+    <xacro:property name="calf_length" value="0.1930"/>
     <!-- leg offset from trunk center value -->
-    <xacro:property name="leg_offset_x" value="0.274"/>
+    <xacro:property name="leg_offset_x" value="0.269"/>
     <xacro:property name="leg_offset_y" value="0.0605"/>
     <xacro:property name="trunk_offset_z" value="0.01675"/> //TODO
@@ -36,7 +36,7 @@
 	<xacro:property name="hip_offset_z" value="0.0"/>
     <!-- kinematic value -->
-    <xacro:property name="thigh_offset" value="0.1095"/>
+    <!-- <xacro:property name="thigh_offset" value="0.1095"/>
     <xacro:property name="thigh_length" value="0.2445"/>
-    <xacro:property name="calf_length" value="0.23704"/>
+    <xacro:property name="calf_length" value="0.23704"/>  -->
 	<xacro:property name="calf_offset_x" value="0.0"/>
 	<xacro:property name="calf_offset_y" value="0.0"/>
@@ -59,48 +59,59 @@
     <!-- dynamics inertial value    total 22.0kg-->
     <!-- trunk -->
-    <xacro:property name="trunk_mass" value="8.4845"/>
-    <xacro:property name="trunk_com_x" value="-0.000466"/>
-    <xacro:property name="trunk_com_y" value="-0.000692"/>
-    <xacro:property name="trunk_com_z" value="-0.008587"/>
-    <xacro:property name="trunk_ixx" value="0.031520962"/>
-    <xacro:property name="trunk_ixy" value="-0.000002732"/>
-    <xacro:property name="trunk_ixz" value="-0.000285792"/>
-    <xacro:property name="trunk_iyy" value="0.143653339"/>
-    <xacro:property name="trunk_iyz" value="0.000011831"/>
-    <xacro:property name="trunk_izz" value="0.159618308"/>
+    <xacro:property name="trunk_mass" value="7.021"/>
+    <xacro:property name="trunk_com_x" value="0.00575"/>
+    <xacro:property name="trunk_com_y" value="0.00126"/>
+    <xacro:property name="trunk_com_z" value="-0.00469"/>
+    <xacro:property name="trunk_ixx" value="0.03769023916"/>
+    <xacro:property name="trunk_ixy" value="0.00001433761"/>
+    <xacro:property name="trunk_ixz" value="0.00051349975"/>
+    <xacro:property name="trunk_iyy" value="0.05008788073"/>
+    <xacro:property name="trunk_iyz" value="0.00015851764"/>
+    <xacro:property name="trunk_izz" value="0.07146322696"/>
     <!-- hip (left front) -->
-    <xacro:property name="hip_mass" value="0.8365"/>
-    <xacro:property name="hip_com_x" value="-0.006155"/>
-    <xacro:property name="hip_com_y" value="-0.006930"/>
-    <xacro:property name="hip_com_z" value="0.000002"/>
-    <xacro:property name="hip_ixx" value="0.000594660"/>
-    <xacro:property name="hip_ixy" value="-0.000009124"/>
-    <xacro:property name="hip_ixz" value="0.000000048"/>
-    <xacro:property name="hip_iyy" value="0.001055081"/>
-    <xacro:property name="hip_iyz" value="0.000000016"/>
-    <xacro:property name="hip_izz" value="0.000764676"/>
+    <xacro:property name="hip_mass" value="1.162"/>
+    <xacro:property name="hip_com_x" value="-0.00758"/>
+    <xacro:property name="hip_com_y" value="-0.00359"/>
+    <xacro:property name="hip_com_z" value="-0.00029"/>
+    <xacro:property name="hip_ixx" value="0.00095157705"/>
+    <xacro:property name="hip_ixy" value="0.00001109670"/>
+    <xacro:property name="hip_ixz" value="-0.00000266665"/>
+    <xacro:property name="hip_iyy" value="0.00159323348"/>
+    <xacro:property name="hip_iyz" value="-0.00001267180"/>
+    <xacro:property name="hip_izz" value="0.00125451931"/>
     <!-- thigh -->
-    <xacro:property name="thigh_mass" value="1.987"/>
-    <xacro:property name="thigh_com_x" value="0.003996"/>
-    <xacro:property name="thigh_com_y" value="0.028346"/>
-    <xacro:property name="thigh_com_z" value="-0.020538"/>
-    <xacro:property name="thigh_ixx" value="0.008811372"/>
-    <xacro:property name="thigh_ixy" value="-0.000167657"/>
-    <xacro:property name="thigh_ixz" value="-0.000632186"/>
-    <xacro:property name="thigh_iyy" value="0.007563533"/>
-    <xacro:property name="thigh_iyz" value="0.001133315"/>
-    <xacro:property name="thigh_izz" value="0.003133589"/>
+    <xacro:property name="thigh_mass" value="1.528"/>
+    <xacro:property name="thigh_com_x" value="0.00033"/>
+    <xacro:property name="thigh_com_y" value="0.03334"/>
+    <xacro:property name="thigh_com_z" value="-0.02983"/>
+    <xacro:property name="thigh_ixx" value="0.00884041519"/>
+    <xacro:property name="thigh_ixy" value="-0.00003381758"/>
+    <xacro:property name="thigh_ixz" value="-0.00005336860"/>
+    <xacro:property name="thigh_iyy" value="0.00784145389"/>
+    <xacro:property name="thigh_iyz" value="0.00128350622"/>
+    <xacro:property name="thigh_izz" value="0.00260045020"/>
     <!-- calf -->
-    <xacro:property name="calf_mass" value="0.213"/>
-    <xacro:property name="calf_com_x" value="-0.000873"/>
-    <xacro:property name="calf_com_y" value="0.000"/>
-    <xacro:property name="calf_com_z" value="-0.114455"/>
-    <xacro:property name="calf_ixx" value="0.001561890"/>
-    <xacro:property name="calf_ixy" value="-0.000"/>
-    <xacro:property name="calf_ixz" value="0.000021547"/>
-    <xacro:property name="calf_iyy" value="0.001566663"/>
-    <xacro:property name="calf_iyz" value="0.000000001"/>
-    <xacro:property name="calf_izz" value="0.000019643"/>
+    <xacro:property name="calf_mass" value="0.132"/>
+    <xacro:property name="calf_com_x" value="0.0016"/>
+    <xacro:property name="calf_com_y" value="0.00438"/>
+    <xacro:property name="calf_com_z" value="-0.12232"/>
+    <xacro:property name="calf_ixx" value="0.00228050753"/>
+    <xacro:property name="calf_ixy" value="-0.00000033551"/>
+    <xacro:property name="calf_ixz" value="0.00000826635"/>
+    <xacro:property name="calf_iyy" value="0.00225891907"/>
+    <xacro:property name="calf_iyz" value="0.00010727008"/>
+    <xacro:property name="calf_izz" value="0.00005160443"/>
 	<!-- foot -->
 	<xacro:property name="foot_mass" value="0.06"/>
+    <!-- pricmatic joint -->
+    <xacro:property name="box_effort_max" value="50"/>
+    <xacro:property name="box_velocity_max" value="50"/>
+    <!-- adjustable leg -->
+    <xacro:property name="box_length" value="0.1691"/>
+    <xacro:property name="box_width" value="0.02"/>
+    <xacro:property name="box_height" value="0.05"/>
+    <xacro:property name="box_mass" value="0.132"/>
+    <xacro:property name="box_ixx" value="0.00228050753"/>
+    <xacro:property name="box_iyy" value="0.00225891907"/>
+    <xacro:property name="box_izz" value="0.00005160443"/>
 </robot>

File: robot_description/arcdog_adjustable_leg_description/xacro/leg.xacro (robot description, xacro)
@@ -1,5 +1,5 @@
 <?xml version="1.0"?>
 <robot xmlns:xacro="http://www.ros.org/wiki/xacro">
-    <xacro:include filename="$(find arcdog_description)/xacro/transmission.xacro"/>
+    <xacro:include filename="$(find arcdog_adjustable_leg_description)/xacro/transmission.xacro"/>
     <xacro:macro name="leg" params="prefix mirror mirror_dae front_hind front_hind_dae simulator robot_type *origin">
         <xacro:if value="${simulator == 'ocs2'}">
@@ -68,16 +68,8 @@
                     <origin rpy="${pi} ${pi} 0" xyz="0 0 0"/>
                 </xacro:if>
-                <xacro:if value="${robot_type == 'arcdog'}">
-                <geometry>
-                    <mesh filename="package://arcdog_description/meshes/hip.stl"
+                <geometry>
+                    <mesh filename="package://arcdog_adjustable_leg_description/assets/hip.stl"
                           scale="1 1 1"/>
                 </geometry>
-                </xacro:if>
-                <xacro:if value="${robot_type == 'arcdog_mini'}">
-                <geometry>
-                    <mesh filename="package://arcdog_description/meshes/hip.stl"
-                          scale="1 1 1"/>
-                </geometry>
-                </xacro:if>
                 <material name="orange"/>
             </visual>
@@ -133,28 +125,14 @@
             <visual>
                 <origin rpy="0 0 0" xyz="0 0 0"/>
-                <xacro:if value="${robot_type == 'arcdog'}">
                 <geometry>
                     <xacro:if value="${mirror_dae == True}">
-                        <mesh filename="package://arcdog_description/meshes/thigh.stl"
+                        <mesh filename="package://arcdog_adjustable_leg_description/assets/thigh.stl"
                               scale="1 1 1"/>
                     </xacro:if>
                     <xacro:if value="${mirror_dae == False}">
-                        <mesh filename="package://arcdog_description/meshes/thigh_mirror.stl"
+                        <mesh filename="package://arcdog_adjustable_leg_description/assets/thigh_mirror.stl"
                               scale="1 1 1"/>
                     </xacro:if>
                 </geometry>
-                </xacro:if>
-                <xacro:if value="${robot_type == 'arcdog_mini'}">
-                <geometry>
-                    <xacro:if value="${mirror_dae == True}">
-                        <mesh filename="package://arcdog_description/meshes/arcdog_mini/thigh.stl"
-                              scale="1 1 1"/>
-                    </xacro:if>
-                    <xacro:if value="${mirror_dae == False}">
-                        <mesh filename="package://arcdog_description/meshes/thigh_mirror.stl"
-                              scale="1 1 1"/>
-                    </xacro:if>
-                </geometry>
-                </xacro:if>
                 <material name="orange"/>
             </visual>
@@ -213,16 +191,8 @@
             <visual>
                 <origin rpy="0 0 0" xyz="0 0 0"/>
-                <xacro:if value="${robot_type == 'arcdog'}">
-                <geometry>
-                    <mesh filename="package://arcdog_description/meshes/calf.stl"
+                <geometry>
+                    <mesh filename="package://arcdog_adjustable_leg_description/assets/calf.stl"
                           scale="1 1 1"/>
                 </geometry>
-                </xacro:if>
-                <xacro:if value="${robot_type == 'arcdog_mini'}">
-                <geometry>
-                    <mesh filename="package://arcdog_description/meshes/calf.stl"
-                          scale="1 1 1"/>
-                </geometry>
-                </xacro:if>
                 <material name="orange"/>
             </visual>
@@ -242,7 +212,41 @@
             </inertial>
         </link>
+        <!-- 在 calf 和 foot 之间添加 box link -->
+        <link name="${prefix}_box">
+            <visual>
+                <origin rpy="0 0 0" xyz="0 0 0"/>
+                <geometry>
+                    <mesh filename="package://arcdog_adjustable_leg_description/assets/adjustable_leg.stl"
+                          scale="1 1 1"/>
+                </geometry>
+                <material name="orange"/>
+            </visual>
+            <collision>
+                <origin rpy="0 0 0" xyz="0 0 0"/>
+                <geometry>
+                    <box size="${box_length} ${box_width} ${box_height}"/>
+                </geometry>
+            </collision>
+            <inertial>
+                <origin rpy="0 0 0" xyz="0 0 0"/>
+                <mass value="${box_mass}"/> <!-- 定义 box 的质量 -->
+                <inertia
+                    ixx="${box_ixx}" ixy="0" ixz="0"
+                    iyy="${box_iyy}" iyz="0"
+                    izz="${box_izz}"/>
+            </inertial>
+        </link>
+        <!-- 添加 prismatic joint -->
+        <joint name="${prefix}_box_joint" type="prismatic">
+            <origin rpy="0 0 0" xyz="0 0 ${-calf_length}"/> <!-- 根据 calf 的长度调整位置 -->
+            <parent link="${prefix}_calf"/>
+            <child link="${prefix}_box"/>
+            <axis xyz="0 0 1"/> <!-- 定义滑动轴 -->
+            <dynamics damping="${damping}" friction="${friction}"/>
+            <limit effort="${box_effort_max}" velocity="${box_velocity_max}" lower="0" upper="${-calf_length}"/> <!-- 定义限制条件 -->
+        </joint>
         <joint name="${prefix}_foot_fixed" type="fixed" dont_collapse="true">
-            <origin rpy="0 0 0" xyz="0 0 ${-(calf_length)}"/>
-            <parent link="${prefix}_calf"/>
+            <origin rpy="0 0 0" xyz="0 0 ${-box_length}"/> <!-- 连接到 box 的底部 -->
+            <parent link="${prefix}_box"/>
             <child link="${prefix}_foot"/>
         </joint>
@@ -290,4 +294,10 @@
             <self_collide>1</self_collide>
         </gazebo>
+        <gazebo reference="${prefix}_box">
+            <mu1>0.4</mu1>  <!-- 根据需要设置静摩擦系数 -->
+            <mu2>0.4</mu2>  <!-- 根据需要设置动摩擦系数 -->
+            <self_collide>0</self_collide>
+            <material>Gazebo/DarkGrey</material>  <!-- 可根据需要更改材料 -->
+        </gazebo>
         <gazebo reference="${prefix}_FOOT">
             <mu1>0.6</mu1>
@@ -298,4 +308,8 @@
             <kd value="100.0"/>
         </gazebo>
+        <gazebo reference="${prefix}_box_joint">
+            <mu1>0.4</mu1>  <!-- 设置滑动关节的摩擦系数 -->
+            <mu2>0.4</mu2>
+        </gazebo>
         <xacro:leg_transmission name="${prefix}"/>
     </xacro:macro>

File: robot_description/arcdog_adjustable_leg_description/xacro/robot.xacro (robot description, xacro)
@@ -1,24 +1,24 @@
 <?xml version="1.0"?>
-<robot name="arcdog" xmlns:xacro="http://www.ros.org/wiki/xacro">
+<robot name="arcdog_adjustable_leg" xmlns:xacro="http://www.ros.org/wiki/xacro">
 	<xacro:arg name="DEBUG" default="false"/>
 	<xacro:arg name="GAZEBO" default="false"/>
 	<xacro:arg name="CLASSIC" default="false"/>
-    <xacro:arg name="robot_type" default="arcdog"/>
+    <xacro:arg name="robot_type" default="arcdog_adjustable_leg"/>
     <xacro:property name="robot_type" value="$(arg robot_type)"/>
 	<xacro:arg name="simulator" default="test"/>
     <xacro:property name="simulator" value="$(arg simulator)"/>
-	<xacro:include filename="$(find arcdog_description)/xacro/const.xacro"/>
-	<xacro:include filename="$(find arcdog_description)/xacro/materials.xacro"/>
-	<xacro:include filename="$(find arcdog_description)/xacro/leg.xacro"/>
+	<xacro:include filename="$(find arcdog_adjustable_leg_description)/xacro/const.xacro"/>
+	<xacro:include filename="$(find arcdog_adjustable_leg_description)/xacro/materials.xacro"/>
+	<xacro:include filename="$(find arcdog_adjustable_leg_description)/xacro/leg.xacro"/>
 	<xacro:if value="$(arg GAZEBO)">
 		<xacro:if value="$(arg CLASSIC)">
-			<xacro:include filename="$(find arcdog_description)/xacro/gazebo_classic.xacro"/>
+			<xacro:include filename="$(find arcdog_adjustable_leg_description)/xacro/gazebo_classic.xacro"/>
 		</xacro:if>
 		<xacro:unless value="$(arg CLASSIC)">
-			<xacro:include filename="$(find arcdog_description)/xacro/gazebo.xacro"/>
+			<xacro:include filename="$(find arcdog_adjustable_leg_description)/xacro/gazebo.xacro"/>
 		</xacro:unless>
 	</xacro:if>
 	<xacro:unless value="$(arg GAZEBO)">
-		<xacro:include filename="$(find arcdog_description)/xacro/ros2_control.xacro"/>
+		<xacro:include filename="$(find arcdog_adjustable_leg_description)/xacro/ros2_control.xacro"/>
 	</xacro:unless>
 	<!-- <xacro:stairs stairs="15" xpos="0" ypos="0" zpos="0" /> -->
@@ -51,5 +51,5 @@
 			<origin rpy="0 0 0" xyz="0 0 0"/>
 			<geometry>
-				<mesh filename="file://$(find arcdog_description)/meshes/trunk.dae" scale="1 1 1"/>
+				<mesh filename="file://$(find arcdog_adjustable_leg_description)/assets/trunk.stl" scale="1 1 1"/>
 			</geometry>
 			<!-- <material name="orange"/> -->
