Commit message: FSM add FixedStandAdjustableLeg

File: robot_description/arcdog_adjustable_leg_description/xacro/ros2_control.xacro (robot description, xacro)
@@ -26,4 +26,14 @@
 		</joint>
 		<joint name="FR_calf_joint">
+			<command_interface name="position"/>
+			<command_interface name="velocity"/>
+			<command_interface name="effort"/>
+			<command_interface name="kp"/>
+			<command_interface name="kd"/>
+			<state_interface name="position"/>
+			<state_interface name="velocity"/>
+			<state_interface name="effort"/>
+		</joint>
+		<joint name="FR_box_joint">
 			<command_interface name="position"/>
 			<command_interface name="velocity"/>
@@ -65,4 +75,14 @@
 			<state_interface name="effort"/>
 		</joint>
+		<joint name="FL_box_joint">
+			<command_interface name="position"/>
+			<command_interface name="velocity"/>
+			<command_interface name="effort"/>
+			<command_interface name="kp"/>
+			<command_interface name="kd"/>
+			<state_interface name="position"/>
+			<state_interface name="velocity"/>
+			<state_interface name="effort"/>
+		</joint>
 		<joint name="RR_hip_joint">
 			<command_interface name="position"/>
@@ -86,4 +106,14 @@
 		</joint>
 		<joint name="RR_calf_joint">
+			<command_interface name="position"/>
+			<command_interface name="velocity"/>
+			<command_interface name="effort"/>
+			<command_interface name="kp"/>
+			<command_interface name="kd"/>
+			<state_interface name="position"/>
+			<state_interface name="velocity"/>
+			<state_interface name="effort"/>
+		</joint>
+		<joint name="RR_box_joint">
 			<command_interface name="position"/>
 			<command_interface name="velocity"/>
@@ -125,4 +155,14 @@
 			<state_interface name="effort"/>
 		</joint>
+		<joint name="RL_box_joint">
+			<command_interface name="position"/>
+			<command_interface name="velocity"/>
+			<command_interface name="effort"/>
+			<command_interface name="kp"/>
+			<command_interface name="kd"/>
+			<state_interface name="position"/>
+			<state_interface name="velocity"/>
+			<state_interface name="effort"/>
+		</joint>
 		<sensor name="imu_sensor">
 			<state_interface name="orientation.w"/>
