Commit message: minor, fix pkg name

File: robot_description/sirius_wheel_description/xacro/const.xacro (robot description, xacro)
@@ -1,4 +1,4 @@
 <?xml version="1.0"?>
-<robot xmlns:xacro="http://www.ros.org/wiki/xacro" name="Sirius_Wheel_description">
+<robot xmlns:xacro="http://www.ros.org/wiki/xacro" name="sirius_wheel_description">
     <!-- Constants for robot dimensions -->
     <xacro:property name="stick_mass" value="0.00001"/>

File: robot_description/sirius_wheel_description/xacro/leg_new_name.xacro (robot description, xacro)
@@ -1,5 +1,5 @@
 <?xml version="1.0" encoding="utf-8" ?>
 <robot xmlns:xacro="http://www.ros.org/wiki/xacro">
-    <xacro:include filename="$(find Sirius_Wheel_description)/xacro/transmission.xacro"/>
+    <xacro:include filename="$(find sirius_wheel_description)/xacro/transmission.xacro"/>
     <!--    left for true, front for true-->
     <xacro:macro name="leg"
@@ -21,17 +21,17 @@
                 <geometry>
                     <xacro:if value="${(left_right_bool == True) and (front_hind_bool == True)}">
-                        <mesh filename="package://Sirius_Wheel_description/simplified_meshes/fl_abad_link.dae"
+                        <mesh filename="package://sirius_wheel_description/simplified_meshes/fl_abad_link.dae"
                               scale="1 1 1"/>
                     </xacro:if>
                     <xacro:if value="${(left_right_bool == False) and (front_hind_bool == True)}">
-                        <mesh filename="package://Sirius_Wheel_description/simplified_meshes/fr_abad_link.dae"
+                        <mesh filename="package://sirius_wheel_description/simplified_meshes/fr_abad_link.dae"
                               scale="1 1 1"/>
                     </xacro:if>
                     <xacro:if value="${(left_right_bool == True) and (front_hind_bool == False)}">
-                        <mesh filename="package://Sirius_Wheel_description/simplified_meshes/rl_abad_link.dae"
+                        <mesh filename="package://sirius_wheel_description/simplified_meshes/rl_abad_link.dae"
                               scale="1 1 1"/>
                     </xacro:if>
                     <xacro:if value="${(left_right_bool == False) and (front_hind_bool == False)}">
-                        <mesh filename="package://Sirius_Wheel_description/simplified_meshes/rr_abad_link.dae"
+                        <mesh filename="package://sirius_wheel_description/simplified_meshes/rr_abad_link.dae"
                               scale="1 1 1"/>
                     </xacro:if>
@@ -52,17 +52,17 @@
             <!--                <geometry>-->
             <!--                    <xacro:if value="${(left_right_bool == True) and (front_hind_bool == True)}">-->
-            <!--                        <mesh filename="package://Sirius_Wheel_description/simplified_meshes/fl_abad_link.dae"-->
+            <!--                        <mesh filename="package://sirius_wheel_description/simplified_meshes/fl_abad_link.dae"-->
             <!--                              scale="1 1 1"/>-->
             <!--                    </xacro:if>-->
             <!--                    <xacro:if value="${(left_right_bool == False) and (front_hind_bool == True)}">-->
-            <!--                        <mesh filename="package://Sirius_Wheel_description/simplified_meshes/fr_abad_link.dae"-->
+            <!--                        <mesh filename="package://sirius_wheel_description/simplified_meshes/fr_abad_link.dae"-->
             <!--                              scale="1 1 1"/>-->
             <!--                    </xacro:if>-->
             <!--                    <xacro:if value="${(left_right_bool == True) and (front_hind_bool == False)}">-->
-            <!--                        <mesh filename="package://Sirius_Wheel_description/simplified_meshes/rl_abad_link.dae"-->
+            <!--                        <mesh filename="package://sirius_wheel_description/simplified_meshes/rl_abad_link.dae"-->
             <!--                              scale="1 1 1"/>-->
             <!--                    </xacro:if>-->
             <!--                    <xacro:if value="${(left_right_bool == False) and (front_hind_bool == False)}">-->
-            <!--                        <mesh filename="package://Sirius_Wheel_description/simplified_meshes/rr_abad_link.dae"-->
+            <!--                        <mesh filename="package://sirius_wheel_description/simplified_meshes/rr_abad_link.dae"-->
             <!--                              scale="1 1 1"/>-->
             <!--                    </xacro:if>-->
@@ -95,17 +95,17 @@
                 <geometry>
                     <xacro:if value="${(left_right_bool == True) and (front_hind_bool == True)}">
-                        <mesh filename="package://Sirius_Wheel_description/simplified_meshes/fl_hip_link.dae"
+                        <mesh filename="package://sirius_wheel_description/simplified_meshes/fl_hip_link.dae"
                               scale="1 1 1"/>
                     </xacro:if>
                     <xacro:if value="${(left_right_bool == False) and (front_hind_bool == True)}">
-                        <mesh filename="package://Sirius_Wheel_description/simplified_meshes/fr_hip_link.dae"
+                        <mesh filename="package://sirius_wheel_description/simplified_meshes/fr_hip_link.dae"
                               scale="1 1 1"/>
                     </xacro:if>
                     <xacro:if value="${(left_right_bool == True) and (front_hind_bool == False)}">
-                        <mesh filename="package://Sirius_Wheel_description/simplified_meshes/rl_hip_link.dae"
+                        <mesh filename="package://sirius_wheel_description/simplified_meshes/rl_hip_link.dae"
                               scale="1 1 1"/>
                     </xacro:if>
                     <xacro:if value="${(left_right_bool == False) and (front_hind_bool == False)}">
-                        <mesh filename="package://Sirius_Wheel_description/simplified_meshes/rr_hip_link.dae"
+                        <mesh filename="package://sirius_wheel_description/simplified_meshes/rr_hip_link.dae"
                               scale="1 1 1"/>
                     </xacro:if>
@@ -159,17 +159,17 @@
                 <geometry>
                     <xacro:if value="${(left_right_bool == True) and (front_hind_bool == True)}">
-                        <mesh filename="package://Sirius_Wheel_description/simplified_meshes/fl_knee_link.dae"
+                        <mesh filename="package://sirius_wheel_description/simplified_meshes/fl_knee_link.dae"
                               scale="1 1 1"/>
                     </xacro:if>
                     <xacro:if value="${(left_right_bool == False) and (front_hind_bool == True)}">
-                        <mesh filename="package://Sirius_Wheel_description/simplified_meshes/fr_knee_link.dae"
+                        <mesh filename="package://sirius_wheel_description/simplified_meshes/fr_knee_link.dae"
                               scale="1 1 1"/>
                     </xacro:if>
                     <xacro:if value="${(left_right_bool == True) and (front_hind_bool == False)}">
-                        <mesh filename="package://Sirius_Wheel_description/simplified_meshes/rl_knee_link.dae"
+                        <mesh filename="package://sirius_wheel_description/simplified_meshes/rl_knee_link.dae"
                               scale="1 1 1"/>
                     </xacro:if>
                     <xacro:if value="${(left_right_bool == False) and (front_hind_bool == False)}">
-                        <mesh filename="package://Sirius_Wheel_description/simplified_meshes/rr_knee_link.dae"
+                        <mesh filename="package://sirius_wheel_description/simplified_meshes/rr_knee_link.dae"
                               scale="1 1 1"/>
                     </xacro:if>
@@ -181,17 +181,17 @@
                 <geometry>
                     <xacro:if value="${(left_right_bool == True) and (front_hind_bool == True)}">
-                        <mesh filename="package://Sirius_Wheel_description/simplified_meshes/fl_knee_link.dae"
+                        <mesh filename="package://sirius_wheel_description/simplified_meshes/fl_knee_link.dae"
                               scale="1 1 1"/>
                     </xacro:if>
                     <xacro:if value="${(left_right_bool == False) and (front_hind_bool == True)}">
-                        <mesh filename="package://Sirius_Wheel_description/simplified_meshes/fr_knee_link.dae"
+                        <mesh filename="package://sirius_wheel_description/simplified_meshes/fr_knee_link.dae"
                               scale="1 1 1"/>
                     </xacro:if>
                     <xacro:if value="${(left_right_bool == True) and (front_hind_bool == False)}">
-                        <mesh filename="package://Sirius_Wheel_description/simplified_meshes/rl_knee_link.dae"
+                        <mesh filename="package://sirius_wheel_description/simplified_meshes/rl_knee_link.dae"
                               scale="1 1 1"/>
                     </xacro:if>
                     <xacro:if value="${(left_right_bool == False) and (front_hind_bool == False)}">
-                        <mesh filename="package://Sirius_Wheel_description/simplified_meshes/rr_knee_link.dae"
+                        <mesh filename="package://sirius_wheel_description/simplified_meshes/rr_knee_link.dae"
                               scale="1 1 1"/>
                     </xacro:if>
@@ -217,5 +217,5 @@
                     <origin rpy="0.0 0 0" xyz="0 0 0"/>
                 <geometry>
-                        <mesh filename="package://Sirius_Wheel_description/simplified_meshes/wheel_motor.STL"
+                        <mesh filename="package://sirius_wheel_description/simplified_meshes/wheel_motor.STL"
                               scale="1 1 1"/>
                 </geometry>
@@ -245,5 +245,5 @@
                     <origin rpy="0 0 0" xyz="0 0 0"/>
                 <geometry>
-                        <mesh filename="package://Sirius_Wheel_description/simplified_meshes/wheel_link.STL"
+                        <mesh filename="package://sirius_wheel_description/simplified_meshes/wheel_link.STL"
                               scale="1 1 1"/>
                 </geometry>

File: robot_description/sirius_wheel_description/xacro/robot.xacro (robot description, xacro)
@@ -1,4 +1,4 @@
 <?xml version="1.0"?>
-<robot xmlns:xacro="http://www.ros.org/wiki/xacro" name="Sirius_Wheel_description">
+<robot xmlns:xacro="http://www.ros.org/wiki/xacro" name="sirius_wheel_description">
     <xacro:arg name="DEBUG" default="false"/>
     <xacro:include filename="$(find sirius_wheel_description)/xacro/materials.xacro"/>

File: robot_description/sirius_wheel_description/xacro/robot_original.xacro (robot description, xacro)
@@ -1,11 +1,11 @@
 <?xml version="1.0"?>
-<robot xmlns:xacro="http://www.ros.org/wiki/xacro" name="Sirius_Wheel_description">
+<robot xmlns:xacro="http://www.ros.org/wiki/xacro" name="sirius_wheel_description">
     <xacro:arg name="DEBUG" default="false"/>
-    <xacro:include filename="$(find Sirius_Wheel_description)/xacro/materials.xacro"/>
-    <xacro:include filename="$(find Sirius_Wheel_description)/xacro/leg.xacro"/>
-    <xacro:include filename="$(find Sirius_Wheel_description)/xacro/gazebo.xacro"/>
-    <xacro:include filename="$(find Sirius_Wheel_description)/xacro/const.xacro"/>
-    <!--   <xacro:include filename="$(find Sirius_Wheel_description)/xacro/ros2_control_real_robot.xacro"/>-->
-    <xacro:include filename="$(find Sirius_Wheel_description)/xacro/ros2_control.xacro"/>
+    <xacro:include filename="$(find sirius_wheel_description)/xacro/materials.xacro"/>
+    <xacro:include filename="$(find sirius_wheel_description)/xacro/leg.xacro"/>
+    <xacro:include filename="$(find sirius_wheel_description)/xacro/gazebo.xacro"/>
+    <xacro:include filename="$(find sirius_wheel_description)/xacro/const.xacro"/>
+    <!--   <xacro:include filename="$(find sirius_wheel_description)/xacro/ros2_control_real_robot.xacro"/>-->
+    <xacro:include filename="$(find sirius_wheel_description)/xacro/ros2_control.xacro"/>
     <xacro:if value="$(arg DEBUG)">
         <link name="world"/>
@@ -33,5 +33,5 @@
             <origin rpy="0 0 0" xyz="-0 0 0"/>
             <geometry>
-                <mesh filename="package://Sirius_Wheel_description/simplified_meshes/base_link.dae" scale="1 1 1"/>
+                <mesh filename="package://sirius_wheel_description/simplified_meshes/base_link.dae" scale="1 1 1"/>
             </geometry>
         </visual>
@@ -39,5 +39,5 @@
             <origin rpy="0 0 0" xyz="0 0 0"/>
             <geometry>
-<!--                <mesh filename="package://Sirius_Wheel_description/simplified_meshes/base_link.dae" scale="1 1 1"/>-->
+<!--                <mesh filename="package://sirius_wheel_description/simplified_meshes/base_link.dae" scale="1 1 1"/>-->
                 <box size="${base_length} ${base_width} ${base_height}"/>
             </geometry>

Commit message: feat: Add height trigger to SiriusW env

File: robot_description/sirius_wheel_description/xacro/const.xacro (robot description, xacro)
@@ -21,5 +21,5 @@
     <xacro:property name="abad_radius" value="0.055"/>
     <xacro:property name="abad_length" value="0.09"/>
-    <xacro:property name="wheel_origin_z" value="-0.024"/>
+    <xacro:property name="wheel_origin_z" value="0.0"/>
     <xacro:property name="wheel_radius" value="0.10025"/>
     <xacro:property name="wheel_length" value="0.05"/>
