Commit message: update new arcdog visual and xacro model

File: robot_description/arcdog_description/xacro/arcdog.xacro (robot description, xacro)
@@ -1,142 +1,77 @@
 <?xml version="1.0"?>
-<robot name="arcdog" xmlns:xacro="http://www.ros.org/wiki/xacro">
-	<xacro:arg name="DEBUG" default="false"/>
-	<xacro:arg name="GAZEBO" default="false"/>
-	<xacro:arg name="CLASSIC" default="false"/>
+<robot xmlns:xacro="http://www.ros.org/wiki/xacro" name="arcdog_description">
     <xacro:arg name="robot_type" default="arcdog"/>
     <xacro:property name="robot_type" value="$(arg robot_type)"/>
-	<xacro:arg name="simulator" default="test"/>
+    <!-- Is the robot to be used with a simulator or control software -->
+    <!-- Supported: none, gazebo, mujoco -->
+    <xacro:arg name="simulator" default="test"/>
     <xacro:property name="simulator" value="$(arg simulator)"/>
-	<xacro:include filename="$(find arcdog_description)/xacro/const.xacro"/>
-	<xacro:include filename="$(find arcdog_description)/xacro/materials.xacro"/>
-	<xacro:include filename="$(find arcdog_description)/xacro/leg.xacro"/>
-	<xacro:if value="$(arg GAZEBO)">
-		<xacro:if value="$(arg CLASSIC)">
-			<xacro:include filename="$(find arcdog_description)/xacro/gazebo_classic.xacro"/>
-		</xacro:if>
-		<xacro:unless value="$(arg CLASSIC)">
-			<xacro:include filename="$(find arcdog_description)/xacro/gazebo.xacro"/>
-		</xacro:unless>
-	</xacro:if>
-	<xacro:unless value="$(arg GAZEBO)">
-		<xacro:include filename="$(find arcdog_description)/xacro/ros2_control.xacro"/>
-	</xacro:unless>
-	<!-- <xacro:stairs stairs="15" xpos="0" ypos="0" zpos="0" /> -->
-	<!-- Rotor related joint and link is only for demonstrate location. -->
-	<!-- Actually, the rotor will rotate and the joint is not fixed. Reduction ratio should be considered. -->
-	<!-- Debug mode will hung up the robot, use "true" or "false" to switch it. -->
-	<xacro:if value="$(arg DEBUG)">
-		<link name="world"/>
-		<joint name="base_static_joint" type="fixed">
-			<origin rpy="0 0 0" xyz="0 0 0"/>
-			<parent link="world"/>
-			<child link="base"/>
-		</joint>
-	</xacro:if>
-	<link name="base">
-		<visual>
-			<origin rpy="0 0 0" xyz="0 0 0"/>
-			<geometry>
-				<box size="0.001 0.001 0.001"/>
-			</geometry>
-		</visual>
-	</link>
-	<joint name="floating_base" type="fixed">
-		<origin rpy="0 0 0" xyz="0 0 0"/>
-		<parent link="base"/>
-		<child link="trunk"/>
-	</joint>
-	<link name="trunk">
-		<visual>
-			<origin rpy="0 0 0" xyz="0 0 0"/>
-			<geometry>
-				<mesh filename="file://$(find arcdog_description)/meshes/trunk.dae" scale="1 1 1"/>
-			</geometry>
-			<!-- <material name="orange"/> -->
-		</visual>
-		<collision>
-			<origin rpy="0 0 0" xyz="0 0 0"/>
-			<geometry>
-				<box size="${trunk_length} ${trunk_width} ${trunk_height}"/>
-			</geometry>
-		</collision>
-		<collision>
-			<origin rpy="0 0 0" xyz="0 0 0"/>
-			<geometry>
-				<box size="0.1881 0.04675 0.057"/>
-			</geometry>
-		</collision>
-		<collision>
-			<origin rpy="0 0 0" xyz="0.285 0 0.01"/>
-			<geometry>
-				<cylinder length="0.05" radius="0.045"/>
-			</geometry>
-		</collision>
-		<collision>
-			<origin rpy="0 0 0" xyz="0.293 0 -0.06"/>
-			<geometry>
-				<box size="0.047 0.047 0.047"/>
-			</geometry>
-		</collision>
-		<inertial>
-			<origin rpy="0 0 0" xyz="${trunk_com_x} ${trunk_com_y} ${trunk_com_z}"/>
-			<mass value="${trunk_mass}"/>
-			<inertia
-							ixx="${trunk_ixx}" ixy="${trunk_ixy}" ixz="${trunk_ixz}"
-							iyy="${trunk_iyy}" iyz="${trunk_iyz}"
-							izz="${trunk_izz}"/>
-		</inertial>
-	</link>
-	<joint name="imu_joint" type="fixed">
-		<parent link="trunk"/>
-		<child link="imu_link"/>
-		<origin rpy="0 0 0" xyz="0 0 0"/>
-	</joint>
-	<link name="imu_link">
-		<inertial>
-			<mass value="0.001"/>
-			<origin rpy="0 0 0" xyz="0 0 0"/>
-			<inertia ixx="0.0001" ixy="0" ixz="0" iyy="0.0001" iyz="0" izz="0.0001"/>
-		</inertial>
-		<visual>
-			<origin rpy="0 0 0" xyz="0 0 0"/>
-			<geometry>
-				<box size="0.001 0.001 0.001"/>
-			</geometry>
-			<!-- <material name="red"/> -->
-		</visual>
-		<collision>
-			<origin rpy="0 0 0" xyz="0 0 0"/>
-			<geometry>
-				<box size=".001 .001 .001"/>
-			</geometry>
-		</collision>
-	</link>
-	<!--
-	<joint name="load_joint" type="fixed">
-			<parent link="trunk"/>
-			<child link="load_link"/>
-			<origin rpy="0 0 0" xyz="0 0 0"/>
-	</joint>
-	<link name="load_link">
-			<inertial>
-					<mass value="5"/>
-					<origin rpy="0 0 0" xyz="0 0 0"/>
-					<inertia ixx="0.01" ixy="0" ixz="0" iyy="0.01" iyz="0" izz="0.01"/>
-			</inertial>
-			<visual>
-					<origin rpy="0 0 0" xyz="0 0 0.2"/>
-					<geometry>
-							<box size="0.5 0.3 0.2"/>
-					</geometry>
-			</visual>
-			<collision>
-					<origin rpy="0 0 0" xyz="0 0 0"/>
-					<geometry>
-							<box size=".001 .001 .001"/>
-					</geometry>
-			</collision>
-	</link>
--->
+   <xacro:include filename="$(find arcdog_description)/xacro/const.xacro"/>
+    <xacro:include filename="$(find arcdog_description)/xacro/materials.xacro"/>
+    <xacro:include filename="$(find arcdog_description)/xacro/leg.xacro"/>
+    <xacro:include filename="$(find arcdog_description)/xacro/gazebo.xacro"/>
+    <xacro:include filename="$(find arcdog_description)/xacro/imu.xacro"/>
+    <link name="body">
+        <visual>
+            <origin rpy="0 0 0" xyz="0 0 0"/>
+            <geometry>
+                <box size="0.001 0.001 0.001"/>
+            </geometry>
+        </visual>
+    </link>
+    <joint name="floating_base" type="fixed">
+        <origin rpy="0 0 0" xyz="0 0 0"/>
+        <parent link="body"/>
+        <child link="base"/>
+    </joint>
+    <link name="base">
+        <visual>
+            <origin rpy="0 0 0" xyz="0 0 0"/>
+            <geometry>
+                <mesh filename="file://$(find arcdog_description)/meshes/trunk.dae" scale="1 1 1"/>
+            </geometry>
+        </visual>
+        <collision>
+            <origin rpy="0 0 0" xyz="0 0 0"/>
+            <geometry>
+                <box size="${trunk_length} ${trunk_width} ${trunk_height}"/>
+            </geometry>
+        </collision>
+        <inertial>
+            <origin rpy="0 0 0" xyz="${trunk_com_x} ${trunk_com_y} ${trunk_com_z}"/>
+            <mass value="${trunk_mass}"/>
+            <inertia
+                    ixx="${trunk_ixx}" ixy="${trunk_ixy}" ixz="${trunk_ixz}"
+                    iyy="${trunk_iyy}" iyz="${trunk_iyz}"
+                    izz="${trunk_izz}"/>
+        </inertial>
+    </link>
+    <joint name="unitree_imu_joint" type="fixed">
+        <origin rpy="0. 0. 0." xyz="0. 0. 0."/>
+        <parent link="base"/>
+        <child link="unitree_imu"/>
+    </joint>
+    <link name="unitree_imu">
+        <inertial>
+            <mass value="0.01"/>
+            <origin rpy="0 0 0" xyz="0 0 0"/>
+            <inertia ixx="0.000001" ixy="0" ixz="0" iyy="0.000001" iyz="0" izz="0.000001"/>
+        </inertial>
+        <visual>
+            <origin rpy="0 0 0" xyz="0 0 0"/>
+            <geometry>
+                <box size="0.015 0.015 0.004"/>
+            </geometry>
+        </visual>
+        <material name="orange">
+            <color rgba="255 108 10 255"/>
+        </material>
+    </link>
+    <gazebo reference="unitree_imu">
+        <material>Gazebo/Orange</material>
+    </gazebo>
+    <gazebo reference="unitree_imu_joint">
+        <disableFixedJointLumping>true</disableFixedJointLumping>
+    </gazebo>
     <xacro:leg prefix="FR" mirror="-1" mirror_dae="False" front_hind="1" front_hind_dae="True" simulator="${simulator}" robot_type="${robot_type}">
         <origin rpy="0 0 0" xyz="${leg_offset_x} ${-leg_offset_y} 0"/>

File: robot_description/arcdog_description/xacro/leg.xacro (robot description, xacro)
@@ -21,7 +21,7 @@
         </xacro:if>
         <xacro:if value="${simulator == 'test'}">
-            <joint name="${prefix}_hip_joint" type="revolute">
+            <joint name="${prefix}_HAA" type="revolute">
                 <xacro:insert_block name="origin"/>
-                <parent link="trunk"/>
+                <parent link="base"/>
                 <child link="${prefix}_hip"/>
                 <axis xyz="1 0 0"/>
@@ -37,21 +37,4 @@
             </joint>
         </xacro:if>
-        <xacro:if value="${simulator == 'mujoco'}">
-            <joint name="${prefix}_hip_joint" type="revolute">
-                <xacro:insert_block name="origin"/>
-                <parent link="trunk"/>
-                <child link="${prefix}_hip"/>
-                <axis xyz="1 0 0"/>
-                <dynamics damping="${damping}" friction="${friction}"/>
-                <xacro:if value="${(mirror_dae == True)}">
-                    <limit effort="${hip_torque_max}" velocity="${hip_velocity_max}" lower="${hip_min}"
-                        upper="${hip_max}"/>
-                </xacro:if>
-                <xacro:if value="${(mirror_dae == False)}">
-                    <limit effort="${hip_torque_max}" velocity="${hip_velocity_max}" lower="${-hip_max}"
-                        upper="${-hip_min}"/>
-                </xacro:if>
-            </joint>
-        </xacro:if>
         <link name="${prefix}_hip">
             <visual>
@@ -68,16 +51,8 @@
                     <origin rpy="${pi} ${pi} 0" xyz="0 0 0"/>
                 </xacro:if>
-                <xacro:if value="${robot_type == 'arcdog'}">
-                <geometry>
-                    <mesh filename="package://arcdog_description/meshes/hip.stl"
+                <geometry>
+                    <mesh filename="package://arcdog_description/meshes/hip.dae"
                           scale="1 1 1"/>
                 </geometry>
-                </xacro:if>
-                <xacro:if value="${robot_type == 'arcdog_mini'}">
-                <geometry>
-                    <mesh filename="package://arcdog_description/meshes/hip.stl"
-                          scale="1 1 1"/>
-                </geometry>
-                </xacro:if>
                 <material name="orange"/>
             </visual>
@@ -109,5 +84,5 @@
         </xacro:if>
         <xacro:if value="${simulator == 'test'}">
-            <joint name="${prefix}_thigh_joint" type="revolute">
+            <joint name="${prefix}_HFE" type="revolute">
                 <origin rpy="0 0 0" xyz="0 ${thigh_offset*mirror} 0"/>
                 <parent link="${prefix}_hip"/>
@@ -119,42 +94,17 @@
             </joint>
         </xacro:if>
-        <xacro:if value="${simulator == 'mujoco'}">
-            <joint name="${prefix}_thigh_joint" type="revolute">
-                <origin rpy="0 0 0" xyz="0 ${thigh_offset*mirror} 0"/>
-                <parent link="${prefix}_hip"/>
-                <child link="${prefix}_thigh"/>
-                <axis xyz="0 1 0"/>
-                <dynamics damping="${damping}" friction="${friction}"/>
-                <limit effort="${thigh_torque_max}" velocity="${thigh_velocity_max}" lower="${thigh_min}"
-                    upper="${thigh_max}"/>
-            </joint>
-        </xacro:if>
         <link name="${prefix}_thigh">
             <visual>
                 <origin rpy="0 0 0" xyz="0 0 0"/>
-                <xacro:if value="${robot_type == 'arcdog'}">
                 <geometry>
                     <xacro:if value="${mirror_dae == True}">
-                        <mesh filename="package://arcdog_description/meshes/thigh.stl"
+                        <mesh filename="package://arcdog_description/meshes/thigh.dae"
                               scale="1 1 1"/>
                     </xacro:if>
                     <xacro:if value="${mirror_dae == False}">
-                        <mesh filename="package://arcdog_description/meshes/thigh_mirror.stl"
+                        <mesh filename="package://arcdog_description/meshes/thigh_mirror.dae"
                               scale="1 1 1"/>
                     </xacro:if>
                 </geometry>
-                </xacro:if>
-                <xacro:if value="${robot_type == 'arcdog_mini'}">
-                <geometry>
-                    <xacro:if value="${mirror_dae == True}">
-                        <mesh filename="package://arcdog_description/meshes/arcdog_mini/thigh.stl"
-                              scale="1 1 1"/>
-                    </xacro:if>
-                    <xacro:if value="${mirror_dae == False}">
-                        <mesh filename="package://arcdog_description/meshes/thigh_mirror.stl"
-                              scale="1 1 1"/>
-                    </xacro:if>
-                </geometry>
-                </xacro:if>
                 <material name="orange"/>
             </visual>
@@ -191,5 +141,5 @@
         </xacro:if>
         <xacro:if value="${simulator == 'test'}">
-            <joint name="${prefix}_calf_joint" type="revolute">
+            <joint name="${prefix}_KFE" type="revolute">
                 <origin rpy="0 0 0" xyz="0 0 ${-thigh_length}"/>
                 <parent link="${prefix}_thigh"/>
@@ -200,29 +150,11 @@
             </joint>
         </xacro:if>
-        <xacro:if value="${simulator == 'mujoco'}">
-            <joint name="${prefix}_calf_joint" type="revolute">
-                <origin rpy="0 0 0" xyz="0 0 ${-thigh_length}"/>
-                <parent link="${prefix}_thigh"/>
-                <child link="${prefix}_calf"/>
-                <axis xyz="0 1 0"/>
-                <dynamics damping="${damping}" friction="${friction}"/>
-                <limit effort="${calf_torque_max}" velocity="${calf_velocity_max}" lower="${calf_min}" upper="${calf_max}"/>
-            </joint>
-        </xacro:if>
         <link name="${prefix}_calf">
             <visual>
                 <origin rpy="0 0 0" xyz="0 0 0"/>
-                <xacro:if value="${robot_type == 'arcdog'}">
-                <geometry>
-                    <mesh filename="package://arcdog_description/meshes/calf.stl"
+                <geometry>
+                   <mesh filename="package://arcdog_description/meshes/calf.dae"
                           scale="1 1 1"/>
                 </geometry>
-                </xacro:if>
-                <xacro:if value="${robot_type == 'arcdog_mini'}">
-                <geometry>
-                    <mesh filename="package://arcdog_description/meshes/calf.stl"
-                          scale="1 1 1"/>
-                </geometry>
-                </xacro:if>
                 <material name="orange"/>
             </visual>
@@ -243,5 +175,5 @@
         </link>
         <joint name="${prefix}_foot_fixed" type="fixed" dont_collapse="true">
-            <origin rpy="0 0 0" xyz="0 0 ${-(calf_length)}"/>
+            <origin rpy="0 0 0" xyz="0 0 ${-calf_length}"/>
             <parent link="${prefix}_calf"/>
             <child link="${prefix}_foot"/>
@@ -260,4 +192,32 @@
                     <sphere radius="${foot_radius}"/>
                 </geometry>
+                <surface>
+                <bounce>
+                    <restitution_coefficient>0</restitution_coefficient>
+                    <threshold>1e+06</threshold>
+                </bounce>
+                <friction>
+                    <ode>
+                    <mu>1.0</mu>
+                    <mu2>1.0</mu2>
+                    </ode>
+                    <bullet>
+                    <rolling_friction>0.3</rolling_friction>
+                    <friction2>50</friction2>
+                    </bullet>
+                </friction>
+                <contact>
+                    <ode>
+                    <kp>30000.0</kp>
+                    <kd>1000.0</kd>
+                    </ode>
+                    <bullet>
+                    <kp>30000.0</kp>
+                    <kd>1000.0</kd>
+                    <split_impulse>1</split_impulse>
+                    <split_impulse_penetration_threshold>-0.01</split_impulse_penetration_threshold>
+                    </bullet>
+                </contact>
+                </surface>
             </collision>
             <inertial>

Commit message: modify size and collision value

File: robot_description/arcdog_description/xacro/arcdog.xacro (robot description, xacro)
@@ -29,5 +29,5 @@
             <origin rpy="0 0 0" xyz="0 0 0"/>
             <geometry>
-                <mesh filename="file://$(find arcdog_description)/meshes/trunk.dae" scale="1 1 1"/>
+                <mesh filename="file://$(find arcdog_description)/meshes/trunk1.dae" scale="1 1 1"/>
             </geometry>
         </visual>

File: robot_description/arcdog_description/xacro/const.xacro (robot description, xacro)
@@ -1,45 +1,31 @@
 <?xml version="1.0"?>
-<robot xmlns:xacro="http://www.ros.org/wiki/xacro">
-	<!-- Constants for robot dimensions -->
-	<xacro:property name="PI" value="3.1415926535897931"/>
-	<xacro:property name="stick_mass" value="0.00001"/>
-	<!-- simplified collision value -->
-    <xacro:property name="trunk_width" value="0.121"/>
-    <xacro:property name="trunk_length" value="0.548"/>
-    <xacro:property name="trunk_height" value="0.116"/>
-    <xacro:property name="hip_radius" value="0.041"/>
-    <xacro:property name="hip_length" value=" 0.1095"/>
-    <xacro:property name="thigh_shoulder_radius" value="0.044"/>
-    <xacro:property name="thigh_shoulder_length" value="0.0985"/>
-    <xacro:property name="thigh_shoulder_y_offset" value="0.0"/> //TODO
-    <xacro:property name="thigh_width" value="0.088"/>
+<robot xmlns:xacro="http://www.ros.org/wiki/xacro" name="arcdog_description">
+    <!-- Constants for robot dimensions -->
+    <xacro:property name="stick_mass" value="0.00001"/>
+    <!-- simplified collision value -->
+    <xacro:property name="trunk_width" value="0.250"/>
+    <xacro:property name="trunk_length" value="0.361"/>
+    <xacro:property name="trunk_height" value="0.114"/>
+    <xacro:property name="hip_radius" value="0.0495"/>
+    <xacro:property name="hip_length" value=" 0.0834"/>
+    <xacro:property name="thigh_shoulder_radius" value="0.0495"/>
+    <xacro:property name="thigh_shoulder_length" value="0.03826"/>
+    <xacro:property name="thigh_shoulder_y_offset" value="0.0"/>
+    <xacro:property name="thigh_width" value="0.040"/> //little larger than real value
     <xacro:property name="thigh_height" value="0.06797"/>
-    <xacro:property name="thigh_x_offset" value="0.000"/> //TODO
+    <xacro:property name="thigh_x_offset" value="0.000"/>
     <xacro:property name="calf_width" value="0.02"/>
     <xacro:property name="calf_height" value="0.05"/>
-    <xacro:property name="calf_x_offset" value="0.000"/> //TODO
-	<xacro:property name="foot_radius" value="0.0265"/>
-	<xacro:property name="stick_radius" value="0.01"/>
-	<xacro:property name="stick_length" value="0.2"/>
-	<!-- kinematic value -->
-	<xacro:property name="thigh_offset" value="0.0955"/>
-	<xacro:property name="thigh_length" value="0.213"/>
-	<xacro:property name="calf_length" value="0.213"/>
+    <xacro:property name="calf_x_offset" value="0.000"/>
+    <xacro:property name="foot_radius" value="0.0265"/>
+    <!-- kinematic value -->
+    <xacro:property name="thigh_offset" value="0.11475"/>
+    <xacro:property name="thigh_length" value="0.245"/>
+    <xacro:property name="calf_length" value="0.19534"/>
     <!-- leg offset from trunk center value -->
-    <xacro:property name="leg_offset_x" value="0.274"/>
+    <xacro:property name="leg_offset_x" value="0.2515"/>
     <xacro:property name="leg_offset_y" value="0.0605"/>
     <xacro:property name="trunk_offset_z" value="0.01675"/> //TODO
     <xacro:property name="hip_offset" value="0.0001"/> //TODO
-	<!-- offset of link locations (left front) -->
-	<xacro:property name="hip_offset_x" value="0.1934"/>
-	<xacro:property name="hip_offset_y" value="0.0465"/>
-	<xacro:property name="hip_offset_z" value="0.0"/>
-    <!-- kinematic value -->
-    <xacro:property name="thigh_offset" value="0.1095"/>
-    <xacro:property name="thigh_length" value="0.2445"/>
-    <xacro:property name="calf_length" value="0.23704"/>
-	<xacro:property name="calf_offset_x" value="0.0"/>
-	<xacro:property name="calf_offset_y" value="0.0"/>
-	<xacro:property name="calf_offset_z" value="-0.213"/>
     <!-- joint limits -->
     <xacro:property name="damping" value="0.05"/>
@@ -102,5 +88,5 @@
     <xacro:property name="calf_iyz" value="0.000000001"/>
     <xacro:property name="calf_izz" value="0.000019643"/>
-	<!-- foot -->
-	<xacro:property name="foot_mass" value="0.06"/>
+    <!-- foot -->
+    <xacro:property name="foot_mass" value="0.06"/>
 </robot>

File: robot_description/arcdog_description/xacro/leg.xacro (robot description, xacro)
@@ -52,5 +52,5 @@
                 </xacro:if>
                 <geometry>
-                    <mesh filename="package://arcdog_description/meshes/hip.dae"
+                    <mesh filename="package://arcdog_description/meshes/hip1.dae"
                           scale="1 1 1"/>
                 </geometry>
@@ -99,9 +99,9 @@
                 <geometry>
                     <xacro:if value="${mirror_dae == True}">
-                        <mesh filename="package://arcdog_description/meshes/thigh.dae"
+                        <mesh filename="package://arcdog_description/meshes/thigh1.dae"
                               scale="1 1 1"/>
                     </xacro:if>
                     <xacro:if value="${mirror_dae == False}">
-                        <mesh filename="package://arcdog_description/meshes/thigh_mirror.dae"
+                        <mesh filename="package://arcdog_description/meshes/thigh_mirror1.dae"
                               scale="1 1 1"/>
                     </xacro:if>
@@ -110,5 +110,5 @@
             </visual>
             <collision>
-                <origin rpy="0 ${pi/2.0+0.1} 0" xyz="${thigh_x_offset} 0 ${-thigh_length/2.0}"/>
+                <origin rpy="0 ${pi/2.0} 0" xyz="${thigh_x_offset} 0 ${-thigh_length/2.0}"/>
                 <geometry>
                     <box size="${thigh_length} ${thigh_width} ${thigh_height}"/>
@@ -154,5 +154,5 @@
                 <origin rpy="0 0 0" xyz="0 0 0"/>
                 <geometry>
-                   <mesh filename="package://arcdog_description/meshes/calf.dae"
+                   <mesh filename="package://arcdog_description/meshes/calf1.dae"
                           scale="1 1 1"/>
                 </geometry>
