Commit message: new arcdog sim to sim

File: robot_description/arcdog_description/xacro/leg copy.xacro (robot description, xacro)
@@ -23,5 +23,22 @@
             <joint name="${prefix}_hip_joint" type="revolute">
                 <xacro:insert_block name="origin"/>
-                <parent link="base"/>
+                <parent link="trunk"/>
+                <child link="${prefix}_hip"/>
+                <axis xyz="1 0 0"/>
+                <dynamics damping="${damping}" friction="${friction}"/>
+                <xacro:if value="${(mirror_dae == True)}">
+                    <limit effort="${hip_torque_max}" velocity="${hip_velocity_max}" lower="${hip_min}"
+                        upper="${hip_max}"/>
+                </xacro:if>
+                <xacro:if value="${(mirror_dae == False)}">
+                    <limit effort="${hip_torque_max}" velocity="${hip_velocity_max}" lower="${-hip_max}"
+                        upper="${-hip_min}"/>
+                </xacro:if>
+            </joint>
+        </xacro:if>
+        <xacro:if value="${simulator == 'mujoco'}">
+            <joint name="${prefix}_hip_joint" type="revolute">
+                <xacro:insert_block name="origin"/>
+                <parent link="trunk"/>
                 <child link="${prefix}_hip"/>
                 <axis xyz="1 0 0"/>
@@ -51,8 +68,16 @@
                     <origin rpy="${pi} ${pi} 0" xyz="0 0 0"/>
                 </xacro:if>
+                <xacro:if value="${robot_type == 'arcdog'}">
                 <geometry>
                     <mesh filename="package://arcdog_description/meshes/hip.stl"
                           scale="1 1 1"/>
                 </geometry>
+                </xacro:if>
+                <xacro:if value="${robot_type == 'arcdog_mini'}">
+                <geometry>
+                    <mesh filename="package://arcdog_description/meshes/hip.stl"
+                          scale="1 1 1"/>
+                </geometry>
+                </xacro:if>
                 <material name="orange"/>
             </visual>
@@ -94,7 +119,19 @@
             </joint>
         </xacro:if>
+        <xacro:if value="${simulator == 'mujoco'}">
+            <joint name="${prefix}_thigh_joint" type="revolute">
+                <origin rpy="0 0 0" xyz="0 ${thigh_offset*mirror} 0"/>
+                <parent link="${prefix}_hip"/>
+                <child link="${prefix}_thigh"/>
+                <axis xyz="0 1 0"/>
+                <dynamics damping="${damping}" friction="${friction}"/>
+                <limit effort="${thigh_torque_max}" velocity="${thigh_velocity_max}" lower="${thigh_min}"
+                    upper="${thigh_max}"/>
+            </joint>
+        </xacro:if>
         <link name="${prefix}_thigh">
             <visual>
                 <origin rpy="0 0 0" xyz="0 0 0"/>
+                <xacro:if value="${robot_type == 'arcdog'}">
                 <geometry>
                     <xacro:if value="${mirror_dae == True}">
@@ -107,8 +144,21 @@
                     </xacro:if>
                 </geometry>
+                </xacro:if>
+                <xacro:if value="${robot_type == 'arcdog_mini'}">
+                <geometry>
+                    <xacro:if value="${mirror_dae == True}">
+                        <mesh filename="package://arcdog_description/meshes/arcdog_mini/thigh.stl"
+                              scale="1 1 1"/>
+                    </xacro:if>
+                    <xacro:if value="${mirror_dae == False}">
+                        <mesh filename="package://arcdog_description/meshes/thigh_mirror.stl"
+                              scale="1 1 1"/>
+                    </xacro:if>
+                </geometry>
+                </xacro:if>
                 <material name="orange"/>
             </visual>
             <collision>
-                <origin rpy="0 ${pi/2.0} 0" xyz="${thigh_x_offset} 0 ${-thigh_length/2.0}"/>
+                <origin rpy="0 ${pi/2.0+0.1} 0" xyz="${thigh_x_offset} 0 ${-thigh_length/2.0}"/>
                 <geometry>
                     <box size="${thigh_length} ${thigh_width} ${thigh_height}"/>
@@ -150,11 +200,29 @@
             </joint>
         </xacro:if>
+        <xacro:if value="${simulator == 'mujoco'}">
+            <joint name="${prefix}_calf_joint" type="revolute">
+                <origin rpy="0 0 0" xyz="0 0 ${-thigh_length}"/>
+                <parent link="${prefix}_thigh"/>
+                <child link="${prefix}_calf"/>
+                <axis xyz="0 1 0"/>
+                <dynamics damping="${damping}" friction="${friction}"/>
+                <limit effort="${calf_torque_max}" velocity="${calf_velocity_max}" lower="${calf_min}" upper="${calf_max}"/>
+            </joint>
+        </xacro:if>
         <link name="${prefix}_calf">
             <visual>
                 <origin rpy="0 0 0" xyz="0 0 0"/>
+                <xacro:if value="${robot_type == 'arcdog'}">
                 <geometry>
                     <mesh filename="package://arcdog_description/meshes/calf.stl"
                           scale="1 1 1"/>
                 </geometry>
+                </xacro:if>
+                <xacro:if value="${robot_type == 'arcdog_mini'}">
+                <geometry>
+                    <mesh filename="package://arcdog_description/meshes/calf.stl"
+                          scale="1 1 1"/>
+                </geometry>
+                </xacro:if>
                 <material name="orange"/>
             </visual>
@@ -175,5 +243,5 @@
         </link>
         <joint name="${prefix}_foot_fixed" type="fixed" dont_collapse="true">
-            <origin rpy="0 0 0" xyz="0 0 ${-calf_length}"/>
+            <origin rpy="0 0 0" xyz="0 0 ${-(calf_length)}"/>
             <parent link="${prefix}_calf"/>
             <child link="${prefix}_foot"/>
@@ -192,32 +260,4 @@
                     <sphere radius="${foot_radius}"/>
                 </geometry>
-                <surface>
-                <bounce>
-                    <restitution_coefficient>0</restitution_coefficient>
-                    <threshold>1e+06</threshold>
-                </bounce>
-                <friction>
-                    <ode>
-                    <mu>1.0</mu>
-                    <mu2>1.0</mu2>
-                    </ode>
-                    <bullet>
-                    <rolling_friction>0.3</rolling_friction>
-                    <friction2>50</friction2>
-                    </bullet>
-                </friction>
-                <contact>
-                    <ode>
-                    <kp>30000.0</kp>
-                    <kd>1000.0</kd>
-                    </ode>
-                    <bullet>
-                    <kp>30000.0</kp>
-                    <kd>1000.0</kd>
-                    <split_impulse>1</split_impulse>
-                    <split_impulse_penetration_threshold>-0.01</split_impulse_penetration_threshold>
-                    </bullet>
-                </contact>
-                </surface>
             </collision>
             <inertial>

File: robot_description/arcdog_description/xacro/robot.xacro (robot description, xacro)
@@ -51,5 +51,5 @@
 			<origin rpy="0 0 0" xyz="0 0 0"/>
 			<geometry>
-				<mesh filename="file://$(find arcdog_description)/meshes/trunk.dae" scale="1 1 1"/>
+				<mesh filename="file://$(find arcdog_description)/meshes/trunk1.dae" scale="1 1 1"/>
 			</geometry>
 			<!-- <material name="orange"/> -->
@@ -59,22 +59,4 @@
 			<geometry>
 				<box size="${trunk_length} ${trunk_width} ${trunk_height}"/>
-			</geometry>
-		</collision>
-		<collision>
-			<origin rpy="0 0 0" xyz="0 0 0"/>
-			<geometry>
-				<box size="0.1881 0.04675 0.057"/>
-			</geometry>
-		</collision>
-		<collision>
-			<origin rpy="0 0 0" xyz="0.285 0 0.01"/>
-			<geometry>
-				<cylinder length="0.05" radius="0.045"/>
-			</geometry>
-		</collision>
-		<collision>
-			<origin rpy="0 0 0" xyz="0.293 0 -0.06"/>
-			<geometry>
-				<box size="0.047 0.047 0.047"/>
 			</geometry>
 		</collision>
@@ -101,42 +83,9 @@
 		<visual>
 			<origin rpy="0 0 0" xyz="0 0 0"/>
-			<geometry>
-				<box size="0.001 0.001 0.001"/>
-			</geometry>
-			<!-- <material name="red"/> -->
+            <geometry>
+			<box size="0.015 0.015 0.004"/>
+            </geometry>
 		</visual>
-		<collision>
-			<origin rpy="0 0 0" xyz="0 0 0"/>
-			<geometry>
-				<box size=".001 .001 .001"/>
-			</geometry>
-		</collision>
-	</link>
-	<!--
-	<joint name="load_joint" type="fixed">
-			<parent link="trunk"/>
-			<child link="load_link"/>
-			<origin rpy="0 0 0" xyz="0 0 0"/>
-	</joint>
-	<link name="load_link">
-			<inertial>
-					<mass value="5"/>
-					<origin rpy="0 0 0" xyz="0 0 0"/>
-					<inertia ixx="0.01" ixy="0" ixz="0" iyy="0.01" iyz="0" izz="0.01"/>
-			</inertial>
-			<visual>
-					<origin rpy="0 0 0" xyz="0 0 0.2"/>
-					<geometry>
-							<box size="0.5 0.3 0.2"/>
-					</geometry>
-			</visual>
-			<collision>
-					<origin rpy="0 0 0" xyz="0 0 0"/>
-					<geometry>
-							<box size=".001 .001 .001"/>
-					</geometry>
-			</collision>
-	</link>
--->
+		</link>
     <xacro:leg prefix="FR" mirror="-1" mirror_dae="False" front_hind="1" front_hind_dae="True" simulator="${simulator}" robot_type="${robot_type}">
         <origin rpy="0 0 0" xyz="${leg_offset_x} ${-leg_offset_y} 0"/>
