Commit message: update arcdog_description

File: robot_description/arcdog_description/xacro/leg.xacro (robot description, xacro)
@@ -21,5 +21,5 @@
         </xacro:if>
         <xacro:if value="${simulator == 'test'}">
-            <joint name="${prefix}_HAA" type="revolute">
+            <joint name="${prefix}_hip_joint" type="revolute">
                 <xacro:insert_block name="origin"/>
                 <parent link="base"/>
@@ -52,5 +52,5 @@
                 </xacro:if>
                 <geometry>
-                    <mesh filename="package://arcdog_description/meshes/hip1.dae"
+                    <mesh filename="package://arcdog_description/meshes/hip.stl"
                           scale="1 1 1"/>
                 </geometry>
@@ -84,5 +84,5 @@
         </xacro:if>
         <xacro:if value="${simulator == 'test'}">
-            <joint name="${prefix}_HFE" type="revolute">
+            <joint name="${prefix}_thigh_joint" type="revolute">
                 <origin rpy="0 0 0" xyz="0 ${thigh_offset*mirror} 0"/>
                 <parent link="${prefix}_hip"/>
@@ -99,9 +99,9 @@
                 <geometry>
                     <xacro:if value="${mirror_dae == True}">
-                        <mesh filename="package://arcdog_description/meshes/thigh1.dae"
+                        <mesh filename="package://arcdog_description/meshes/thigh.stl"
                               scale="1 1 1"/>
                     </xacro:if>
                     <xacro:if value="${mirror_dae == False}">
-                        <mesh filename="package://arcdog_description/meshes/thigh_mirror1.dae"
+                        <mesh filename="package://arcdog_description/meshes/thigh_mirror.stl"
                               scale="1 1 1"/>
                     </xacro:if>
@@ -141,5 +141,5 @@
         </xacro:if>
         <xacro:if value="${simulator == 'test'}">
-            <joint name="${prefix}_KFE" type="revolute">
+            <joint name="${prefix}_calf_joint" type="revolute">
                 <origin rpy="0 0 0" xyz="0 0 ${-thigh_length}"/>
                 <parent link="${prefix}_thigh"/>
@@ -154,5 +154,5 @@
                 <origin rpy="0 0 0" xyz="0 0 0"/>
                 <geometry>
-                   <mesh filename="package://arcdog_description/meshes/calf1.dae"
+                    <mesh filename="package://arcdog_description/meshes/calf.stl"
                           scale="1 1 1"/>
                 </geometry>

File: robot_description/arcdog_description/xacro/real_robot.xacro (robot description, xacro)
@@ -1,153 +1,262 @@
 <?xml version="1.0"?>
-<robot name="arcdog" xmlns:xacro="http://www.ros.org/wiki/xacro">
-	<xacro:arg name="DEBUG" default="false"/>
-	<xacro:arg name="GAZEBO" default="false"/>
-	<xacro:arg name="CLASSIC" default="false"/>
-    <xacro:arg name="robot_type" default="arcdog"/>
-    <xacro:property name="robot_type" value="$(arg robot_type)"/>
-	<xacro:arg name="simulator" default="test"/>
-    <xacro:property name="simulator" value="$(arg simulator)"/>
-	<xacro:include filename="$(find arcdog_description)/xacro/const.xacro"/>
-	<xacro:include filename="$(find arcdog_description)/xacro/materials.xacro"/>
-	<xacro:include filename="$(find arcdog_description)/xacro/leg.xacro"/>
-	<xacro:if value="$(arg GAZEBO)">
-		<xacro:if value="$(arg CLASSIC)">
-			<xacro:include filename="$(find arcdog_description)/xacro/gazebo_classic.xacro"/>
-		</xacro:if>
-		<xacro:unless value="$(arg CLASSIC)">
-			<xacro:include filename="$(find arcdog_description)/xacro/gazebo.xacro"/>
-		</xacro:unless>
-	</xacro:if>
-	<xacro:unless value="$(arg GAZEBO)">
-		<xacro:include filename="$(find arcdog_description)/xacro/ros2_control_real_robot.xacro"/>
-	</xacro:unless>
-	<!-- <xacro:stairs stairs="15" xpos="0" ypos="0" zpos="0" /> -->
-	<!-- Rotor related joint and link is only for demonstrate location. -->
-	<!-- Actually, the rotor will rotate and the joint is not fixed. Reduction ratio should be considered. -->
-	<!-- Debug mode will hung up the robot, use "true" or "false" to switch it. -->
-	<xacro:if value="$(arg DEBUG)">
-		<link name="world"/>
-		<joint name="base_static_joint" type="fixed">
-			<origin rpy="0 0 0" xyz="0 0 0"/>
-			<parent link="world"/>
-			<child link="base"/>
-		</joint>
-	</xacro:if>
-	<link name="base">
-		<visual>
-			<origin rpy="0 0 0" xyz="0 0 0"/>
-			<geometry>
-				<box size="0.001 0.001 0.001"/>
-			</geometry>
-		</visual>
-	</link>
-	<joint name="floating_base" type="fixed">
-		<origin rpy="0 0 0" xyz="0 0 0"/>
-		<parent link="base"/>
-		<child link="trunk"/>
-	</joint>
-	<link name="trunk">
-		<visual>
-			<origin rpy="0 0 0" xyz="0 0 0"/>
-			<geometry>
-				<mesh filename="file://$(find arcdog_description)/meshes/trunk.dae" scale="1 1 1"/>
-			</geometry>
-			<!-- <material name="orange"/> -->
-		</visual>
-		<collision>
-			<origin rpy="0 0 0" xyz="0 0 0"/>
-			<geometry>
-				<box size="${trunk_length} ${trunk_width} ${trunk_height}"/>
-			</geometry>
-		</collision>
-		<collision>
-			<origin rpy="0 0 0" xyz="0 0 0"/>
-			<geometry>
-				<box size="0.1881 0.04675 0.057"/>
-			</geometry>
-		</collision>
-		<collision>
-			<origin rpy="0 0 0" xyz="0.285 0 0.01"/>
-			<geometry>
-				<cylinder length="0.05" radius="0.045"/>
-			</geometry>
-		</collision>
-		<collision>
-			<origin rpy="0 0 0" xyz="0.293 0 -0.06"/>
-			<geometry>
-				<box size="0.047 0.047 0.047"/>
-			</geometry>
-		</collision>
-		<inertial>
-			<origin rpy="0 0 0" xyz="${trunk_com_x} ${trunk_com_y} ${trunk_com_z}"/>
-			<mass value="${trunk_mass}"/>
-			<inertia
-							ixx="${trunk_ixx}" ixy="${trunk_ixy}" ixz="${trunk_ixz}"
-							iyy="${trunk_iyy}" iyz="${trunk_iyz}"
-							izz="${trunk_izz}"/>
-		</inertial>
-	</link>
-	<joint name="imu_joint" type="fixed">
-		<parent link="trunk"/>
-		<child link="imu_link"/>
-		<origin rpy="0 0 0" xyz="0 0 0"/>
-	</joint>
-	<link name="imu_link">
-		<inertial>
-			<mass value="0.001"/>
-			<origin rpy="0 0 0" xyz="0 0 0"/>
-			<inertia ixx="0.0001" ixy="0" ixz="0" iyy="0.0001" iyz="0" izz="0.0001"/>
-		</inertial>
-		<visual>
-			<origin rpy="0 0 0" xyz="0 0 0"/>
-			<geometry>
-				<box size="0.001 0.001 0.001"/>
-			</geometry>
-			<!-- <material name="red"/> -->
-		</visual>
-		<collision>
-			<origin rpy="0 0 0" xyz="0 0 0"/>
-			<geometry>
-				<box size=".001 .001 .001"/>
-			</geometry>
-		</collision>
-	</link>
-	<!--
-	<joint name="load_joint" type="fixed">
-			<parent link="trunk"/>
-			<child link="load_link"/>
-			<origin rpy="0 0 0" xyz="0 0 0"/>
-	</joint>
-	<link name="load_link">
-			<inertial>
-					<mass value="5"/>
-					<origin rpy="0 0 0" xyz="0 0 0"/>
-					<inertia ixx="0.01" ixy="0" ixz="0" iyy="0.01" iyz="0" izz="0.01"/>
-			</inertial>
-			<visual>
-					<origin rpy="0 0 0" xyz="0 0 0.2"/>
-					<geometry>
-							<box size="0.5 0.3 0.2"/>
-					</geometry>
-			</visual>
-			<collision>
-					<origin rpy="0 0 0" xyz="0 0 0"/>
-					<geometry>
-							<box size=".001 .001 .001"/>
-					</geometry>
-			</collision>
-	</link>
--->
-    <xacro:leg prefix="FR" mirror="-1" mirror_dae="False" front_hind="1" front_hind_dae="True" simulator="${simulator}" robot_type="${robot_type}">
-        <origin rpy="0 0 0" xyz="${leg_offset_x} ${-leg_offset_y} 0"/>
-    </xacro:leg>
-    <xacro:leg prefix="FL" mirror="1" mirror_dae="True" front_hind="1" front_hind_dae="True" simulator="${simulator}" robot_type="${robot_type}">
-        <origin rpy="0 0 0" xyz="${leg_offset_x} ${leg_offset_y} 0"/>
-    </xacro:leg>
-    <xacro:leg prefix="RR" mirror="-1" mirror_dae="False" front_hind="-1" front_hind_dae="False" simulator="${simulator}" robot_type="${robot_type}">
-        <origin rpy="0 0 0" xyz="${-leg_offset_x} ${-leg_offset_y} 0"/>
-    </xacro:leg>
-    <xacro:leg prefix="RL" mirror="1" mirror_dae="True" front_hind="-1" front_hind_dae="False" simulator="${simulator}" robot_type="${robot_type}">
-        <origin rpy="0 0 0" xyz="${-leg_offset_x} ${leg_offset_y} 0"/>
-    </xacro:leg>
+<robot xmlns:xacro="http://www.ros.org/wiki/xacro">
+    <xacro:include filename="$(find arcdog_description)/xacro/transmission.xacro"/>
+    <xacro:macro name="leg" params="prefix mirror mirror_dae front_hind front_hind_dae simulator robot_type *origin">
+        <xacro:if value="${simulator == 'ocs2'}">
+            <joint name="${prefix}_HAA" type="revolute">
+                <xacro:insert_block name="origin"/>
+                <parent link="trunk"/>
+                <child link="${prefix}_hip"/>
+                <axis xyz="1 0 0"/>
+                <dynamics damping="${damping}" friction="${friction}"/>
+                <xacro:if value="${(mirror_dae == True)}">
+                    <limit effort="${hip_torque_max}" velocity="${hip_velocity_max}" lower="${hip_min}"
+                        upper="${hip_max}"/>
+                </xacro:if>
+                <xacro:if value="${(mirror_dae == False)}">
+                    <limit effort="${hip_torque_max}" velocity="${hip_velocity_max}" lower="${-hip_max}"
+                        upper="${-hip_min}"/>
+                </xacro:if>
+            </joint>
+        </xacro:if>
+        <xacro:if value="${simulator == 'test'}">
+            <joint name="${prefix}_hip_joint" type="revolute">
+                <xacro:insert_block name="origin"/>
+                <parent link="base"/>
+                <child link="${prefix}_hip"/>
+                <axis xyz="1 0 0"/>
+                <dynamics damping="${damping}" friction="${friction}"/>
+                <xacro:if value="${(mirror_dae == True)}">
+                    <limit effort="${hip_torque_max}" velocity="${hip_velocity_max}" lower="${hip_min}"
+                        upper="${hip_max}"/>
+                </xacro:if>
+                <xacro:if value="${(mirror_dae == False)}">
+                    <limit effort="${hip_torque_max}" velocity="${hip_velocity_max}" lower="${-hip_max}"
+                        upper="${-hip_min}"/>
+                </xacro:if>
+            </joint>
+        </xacro:if>
+        <link name="${prefix}_hip">
+            <visual>
+                <xacro:if value="${(mirror_dae == True) and (front_hind_dae == True)}">
+                    <origin rpy="0 0 0" xyz="0 0 0"/>
+                </xacro:if>
+                <xacro:if value="${(mirror_dae == False) and (front_hind_dae == True)}">
+                    <origin rpy="${pi} 0 0" xyz="0 0 0"/>
+                </xacro:if>
+                <xacro:if value="${(mirror_dae == True) and (front_hind_dae == False)}">
+                    <origin rpy="0 ${pi} 0" xyz="0 0 0"/>
+                </xacro:if>
+                <xacro:if value="${(mirror_dae == False) and (front_hind_dae == False)}">
+                    <origin rpy="${pi} ${pi} 0" xyz="0 0 0"/>
+                </xacro:if>
+                <geometry>
+                    <mesh filename="package://arcdog_description/meshes/hip.stl"
+                          scale="1 1 1"/>
+                </geometry>
+                <material name="orange"/>
+            </visual>
+            <collision>
+                <origin rpy="${pi/2.0} 0 0" xyz="0 0 0"/>
+                <geometry>
+                    <cylinder length="${hip_length}" radius="${hip_radius}"/>
+                </geometry>
+            </collision>
+            <inertial>
+                <origin rpy="0 0 0" xyz="${hip_com_x*front_hind} ${hip_com_y*mirror} ${hip_com_z}"/>
+                <mass value="${hip_mass}"/>
+                <inertia
+                        ixx="${hip_ixx}" ixy="${hip_ixy*mirror*front_hind}" ixz="${hip_ixz*front_hind}"
+                        iyy="${hip_iyy}" iyz="${hip_iyz*mirror}"
+                        izz="${hip_izz}"/>
+            </inertial>
+        </link>
+        <xacro:if value="${simulator == 'ocs2'}">
+            <joint name="${prefix}_HFE" type="revolute">
+                <origin rpy="0 0 0" xyz="0 ${thigh_offset*mirror} 0"/>
+                <parent link="${prefix}_hip"/>
+                <child link="${prefix}_thigh"/>
+                <axis xyz="0 1 0"/>
+                <dynamics damping="${damping}" friction="${friction}"/>
+                <limit effort="${thigh_torque_max}" velocity="${thigh_velocity_max}" lower="${thigh_min}"
+                    upper="${thigh_max}"/>
+            </joint>
+        </xacro:if>
+        <xacro:if value="${simulator == 'test'}">
+            <joint name="${prefix}_thigh_joint" type="revolute">
+                <origin rpy="0 0 0" xyz="0 ${thigh_offset*mirror} 0"/>
+                <parent link="${prefix}_hip"/>
+                <child link="${prefix}_thigh"/>
+                <axis xyz="0 1 0"/>
+                <dynamics damping="${damping}" friction="${friction}"/>
+                <limit effort="${thigh_torque_max}" velocity="${thigh_velocity_max}" lower="${thigh_min}"
+                    upper="${thigh_max}"/>
+            </joint>
+        </xacro:if>
+        <link name="${prefix}_thigh">
+            <visual>
+                <origin rpy="0 0 0" xyz="0 0 0"/>
+                <geometry>
+                    <xacro:if value="${mirror_dae == True}">
+                        <mesh filename="package://arcdog_description/meshes/thigh.stl"
+                              scale="1 1 1"/>
+                    </xacro:if>
+                    <xacro:if value="${mirror_dae == False}">
+                        <mesh filename="package://arcdog_description/meshes/thigh_mirror.stl"
+                              scale="1 1 1"/>
+                    </xacro:if>
+                </geometry>
+                <material name="orange"/>
+            </visual>
+            <collision>
+                <origin rpy="0 ${pi/2.0} 0" xyz="${thigh_x_offset} 0 ${-thigh_length/2.0}"/>
+                <geometry>
+                    <box size="${thigh_length} ${thigh_width} ${thigh_height}"/>
+                </geometry>
+            </collision>
+            <collision>
+                <origin rpy="${pi/2.0} 0 0" xyz="0 ${mirror*thigh_shoulder_y_offset} 0"/>
+                <geometry>
+                    <cylinder length="${thigh_shoulder_length}" radius="${thigh_shoulder_radius}"/>
+                </geometry>
+            </collision>
+            <inertial>
+                <origin rpy="0 0 0" xyz="${thigh_com_x} ${thigh_com_y*mirror} ${thigh_com_z}"/>
+                <mass value="${thigh_mass}"/>
+                <inertia
+                        ixx="${thigh_ixx}" ixy="${thigh_ixy*mirror}" ixz="${thigh_ixz}"
+                        iyy="${thigh_iyy}" iyz="${thigh_iyz*mirror}"
+                        izz="${thigh_izz}"/>
+            </inertial>
+        </link>
+        <xacro:if value="${simulator == 'ocs2'}">
+            <joint name="${prefix}_KFE" type="revolute">
+                <origin rpy="0 0 0" xyz="0 0 ${-thigh_length}"/>
+                <parent link="${prefix}_thigh"/>
+                <child link="${prefix}_calf"/>
+                <axis xyz="0 1 0"/>
+                <dynamics damping="${damping}" friction="${friction}"/>
+                <limit effort="${calf_torque_max}" velocity="${calf_velocity_max}" lower="${calf_min}" upper="${calf_max}"/>
+            </joint>
+        </xacro:if>
+        <xacro:if value="${simulator == 'test'}">
+            <joint name="${prefix}_calf_joint" type="revolute">
+                <origin rpy="0 0 0" xyz="0 0 ${-thigh_length}"/>
+                <parent link="${prefix}_thigh"/>
+                <child link="${prefix}_calf"/>
+                <axis xyz="0 1 0"/>
+                <dynamics damping="${damping}" friction="${friction}"/>
+                <limit effort="${calf_torque_max}" velocity="${calf_velocity_max}" lower="${calf_min}" upper="${calf_max}"/>
+            </joint>
+        </xacro:if>
+        <link name="${prefix}_calf">
+            <visual>
+                <origin rpy="0 0 0" xyz="0 0 0"/>
+                <geometry>
+                    <mesh filename="package://arcdog_description/meshes/calf.stl"
+                          scale="1 1 1"/>
+                </geometry>
+                <material name="orange"/>
+            </visual>
+            <collision>
+                <origin rpy="0 ${pi/2.0} 0" xyz="${calf_x_offset} 0 ${-calf_length/2.0}"/>
+                <geometry>
+                    <box size="${calf_length} ${calf_width} ${calf_height}"/>
+                </geometry>
+            </collision>
+            <inertial>
+                <origin rpy="0 0 0" xyz="${calf_com_x} ${calf_com_y} ${calf_com_z}"/>
+                <mass value="${calf_mass}"/>
+                <inertia
+                        ixx="${calf_ixx}" ixy="${calf_ixy}" ixz="${calf_ixz}"
+                        iyy="${calf_iyy}" iyz="${calf_iyz}"
+                        izz="${calf_izz}"/>
+            </inertial>
+        </link>
+        <joint name="${prefix}_foot_fixed" type="fixed" dont_collapse="true">
+            <origin rpy="0 0 0" xyz="0 0 ${-calf_length}"/>
+            <parent link="${prefix}_calf"/>
+            <child link="${prefix}_foot"/>
+        </joint>
+        <link name="${prefix}_foot">
+            <visual>
+                <origin rpy="0 0 0" xyz="0 0 0"/>
+                <geometry>
+                    <sphere radius="${foot_radius-0.01}"/>
+                </geometry>
+                <material name="orange"/>
+            </visual>
+            <collision>
+                <origin rpy="0 0 0" xyz="0 0 0"/>
+                <geometry>
+                    <sphere radius="${foot_radius}"/>
+                </geometry>
+                <surface>
+                <bounce>
+                    <restitution_coefficient>0</restitution_coefficient>
+                    <threshold>1e+06</threshold>
+                </bounce>
+                <friction>
+                    <ode>
+                    <mu>1.0</mu>
+                    <mu2>1.0</mu2>
+                    </ode>
+                    <bullet>
+                    <rolling_friction>0.3</rolling_friction>
+                    <friction2>50</friction2>
+                    </bullet>
+                </friction>
+                <contact>
+                    <ode>
+                    <kp>30000.0</kp>
+                    <kd>1000.0</kd>
+                    </ode>
+                    <bullet>
+                    <kp>30000.0</kp>
+                    <kd>1000.0</kd>
+                    <split_impulse>1</split_impulse>
+                    <split_impulse_penetration_threshold>-0.01</split_impulse_penetration_threshold>
+                    </bullet>
+                </contact>
+                </surface>
+            </collision>
+            <inertial>
+                <mass value="${foot_mass}"/>
+                <inertia
+                        ixx="${(2*foot_mass)/5.0*(foot_radius*foot_radius)}" ixy="0.0" ixz="0.0"
+                        iyy="${(2*foot_mass)/5.0*(foot_radius*foot_radius)}" iyz="0.0"
+                        izz="${(2*foot_mass)/5.0*(foot_radius*foot_radius)}"/>
+            </inertial>
+        </link>
+        <gazebo reference="${prefix}_foot_fixed">
+            <disableFixedJointLumping>true</disableFixedJointLumping>
+        </gazebo>
+        <gazebo reference="${prefix}_hip">
+            <mu1>0.2</mu1>
+            <mu2>0.2</mu2>
+            <material>Gazebo/DarkGrey</material>
+        </gazebo>
+        <gazebo reference="${prefix}_thigh">
+            <mu1>0.2</mu1>
+            <mu2>0.2</mu2>
+            <self_collide>0</self_collide>
+            <material>Gazebo/DarkGrey</material>
+            <kp value="1000000.0"/>
+            <kd value="100.0"/>
+        </gazebo>
+        <gazebo reference="${prefix}_calf">
+            <mu1>0.6</mu1>
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
File: robot_description/arcdog_description/xacro/robot.xacro (robot description, xacro)
@@ -51,5 +51,5 @@
 			<origin rpy="0 0 0" xyz="0 0 0"/>
 			<geometry>
-				<mesh filename="file://$(find arcdog_description)/meshes/trunk.dae" scale="1 1 1"/>
+				<mesh filename="file://$(find arcdog_description)/meshes/trunk1.dae" scale="1 1 1"/>
 			</geometry>
 			<!-- <material name="orange"/> -->
@@ -59,22 +59,4 @@
 			<geometry>
 				<box size="${trunk_length} ${trunk_width} ${trunk_height}"/>
-			</geometry>
-		</collision>
-		<collision>
-			<origin rpy="0 0 0" xyz="0 0 0"/>
-			<geometry>
-				<box size="0.1881 0.04675 0.057"/>
-			</geometry>
-		</collision>
-		<collision>
-			<origin rpy="0 0 0" xyz="0.285 0 0.01"/>
-			<geometry>
-				<cylinder length="0.05" radius="0.045"/>
-			</geometry>
-		</collision>
-		<collision>
-			<origin rpy="0 0 0" xyz="0.293 0 -0.06"/>
-			<geometry>
-				<box size="0.047 0.047 0.047"/>
 			</geometry>
 		</collision>
@@ -97,46 +79,13 @@
 			<mass value="0.001"/>
 			<origin rpy="0 0 0" xyz="0 0 0"/>
-			<inertia ixx="0.0001" ixy="0" ixz="0" iyy="0.0001" iyz="0" izz="0.0001"/>
+			<inertia ixx="0.000001" ixy="0" ixz="0" iyy="0.000001" iyz="0" izz="0.000001"/>
 		</inertial>
 		<visual>
 			<origin rpy="0 0 0" xyz="0 0 0"/>
-			<geometry>
-				<box size="0.001 0.001 0.001"/>
-			</geometry>
-			<!-- <material name="red"/> -->
+            <geometry>
+			<box size="0.015 0.015 0.004"/>
+            </geometry>
 		</visual>
-		<collision>
-			<origin rpy="0 0 0" xyz="0 0 0"/>
-			<geometry>
-				<box size=".001 .001 .001"/>
-			</geometry>
-		</collision>
-	</link>
-	<!--
-	<joint name="load_joint" type="fixed">
-			<parent link="trunk"/>
-			<child link="load_link"/>
-			<origin rpy="0 0 0" xyz="0 0 0"/>
-	</joint>
-	<link name="load_link">
-			<inertial>
-					<mass value="5"/>
-					<origin rpy="0 0 0" xyz="0 0 0"/>
-					<inertia ixx="0.01" ixy="0" ixz="0" iyy="0.01" iyz="0" izz="0.01"/>
-			</inertial>
-			<visual>
-					<origin rpy="0 0 0" xyz="0 0 0.2"/>
-					<geometry>
-							<box size="0.5 0.3 0.2"/>
-					</geometry>
-			</visual>
-			<collision>
-					<origin rpy="0 0 0" xyz="0 0 0"/>
-					<geometry>
-							<box size=".001 .001 .001"/>
-					</geometry>
-			</collision>
-	</link>
--->
+		</link>
     <xacro:leg prefix="FR" mirror="-1" mirror_dae="False" front_hind="1" front_hind_dae="True" simulator="${simulator}" robot_type="${robot_type}">
         <origin rpy="0 0 0" xyz="${leg_offset_x} ${-leg_offset_y} 0"/>
