Commit message: modify robot.xacro

File: robot_description/arcdog_description/xacro/robot.xacro (robot description, xacro)
@@ -79,5 +79,5 @@
 			<mass value="0.001"/>
 			<origin rpy="0 0 0" xyz="0 0 0"/>
-			<inertia ixx="0.0001" ixy="0" ixz="0" iyy="0.0001" iyz="0" izz="0.0001"/>
+			<inertia ixx="0.000001" ixy="0" ixz="0" iyy="0.000001" iyz="0" izz="0.000001"/>
 		</inertial>
 		<visual>

Commit message: update xacro model (half way)

File: robot_description/arcdog_description/xacro/robot.xacro (robot description, xacro)
@@ -4,8 +4,4 @@
 	<xacro:arg name="GAZEBO" default="false"/>
 	<xacro:arg name="CLASSIC" default="false"/>
-    <xacro:arg name="robot_type" default="arcdog"/>
-    <xacro:property name="robot_type" value="$(arg robot_type)"/>
-	<xacro:arg name="simulator" default="test"/>
-    <xacro:property name="simulator" value="$(arg simulator)"/>
 	<xacro:include filename="$(find arcdog_description)/xacro/const.xacro"/>
 	<xacro:include filename="$(find arcdog_description)/xacro/materials.xacro"/>

File: robot_description/go2_description/xacro/leg.xacro (robot description, xacro)
@@ -129,5 +129,5 @@
 			</inertial>
 		</link>
-		<joint name="${name}_foot_fixed" type="fixed">0
+		<joint name="${name}_foot_fixed" type="fixed">
 			<origin rpy="0 0 0" xyz="0 0 ${-(calf_length)}"/>
 			<parent link="${name}_calf"/>
@@ -155,27 +155,4 @@
 			</inertial>
 		</link>
-		<gazebo reference="${name}_hip">
-			<mu1>0.2</mu1>
-			<mu2>0.2</mu2>
-		</gazebo>
-		<gazebo reference="${name}_thigh">
-			<mu1>0.2</mu1>
-			<mu2>0.2</mu2>
-			<self_collide>0</self_collide>
-			<kp value="1000000.0"/>
-			<kd value="100.0"/>
-		</gazebo>
-		<gazebo reference="${name}_calf">
-			<mu1>0.6</mu1>
-			<mu2>0.6</mu2>
-			<self_collide>1</self_collide>
-		</gazebo>
-		<gazebo reference="${name}_foot">
-			<mu1>0.6</mu1>
-			<mu2>0.6</mu2>
-			<self_collide>1</self_collide>
-			<kp value="1000000.0"/>
-			<kd value="100.0"/>
-		</gazebo>
 		<xacro:leg_transmission name="${name}"/>
 	</xacro:macro>

File: robot_description/go2_description/xacro/robot.xacro (robot description, xacro)
@@ -55,22 +55,4 @@
 			<geometry>
 				<box size="${trunk_length} ${trunk_width} ${trunk_height}"/>
-			</geometry>
-		</collision>
-		<collision>
-			<origin rpy="0 0 0" xyz="0 0 0"/>
-			<geometry>
-				<box size="0.1881 0.04675 0.057"/>
-			</geometry>
-		</collision>
-		<collision>
-			<origin rpy="0 0 0" xyz="0.285 0 0.01"/>
-			<geometry>
-				<cylinder length="0.05" radius="0.045"/>
-			</geometry>
-		</collision>
-		<collision>
-			<origin rpy="0 0 0" xyz="0.293 0 -0.06"/>
-			<geometry>
-				<box size="0.047 0.047 0.047"/>
 			</geometry>
 		</collision>
