Commit message: update arcdog xacro model

File: robot_description/arcdog_description/xacro/const.xacro (robot description, xacro)
@@ -2,4 +2,5 @@
 <robot xmlns:xacro="http://www.ros.org/wiki/xacro" name="arcdog_description">
     <!-- Constants for robot dimensions -->
+    <xacro:property name="PI" value="3.1415926535897931"/>
     <xacro:property name="stick_mass" value="0.00001"/>
     <!-- simplified collision value -->
@@ -11,12 +12,11 @@
     <xacro:property name="thigh_shoulder_radius" value="0.0495"/>
     <xacro:property name="thigh_shoulder_length" value="0.03826"/>
-    <xacro:property name="thigh_shoulder_y_offset" value="0.0"/>
-    <xacro:property name="thigh_width" value="0.040"/> //little larger than real value
+    <xacro:property name="thigh_width" value="?"/> //little larger than real value
     <xacro:property name="thigh_height" value="0.06797"/>
-    <xacro:property name="thigh_x_offset" value="0.000"/>
     <xacro:property name="calf_width" value="0.02"/>
     <xacro:property name="calf_height" value="0.05"/>
-    <xacro:property name="calf_x_offset" value="0.000"/>
     <xacro:property name="foot_radius" value="0.0265"/>
+    <!-- <xacro:property name="stick_radius" value="?"/>
+	<xacro:property name="stick_length" value="?"/> -->
     <!-- kinematic value -->
     <xacro:property name="thigh_offset" value="0.11475"/>
@@ -26,19 +26,29 @@
     <xacro:property name="leg_offset_x" value="0.2515"/>
     <xacro:property name="leg_offset_y" value="0.0605"/>
-    <xacro:property name="trunk_offset_z" value="0.01675"/> //TODO
-    <xacro:property name="hip_offset" value="0.0001"/> //TODO
+    <!-- <xacro:property name="trunk_offset_z" value="0.01675"/> //TODO -->
+    <xacro:property name="hip_offset" value="0.11475"/> //go2 special point, puting hip collision model at thigh position
+    <!-- offset of link locations (left front) -->
+    <!-- <xacro:property name="hip_offset_x" value="?"/>
+	<xacro:property name="hip_offset_y" value="?"/>
+	<xacro:property name="hip_offset_z" value="?"/>
+	<xacro:property name="thigh_offset_x" value="?"/>
+	<xacro:property name="thigh_offset_y" value="?"/>
+	<xacro:property name="thigh_offset_z" value="?"/>
+	<xacro:property name="calf_offset_x" value="?"/>
+	<xacro:property name="calf_offset_y" value="?"/>
+	<xacro:property name="calf_offset_z" value="?"/> -->
     <!-- joint limits -->
     <xacro:property name="damping" value="0.05"/>
     <xacro:property name="friction" value="0.01"/>
-    <xacro:property name="hip_max" value="${70*pi/180.0}"/>
-    <xacro:property name="hip_min" value="${-70*pi/180.0}"/>
+    <xacro:property name="hip_position_max" value="${70*pi/180.0}"/>
+    <xacro:property name="hip_position_min" value="${-70*pi/180.0}"/>
     <xacro:property name="hip_velocity_max" value="20"/>
     <xacro:property name="hip_torque_max" value="35.278"/>
-    <xacro:property name="thigh_max" value="3.4907"/>
-    <xacro:property name="thigh_min" value="-1.5708"/>
+    <xacro:property name="thigh_position_max" value="3.4907"/>
+    <xacro:property name="thigh_position_min" value="-1.5708"/>
     <xacro:property name="thigh_velocity_max" value="20"/>
     <xacro:property name="thigh_torque_max" value="35.278"/>
-    <xacro:property name="calf_max" value="${-37*pi/180.0}"/>
-    <xacro:property name="calf_min" value="${-159*pi/180.0}"/>
+    <xacro:property name="calf_position_max" value="${-37*pi/180.0}"/>
+    <xacro:property name="calf_position_min" value="${-159*pi/180.0}"/>
     <xacro:property name="calf_velocity_max" value="15.89"/>
     <xacro:property name="calf_torque_max" value="44.4"/>

File: robot_description/arcdog_description/xacro/leg.xacro (robot description, xacro)
@@ -2,61 +2,51 @@
 <robot xmlns:xacro="http://www.ros.org/wiki/xacro">
     <xacro:include filename="$(find arcdog_description)/xacro/transmission.xacro"/>
-    <xacro:macro name="leg" params="prefix mirror mirror_dae front_hind front_hind_dae simulator robot_type *origin">
-        <xacro:if value="${simulator == 'ocs2'}">
-            <joint name="${prefix}_HAA" type="revolute">
-                <xacro:insert_block name="origin"/>
-                <parent link="trunk"/>
-                <child link="${prefix}_hip"/>
+    <xacro:macro name="leg" params="name mirror mirror_dae front_hind front_hind_dae">
+		<joint name="${name}_hip_joint" type="revolute">
+			<xacro:if value="${(mirror_dae == False) and (front_hind_dae == True)}">
+				<origin rpy="0 0 0" xyz="${leg_offset_x} ${-leg_offset_y} 0"/>
+			</xacro:if>
+			<xacro:if value="${(mirror_dae == True) and (front_hind_dae == True)}">
+				<origin rpy="0 0 0" xyz="${leg_offset_x} ${leg_offset_y} 0"/>
+			</xacro:if>
+			<xacro:if value="${(mirror_dae == False) and (front_hind_dae == False)}">
+				<origin rpy="0 0 0" xyz="${-leg_offset_x} ${-leg_offset_y} 0"/>
+			</xacro:if>
+			<xacro:if value="${(mirror_dae == True) and (front_hind_dae == False)}">
+				<origin rpy="0 0 0" xyz="${-leg_offset_x} ${leg_offset_y} 0"/>
+			</xacro:if>
+			<parent link="trunk"/>
+			<child link="${name}_hip"/>
                 <axis xyz="1 0 0"/>
                 <dynamics damping="${damping}" friction="${friction}"/>
-                <xacro:if value="${(mirror_dae == True)}">
-                    <limit effort="${hip_torque_max}" velocity="${hip_velocity_max}" lower="${hip_min}"
-                        upper="${hip_max}"/>
-                </xacro:if>
-                <xacro:if value="${(mirror_dae == False)}">
-                    <limit effort="${hip_torque_max}" velocity="${hip_velocity_max}" lower="${-hip_max}"
-                        upper="${-hip_min}"/>
+			<xacro:if value="${(mirror_dae == True)}">
+				<limit effort="${hip_torque_max}" velocity="${hip_velocity_max}" lower="${hip_position_min}"
+							 upper="${hip_position_max}"/>
+			</xacro:if>
+			<xacro:if value="${(mirror_dae == False)}">
+				<limit effort="${hip_torque_max}" velocity="${hip_velocity_max}" lower="${-hip_position_max}"
+							 upper="${-hip_position_min}"/>
                 </xacro:if>
             </joint>
-        </xacro:if>
-        <xacro:if value="${simulator == 'test'}">
-            <joint name="${prefix}_hip_joint" type="revolute">
-                <xacro:insert_block name="origin"/>
-                <parent link="base"/>
-                <child link="${prefix}_hip"/>
-                <axis xyz="1 0 0"/>
-                <dynamics damping="${damping}" friction="${friction}"/>
-                <xacro:if value="${(mirror_dae == True)}">
-                    <limit effort="${hip_torque_max}" velocity="${hip_velocity_max}" lower="${hip_min}"
-                        upper="${hip_max}"/>
-                </xacro:if>
-                <xacro:if value="${(mirror_dae == False)}">
-                    <limit effort="${hip_torque_max}" velocity="${hip_velocity_max}" lower="${-hip_max}"
-                        upper="${-hip_min}"/>
-                </xacro:if>
-            </joint>
-        </xacro:if>
-        <link name="${prefix}_hip">
-            <visual>
-                <xacro:if value="${(mirror_dae == True) and (front_hind_dae == True)}">
-                    <origin rpy="0 0 0" xyz="0 0 0"/>
-                </xacro:if>
-                <xacro:if value="${(mirror_dae == False) and (front_hind_dae == True)}">
-                    <origin rpy="${pi} 0 0" xyz="0 0 0"/>
-                </xacro:if>
-                <xacro:if value="${(mirror_dae == True) and (front_hind_dae == False)}">
-                    <origin rpy="0 ${pi} 0" xyz="0 0 0"/>
-                </xacro:if>
-                <xacro:if value="${(mirror_dae == False) and (front_hind_dae == False)}">
-                    <origin rpy="${pi} ${pi} 0" xyz="0 0 0"/>
-                </xacro:if>
+		<link name="${name}_hip">
+			<visual>
+				<xacro:if value="${(mirror_dae == True) and (front_hind_dae == True)}">
+					<origin rpy="0 0 0" xyz="0 0 0"/>
+				</xacro:if>
+				<xacro:if value="${(mirror_dae == False) and (front_hind_dae == True)}">
+					<origin rpy="${PI} 0 0" xyz="0 0 0"/>
+				</xacro:if>
+				<xacro:if value="${(mirror_dae == True) and (front_hind_dae == False)}">
+					<origin rpy="0 ${PI} 0" xyz="0 0 0"/>
+				</xacro:if>
+				<xacro:if value="${(mirror_dae == False) and (front_hind_dae == False)}">
+					<origin rpy="${PI} ${PI} 0" xyz="0 0 0"/>
+				</xacro:if>
                 <geometry>
-                    <mesh filename="package://arcdog_description/meshes/hip.stl"
-                          scale="1 1 1"/>
+                    <mesh filename="package://arcdog_description/meshes/hip.stl" scale="1 1 1"/>
                 </geometry>
-                <material name="orange"/>
             </visual>
             <collision>
-                <origin rpy="${pi/2.0} 0 0" xyz="0 0 0"/>
+                <origin rpy="${PI/2.0} 0 0" xyz="0 ${hip_offset*mirror} 0"/>
                 <geometry>
                     <cylinder length="${hip_length}" radius="${hip_radius}"/>
@@ -72,51 +62,29 @@
             </inertial>
         </link>
-        <xacro:if value="${simulator == 'ocs2'}">
-            <joint name="${prefix}_HFE" type="revolute">
-                <origin rpy="0 0 0" xyz="0 ${thigh_offset*mirror} 0"/>
-                <parent link="${prefix}_hip"/>
-                <child link="${prefix}_thigh"/>
-                <axis xyz="0 1 0"/>
-                <dynamics damping="${damping}" friction="${friction}"/>
-                <limit effort="${thigh_torque_max}" velocity="${thigh_velocity_max}" lower="${thigh_min}"
-                    upper="${thigh_max}"/>
-            </joint>
-        </xacro:if>
-        <xacro:if value="${simulator == 'test'}">
-            <joint name="${prefix}_thigh_joint" type="revolute">
-                <origin rpy="0 0 0" xyz="0 ${thigh_offset*mirror} 0"/>
-                <parent link="${prefix}_hip"/>
-                <child link="${prefix}_thigh"/>
-                <axis xyz="0 1 0"/>
-                <dynamics damping="${damping}" friction="${friction}"/>
-                <limit effort="${thigh_torque_max}" velocity="${thigh_velocity_max}" lower="${thigh_min}"
-                    upper="${thigh_max}"/>
-            </joint>
-        </xacro:if>
-        <link name="${prefix}_thigh">
+		<joint name="${name}_thigh_joint" type="revolute">
+			<origin rpy="0 0 0" xyz="0 ${thigh_offset*mirror} 0"/>
+			<parent link="${name}_hip"/>
+			<child link="${name}_thigh"/>
+			<axis xyz="0 1 0"/>
+			<dynamics damping="${damping}" friction="${friction}"/>
+			<limit effort="${thigh_torque_max}" velocity="${thigh_velocity_max}" lower="${thigh_position_min}"
+						 upper="${thigh_position_max}"/>
+		</joint>
+        <link name="${name}_thigh">
             <visual>
                 <origin rpy="0 0 0" xyz="0 0 0"/>
                 <geometry>
                     <xacro:if value="${mirror_dae == True}">
-                        <mesh filename="package://arcdog_description/meshes/thigh.stl"
-                              scale="1 1 1"/>
+                        <mesh filename="package://arcdog_description/meshes/thigh.stl" scale="1 1 1"/>
                     </xacro:if>
                     <xacro:if value="${mirror_dae == False}">
-                        <mesh filename="package://arcdog_description/meshes/thigh_mirror.stl"
-                              scale="1 1 1"/>
+                        <mesh filename="package://arcdog_description/meshes/thigh_mirror.stl" scale="1 1 1"/>
                     </xacro:if>
                 </geometry>
-                <material name="orange"/>
             </visual>
             <collision>
-                <origin rpy="0 ${pi/2.0} 0" xyz="${thigh_x_offset} 0 ${-thigh_length/2.0}"/>
+                <origin rpy="0 ${PI/2.0} 0" xyz="0 0 ${-thigh_length/2.0}"/>
                 <geometry>
                     <box size="${thigh_length} ${thigh_width} ${thigh_height}"/>
-                </geometry>
-            </collision>
-            <collision>
-                <origin rpy="${pi/2.0} 0 0" xyz="0 ${mirror*thigh_shoulder_y_offset} 0"/>
-                <geometry>
-                    <cylinder length="${thigh_shoulder_length}" radius="${thigh_shoulder_radius}"/>
                 </geometry>
             </collision>
@@ -130,35 +98,22 @@
             </inertial>
         </link>
-        <xacro:if value="${simulator == 'ocs2'}">
-            <joint name="${prefix}_KFE" type="revolute">
-                <origin rpy="0 0 0" xyz="0 0 ${-thigh_length}"/>
-                <parent link="${prefix}_thigh"/>
-                <child link="${prefix}_calf"/>
-                <axis xyz="0 1 0"/>
-                <dynamics damping="${damping}" friction="${friction}"/>
-                <limit effort="${calf_torque_max}" velocity="${calf_velocity_max}" lower="${calf_min}" upper="${calf_max}"/>
-            </joint>
-        </xacro:if>
-        <xacro:if value="${simulator == 'test'}">
-            <joint name="${prefix}_calf_joint" type="revolute">
-                <origin rpy="0 0 0" xyz="0 0 ${-thigh_length}"/>
-                <parent link="${prefix}_thigh"/>
-                <child link="${prefix}_calf"/>
-                <axis xyz="0 1 0"/>
-                <dynamics damping="${damping}" friction="${friction}"/>
-                <limit effort="${calf_torque_max}" velocity="${calf_velocity_max}" lower="${calf_min}" upper="${calf_max}"/>
-            </joint>
-        </xacro:if>
-        <link name="${prefix}_calf">
+		<joint name="${name}_calf_joint" type="revolute">
+			<origin rpy="0 0 0" xyz="0 0 ${-thigh_length}"/>
+			<parent link="${name}_thigh"/>
+			<child link="${name}_calf"/>
+			<axis xyz="0 1 0"/>
+			<dynamics damping="${damping}" friction="${friction}"/>
+			<limit effort="${calf_torque_max}" velocity="${calf_velocity_max}" lower="${calf_position_min}"
+						 upper="${calf_position_max}"/>
+		</joint>
+        <link name="${name}_calf">
             <visual>
                 <origin rpy="0 0 0" xyz="0 0 0"/>
                 <geometry>
-                    <mesh filename="package://arcdog_description/meshes/calf.stl"
-                          scale="1 1 1"/>
+                    <mesh filename="package://arcdog_description/meshes/calf.stl" scale="1 1 1"/>
                 </geometry>
-                <material name="orange"/>
             </visual>
             <collision>
-                <origin rpy="0 ${pi/2.0} 0" xyz="${calf_x_offset} 0 ${-calf_length/2.0}"/>
+                <origin rpy="0 ${PI/2.0} 0" xyz="0 0 ${-calf_length/2.0}"/>
                 <geometry>
                     <box size="${calf_length} ${calf_width} ${calf_height}"/>
@@ -174,10 +129,10 @@
             </inertial>
         </link>
-        <joint name="${prefix}_foot_fixed" type="fixed" dont_collapse="true">
-            <origin rpy="0 0 0" xyz="0 0 ${-calf_length}"/>
-            <parent link="${prefix}_calf"/>
-            <child link="${prefix}_foot"/>
+        <joint name="${name}_foot_fixed" type="fixed">
+			<origin rpy="0 0 0" xyz="0 0 ${-(calf_length)}"/>
+			<parent link="${name}_calf"/>
+			<child link="${name}_foot"/>
         </joint>
-        <link name="${prefix}_foot">
+        <link name="${name}_foot">
             <visual>
                 <origin rpy="0 0 0" xyz="0 0 0"/>
@@ -185,5 +140,4 @@
                     <sphere radius="${foot_radius-0.01}"/>
                 </geometry>
-                <material name="orange"/>
             </visual>
             <collision>
@@ -192,32 +146,4 @@
                     <sphere radius="${foot_radius}"/>
                 </geometry>
-                <surface>
-                <bounce>
-                    <restitution_coefficient>0</restitution_coefficient>
-                    <threshold>1e+06</threshold>
-                </bounce>
-                <friction>
-                    <ode>
-                    <mu>1.0</mu>
-                    <mu2>1.0</mu2>
-                    </ode>
-                    <bullet>
-                    <rolling_friction>0.3</rolling_friction>
-                    <friction2>50</friction2>
-                    </bullet>
-                </friction>
-                <contact>
-                    <ode>
-                    <kp>30000.0</kp>
-                    <kd>1000.0</kd>
-                    </ode>
-                    <bullet>
-                    <kp>30000.0</kp>
-                    <kd>1000.0</kd>
-                    <split_impulse>1</split_impulse>
-                    <split_impulse_penetration_threshold>-0.01</split_impulse_penetration_threshold>
-                    </bullet>
-                </contact>
-                </surface>
             </collision>
             <inertial>
@@ -229,34 +155,5 @@
             </inertial>
         </link>
-        <gazebo reference="${prefix}_foot_fixed">
-            <disableFixedJointLumping>true</disableFixedJointLumping>
-        </gazebo>
-        <gazebo reference="${prefix}_hip">
-            <mu1>0.2</mu1>
-            <mu2>0.2</mu2>
-            <material>Gazebo/DarkGrey</material>
-        </gazebo>
-        <gazebo reference="${prefix}_thigh">
-            <mu1>0.2</mu1>
-            <mu2>0.2</mu2>
-            <self_collide>0</self_collide>
-            <material>Gazebo/DarkGrey</material>
-            <kp value="1000000.0"/>
-            <kd value="100.0"/>
-        </gazebo>
-        <gazebo reference="${prefix}_calf">
-            <mu1>0.6</mu1>
-            <mu2>0.6</mu2>
-            <self_collide>1</self_collide>
-        </gazebo>
-        <gazebo reference="${prefix}_FOOT">
-            <mu1>0.6</mu1>
-            <mu2>0.6</mu2>
-            <self_collide>1</self_collide>
-            <material>Gazebo/DarkGrey</material>
-            <kp value="1000000.0"/>
-            <kd value="100.0"/>
-        </gazebo>
-        <xacro:leg_transmission name="${prefix}"/>
+        <xacro:leg_transmission name="${name}"/>
     </xacro:macro>
 </robot>

File: robot_description/arcdog_description/xacro/robot.xacro (robot description, xacro)
@@ -75,24 +75,49 @@
 			<mass value="0.001"/>
 			<origin rpy="0 0 0" xyz="0 0 0"/>
-			<inertia ixx="0.000001" ixy="0" ixz="0" iyy="0.000001" iyz="0" izz="0.000001"/>
+			<inertia ixx="0.0001" ixy="0" ixz="0" iyy="0.0001" iyz="0" izz="0.0001"/>
 		</inertial>
 		<visual>
 			<origin rpy="0 0 0" xyz="0 0 0"/>
-            <geometry>
-			<box size="0.015 0.015 0.004"/>
-            </geometry>
+			<geometry>
+				<box size="0.001 0.001 0.001"/>
+			</geometry>
+			<!-- <material name="red"/> -->
 		</visual>
+		<collision>
+			<origin rpy="0 0 0" xyz="0 0 0"/>
+			<geometry>
+				<box size=".001 .001 .001"/>
+			</geometry>
+		</collision>
 		</link>
-    <xacro:leg prefix="FR" mirror="-1" mirror_dae="False" front_hind="1" front_hind_dae="True" simulator="${simulator}" robot_type="${robot_type}">
-        <origin rpy="0 0 0" xyz="${leg_offset_x} ${-leg_offset_y} 0"/>
-    </xacro:leg>
-    <xacro:leg prefix="FL" mirror="1" mirror_dae="True" front_hind="1" front_hind_dae="True" simulator="${simulator}" robot_type="${robot_type}">
-        <origin rpy="0 0 0" xyz="${leg_offset_x} ${leg_offset_y} 0"/>
-    </xacro:leg>
-    <xacro:leg prefix="RR" mirror="-1" mirror_dae="False" front_hind="-1" front_hind_dae="False" simulator="${simulator}" robot_type="${robot_type}">
-        <origin rpy="0 0 0" xyz="${-leg_offset_x} ${-leg_offset_y} 0"/>
-    </xacro:leg>
-    <xacro:leg prefix="RL" mirror="1" mirror_dae="True" front_hind="-1" front_hind_dae="False" simulator="${simulator}" robot_type="${robot_type}">
-        <origin rpy="0 0 0" xyz="${-leg_offset_x} ${leg_offset_y} 0"/>
-    </xacro:leg>
+		<!--
+	<joint name="load_joint" type="fixed">
+			<parent link="trunk"/>
+			<child link="load_link"/>
+			<origin rpy="0 0 0" xyz="0 0 0"/>
+	</joint>
+	<link name="load_link">
+			<inertial>
+					<mass value="5"/>
+					<origin rpy="0 0 0" xyz="0 0 0"/>
+					<inertia ixx="0.01" ixy="0" ixz="0" iyy="0.01" iyz="0" izz="0.01"/>
+			</inertial>
+			<visual>
+					<origin rpy="0 0 0" xyz="0 0 0.2"/>
+					<geometry>
+							<box size="0.5 0.3 0.2"/>
+					</geometry>
+			</visual>
+			<collision>
+					<origin rpy="0 0 0" xyz="0 0 0"/>
+					<geometry>
+							<box size=".001 .001 .001"/>
+					</geometry>
+			</collision>
+	</link>
+-->
+	<xacro:leg name="FR" mirror="-1" mirror_dae="False" front_hind="1" front_hind_dae="True"/>
+	<xacro:leg name="FL" mirror="1" mirror_dae="True" front_hind="1" front_hind_dae="True"/>
+	<xacro:leg name="RR" mirror="-1" mirror_dae="False" front_hind="-1" front_hind_dae="False"/>
+	<xacro:leg name="RL" mirror="1" mirror_dae="True" front_hind="-1" front_hind_dae="False"/>
 </robot>
