Commit message: update xacro and urdf model (arcdog_test is the newest urdf model)

File: robot_description/arcdog_description/xacro/const.xacro (robot description, xacro)
@@ -5,5 +5,5 @@
     <xacro:property name="stick_mass" value="0.00001"/>
     <!-- simplified collision value -->
-    <xacro:property name="trunk_width" value="0.250"/>
+    <xacro:property name="trunk_width" value="0.121"/>
     <xacro:property name="trunk_length" value="0.361"/>
     <xacro:property name="trunk_height" value="0.114"/>
@@ -12,11 +12,11 @@
     <xacro:property name="thigh_shoulder_radius" value="0.0495"/>
     <xacro:property name="thigh_shoulder_length" value="0.03826"/>
-    <xacro:property name="thigh_width" value="?"/> //little larger than real value
+    <xacro:property name="thigh_width" value="0.040"/>
     <xacro:property name="thigh_height" value="0.06797"/>
     <xacro:property name="calf_width" value="0.02"/>
     <xacro:property name="calf_height" value="0.05"/>
     <xacro:property name="foot_radius" value="0.0265"/>
-    <!-- <xacro:property name="stick_radius" value="?"/>
-	<xacro:property name="stick_length" value="?"/> -->
+    <xacro:property name="stick_radius" value="?"/> //TODO
+	<xacro:property name="stick_length" value="?"/> //TODO
     <!-- kinematic value -->
     <xacro:property name="thigh_offset" value="0.11475"/>
@@ -26,16 +26,16 @@
     <xacro:property name="leg_offset_x" value="0.2515"/>
     <xacro:property name="leg_offset_y" value="0.0605"/>
-    <!-- <xacro:property name="trunk_offset_z" value="0.01675"/> //TODO -->
+    <xacro:property name="trunk_offset_z" value="0.01675"/> //TODO
     <xacro:property name="hip_offset" value="0.11475"/> //go2 special point, puting hip collision model at thigh position
     <!-- offset of link locations (left front) -->
-    <!-- <xacro:property name="hip_offset_x" value="?"/>
-	<xacro:property name="hip_offset_y" value="?"/>
-	<xacro:property name="hip_offset_z" value="?"/>
-	<xacro:property name="thigh_offset_x" value="?"/>
-	<xacro:property name="thigh_offset_y" value="?"/>
-	<xacro:property name="thigh_offset_z" value="?"/>
-	<xacro:property name="calf_offset_x" value="?"/>
-	<xacro:property name="calf_offset_y" value="?"/>
-	<xacro:property name="calf_offset_z" value="?"/> -->
+    <xacro:property name="hip_offset_x" value="?"/> //TODO
+	<xacro:property name="hip_offset_y" value="?"/> //TODO
+	<xacro:property name="hip_offset_z" value="?"/> //TODO
+	<xacro:property name="thigh_offset_x" value="?"/> //TODO
+	<xacro:property name="thigh_offset_y" value="?"/> //TODO
+	<xacro:property name="thigh_offset_z" value="?"/> //TODO
+	<xacro:property name="calf_offset_x" value="?"/> //TODO
+	<xacro:property name="calf_offset_y" value="?"/> //TODO
+	<xacro:property name="calf_offset_z" value="?"/> //TODO
     <!-- joint limits -->
     <xacro:property name="damping" value="0.05"/>

File: robot_description/go2_description/urdf/go2_test.urdf (robot description, URDF)
Before this commit: robot arcdog, 19 links, 18 joints
Links:
- link FL_calf: mass 0.18 -> 0.154; geometry collision box size=0.213 0.016 0.016; visual mesh filename=file:///home/lxq/colcon_ws/install/go2_description/share/go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 scale=1 1 1
- link FL_foot: geometry collision sphere radius=0.02; visual sphere radius=0.01
- link FL_hip: mass 1.108 -> 0.678; geometry collision cylinder length=0.04 radius=0.046; visual mesh filename=file:///home/lxq/colcon_ws/install/go2_description/share/go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 scale=1 1 1
- link FL_thigh: mass 1.636 -> 1.152; geometry collision box size=0.213 0.0245 0.034; visual mesh filename=file:///home/lxq/colcon_ws/install/go2_description/share/go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 scale=1 1 1
- link FR_calf: mass 0.18 -> 0.154; geometry collision box size=0.213 0.016 0.016; visual mesh filename=file:///home/lxq/colcon_ws/install/go2_description/share/go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 scale=1 1 1
- link FR_foot: geometry collision sphere radius=0.02; visual sphere radius=0.01
- link FR_hip: mass 1.108 -> 0.678; geometry collision cylinder length=0.04 radius=0.046; visual mesh filename=file:///home/lxq/colcon_ws/install/go2_description/share/go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 scale=1 1 1
- link FR_thigh: mass 1.636 -> 1.152; geometry collision box size=0.213 0.0245 0.034; visual mesh filename=file:///home/lxq/colcon_ws/install/go2_description/share/go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 scale=1 1 1
- link RL_calf: mass 0.18 -> 0.154; geometry collision box size=0.213 0.016 0.016; visual mesh filename=file:///home/lxq/colcon_ws/install/go2_description/share/go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 scale=1 1 1
- link RL_foot: geometry collision sphere radius=0.02; visual sphere radius=0.01
- link RL_hip: mass 1.108 -> 0.678; geometry collision cylinder length=0.04 radius=0.046; visual mesh filename=file:///home/lxq/colcon_ws/install/go2_description/share/go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 scale=1 1 1
- link RL_thigh: mass 1.636 -> 1.152; geometry collision box size=0.213 0.0245 0.034; visual mesh filename=file:///home/lxq/colcon_ws/install/go2_description/share/go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 scale=1 1 1
- link RR_calf: mass 0.18 -> 0.154; geometry collision box size=0.213 0.016 0.016; visual mesh filename=file:///home/lxq/colcon_ws/install/go2_description/share/go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 scale=1 1 1
- link RR_foot: geometry collision sphere radius=0.02; visual sphere radius=0.01
- link RR_hip: mass 1.108 -> 0.678; geometry collision cylinder length=0.04 radius=0.046; visual mesh filename=file:///home/lxq/colcon_ws/install/go2_description/share/go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 scale=1 1 1
- link RR_thigh: mass 1.636 -> 1.152; geometry collision box size=0.213 0.0245 0.034; visual mesh filename=file:///home/lxq/colcon_ws/install/go2_description/share/go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 scale=1 1 1
- link trunk: mass 5.742 -> 6.921; geometry collision box size=0.3762 0.0935 0.114; visual mesh filename=file:///home/lxq/colcon_ws/install/go2_description/share/go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 scale=1 1 1
Joints:
- joint FL_calf_joint: limit lower=-2.775073510670984 upper=-0.6457718232379019 effort=44.4 velocity=15.89 -> lower=-2.7227 upper=-0.83776 effort=35.55 velocity=20.06; origin xyz=0 0 -0.245 rpy=0 0 0 -> xyz=0 0 -0.213 rpy=0 0 0
- joint FL_foot_fixed: origin xyz=0 0 -0.19534 rpy=0 0 0 -> xyz=0 0 -0.213 rpy=0 0 0
- joint FL_hip_joint: limit lower=-1.2217304763960306 upper=1.2217304763960306 effort=35.278 velocity=20 -> lower=-1.0472 upper=1.0472 effort=23.7 velocity=30.1; origin xyz=0.2515 0.0605 0 rpy=0 0 0 -> xyz=0.1934 0.0465 0 rpy=0 0 0
- joint FL_thigh_joint: limit lower=-1.5708 upper=3.4907 effort=35.278 velocity=20 -> lower=-1.5708 upper=3.4907 effort=23.7 velocity=30.1; origin xyz=0 0.11475 0 rpy=0 0 0 -> xyz=0 0.0955 0 rpy=0 0 0
- joint FR_calf_joint: limit lower=-2.775073510670984 upper=-0.6457718232379019 effort=44.4 velocity=15.89 -> lower=-2.7227 upper=-0.83776 effort=35.55 velocity=20.06; origin xyz=0 0 -0.245 rpy=0 0 0 -> xyz=0 0 -0.213 rpy=0 0 0
- joint FR_foot_fixed: origin xyz=0 0 -0.19534 rpy=0 0 0 -> xyz=0 0 -0.213 rpy=0 0 0
- joint FR_hip_joint: limit lower=-1.2217304763960306 upper=1.2217304763960306 effort=35.278 velocity=20 -> lower=-1.0472 upper=1.0472 effort=23.7 velocity=30.1; origin xyz=0.2515 -0.0605 0 rpy=0 0 0 -> xyz=0.1934 -0.0465 0 rpy=0 0 0
- joint FR_thigh_joint: limit lower=-1.5708 upper=3.4907 effort=35.278 velocity=20 -> lower=-1.5708 upper=3.4907 effort=23.7 velocity=30.1; origin xyz=0 -0.11475 0 rpy=0 0 0 -> xyz=0 -0.0955 0 rpy=0 0 0
- joint RL_calf_joint: limit lower=-2.775073510670984 upper=-0.6457718232379019 effort=44.4 velocity=15.89 -> lower=-2.7227 upper=-0.83776 effort=35.55 velocity=20.06; origin xyz=0 0 -0.245 rpy=0 0 0 -> xyz=0 0 -0.213 rpy=0 0 0
- joint RL_foot_fixed: origin xyz=0 0 -0.19534 rpy=0 0 0 -> xyz=0 0 -0.213 rpy=0 0 0
- joint RL_hip_joint: limit lower=-1.2217304763960306 upper=1.2217304763960306 effort=35.278 velocity=20 -> lower=-1.0472 upper=1.0472 effort=23.7 velocity=30.1; origin xyz=-0.2515 0.0605 0 rpy=0 0 0 -> xyz=-0.1934 0.0465 0 rpy=0 0 0
- joint RL_thigh_joint: limit lower=-1.5708 upper=3.4907 effort=35.278 velocity=20 -> lower=-1.5708 upper=3.4907 effort=23.7 velocity=30.1; origin xyz=0 0.11475 0 rpy=0 0 0 -> xyz=0 0.0955 0 rpy=0 0 0
- joint RR_calf_joint: limit lower=-2.775073510670984 upper=-0.6457718232379019 effort=44.4 velocity=15.89 -> lower=-2.7227 upper=-0.83776 effort=35.55 velocity=20.06; origin xyz=0 0 -0.245 rpy=0 0 0 -> xyz=0 0 -0.213 rpy=0 0 0
- joint RR_foot_fixed: origin xyz=0 0 -0.19534 rpy=0 0 0 -> xyz=0 0 -0.213 rpy=0 0 0
- joint RR_hip_joint: limit lower=-1.2217304763960306 upper=1.2217304763960306 effort=35.278 velocity=20 -> lower=-1.0472 upper=1.0472 effort=23.7 velocity=30.1; origin xyz=-0.2515 -0.0605 0 rpy=0 0 0 -> xyz=-0.1934 -0.0465 0 rpy=0 0 0
- joint RR_thigh_joint: limit lower=-1.5708 upper=3.4907 effort=35.278 velocity=20 -> lower=-1.5708 upper=3.4907 effort=23.7 velocity=30.1; origin xyz=0 -0.11475 0 rpy=0 0 0 -> xyz=0 -0.0955 0 rpy=0 0 0
