Commit message: update dynamic value

File: robot_description/arcdog_description/urdf/arcdog_test.urdf (robot description, URDF)
Before this commit: robot arcdog_description, 19 links, 18 joints
Links:
- link FL_calf: mass 0.213 -> 0.18
- link FL_hip: mass 0.8365 -> 1.108
- link FL_thigh: mass 1.987 -> 1.636
- link FR_calf: mass 0.213 -> 0.18
- link FR_hip: mass 0.8365 -> 1.108
- link FR_thigh: mass 1.987 -> 1.636
- link RL_calf: mass 0.213 -> 0.18
- link RL_hip: mass 0.8365 -> 1.108
- link RL_thigh: mass 1.987 -> 1.636
- link RR_calf: mass 0.213 -> 0.18
- link RR_hip: mass 0.8365 -> 1.108
- link RR_thigh: mass 1.987 -> 1.636
- link base: mass 8.4845 -> 5.742

File: robot_description/arcdog_description/xacro/const.xacro (robot description, xacro)
@@ -43,49 +43,49 @@
     <xacro:property name="calf_velocity_max" value="15.89"/>
     <xacro:property name="calf_torque_max" value="44.4"/>
-    <!-- dynamics inertial value    total 22.0kg-->
+    <!-- dynamics inertial value    total 17.43kg-->
     <!-- trunk -->
-    <xacro:property name="trunk_mass" value="8.4845"/>
-    <xacro:property name="trunk_com_x" value="-0.000466"/>
-    <xacro:property name="trunk_com_y" value="-0.000692"/>
-    <xacro:property name="trunk_com_z" value="-0.008587"/>
-    <xacro:property name="trunk_ixx" value="0.031520962"/>
-    <xacro:property name="trunk_ixy" value="-0.000002732"/>
-    <xacro:property name="trunk_ixz" value="-0.000285792"/>
-    <xacro:property name="trunk_iyy" value="0.143653339"/>
-    <xacro:property name="trunk_iyz" value="0.000011831"/>
-    <xacro:property name="trunk_izz" value="0.159618308"/>
+    <xacro:property name="trunk_mass" value="5.742"/>
+    <xacro:property name="trunk_com_x" value="-0.002250"/>
+    <xacro:property name="trunk_com_y" value="0.000116"/>
+    <xacro:property name="trunk_com_z" value="-0.001452"/>
+    <xacro:property name="trunk_ixx" value="0.037914363"/>
+    <xacro:property name="trunk_ixy" value="0.000098848"/>
+    <xacro:property name="trunk_ixz" value="-0.000073338"/>
+    <xacro:property name="trunk_iyy" value="0.119267297"/>
+    <xacro:property name="trunk_iyz" value="0.000013463"/>
+    <xacro:property name="trunk_izz" value="0.142804844"/>
     <!-- hip (left front) -->
-    <xacro:property name="hip_mass" value="0.8365"/>
-    <xacro:property name="hip_com_x" value="-0.006155"/>
-    <xacro:property name="hip_com_y" value="-0.006930"/>
-    <xacro:property name="hip_com_z" value="0.000002"/>
-    <xacro:property name="hip_ixx" value="0.000594660"/>
-    <xacro:property name="hip_ixy" value="-0.000009124"/>
-    <xacro:property name="hip_ixz" value="0.000000048"/>
-    <xacro:property name="hip_iyy" value="0.001055081"/>
-    <xacro:property name="hip_iyz" value="0.000000016"/>
-    <xacro:property name="hip_izz" value="0.000764676"/>
+    <xacro:property name="hip_mass" value="1.108"/>
+    <xacro:property name="hip_com_x" value="-0.0082"/>
+    <xacro:property name="hip_com_y" value="0.000984"/>
+    <xacro:property name="hip_com_z" value="0.000162"/>
+    <xacro:property name="hip_ixx" value="0.000972670"/>
+    <xacro:property name="hip_ixy" value="0.000004550"/>
+    <xacro:property name="hip_ixz" value="0.000000139"/>
+    <xacro:property name="hip_iyy" value="0.001754403"/>
+    <xacro:property name="hip_iyz" value="0.000001705"/>
+    <xacro:property name="hip_izz" value="0.001311138"/>
     <!-- thigh -->
-    <xacro:property name="thigh_mass" value="1.987"/>
-    <xacro:property name="thigh_com_x" value="0.003996"/>
-    <xacro:property name="thigh_com_y" value="0.028346"/>
-    <xacro:property name="thigh_com_z" value="-0.020538"/>
-    <xacro:property name="thigh_ixx" value="0.008811372"/>
-    <xacro:property name="thigh_ixy" value="-0.000167657"/>
-    <xacro:property name="thigh_ixz" value="-0.000632186"/>
-    <xacro:property name="thigh_iyy" value="0.007563533"/>
-    <xacro:property name="thigh_iyz" value="0.001133315"/>
-    <xacro:property name="thigh_izz" value="0.003133589"/>
+    <xacro:property name="thigh_mass" value="1.636"/>
+    <xacro:property name="thigh_com_x" value="-0.004484"/>
+    <xacro:property name="thigh_com_y" value="-0.033084"/>
+    <xacro:property name="thigh_com_z" value="-0.030728"/>
+    <xacro:property name="thigh_ixx" value="0.009596889"/>
+    <xacro:property name="thigh_ixy" value="-0.000241414"/>
+    <xacro:property name="thigh_ixz" value="0.000789459"/>
+    <xacro:property name="thigh_iyy" value="0.009201469"/>
+    <xacro:property name="thigh_iyz" value="-0.001676085"/>
+    <xacro:property name="thigh_izz" value="0.002385568"/>
     <!-- calf -->
-    <xacro:property name="calf_mass" value="0.213"/>
-    <xacro:property name="calf_com_x" value="-0.000873"/>
+    <xacro:property name="calf_mass" value="0.180"/>
+    <xacro:property name="calf_com_x" value="0.005552"/>
     <xacro:property name="calf_com_y" value="0.000"/>
-    <xacro:property name="calf_com_z" value="-0.114455"/>
-    <xacro:property name="calf_ixx" value="0.001561890"/>
+    <xacro:property name="calf_com_z" value="-0.108279"/>
+    <xacro:property name="calf_ixx" value="0.001206453"/>
     <xacro:property name="calf_ixy" value="-0.000"/>
-    <xacro:property name="calf_ixz" value="0.000021547"/>
-    <xacro:property name="calf_iyy" value="0.001566663"/>
+    <xacro:property name="calf_ixz" value="-0.000026747"/>
+    <xacro:property name="calf_iyy" value="0.001233919"/>
     <xacro:property name="calf_iyz" value="0.000000001"/>
-    <xacro:property name="calf_izz" value="0.000019643"/>
+    <xacro:property name="calf_izz" value="0.000039128"/>
     <!-- foot -->
     <xacro:property name="foot_mass" value="0.06"/>

Commit message: update arcdog urdf

File: robot_description/arcdog_description/urdf/arcdog_test.urdf (robot description, URDF)
Before this commit: robot arcdog_description, 19 links, 18 joints
Joints:
- removed joint FL_HAA
- removed joint FL_HFE
- removed joint FL_KFE
- removed joint FR_HAA
- removed joint FR_HFE
- removed joint FR_KFE
- removed joint RL_HAA
- removed joint RL_HFE
- removed joint RL_KFE
- removed joint RR_HAA
- removed joint RR_HFE
- removed joint RR_KFE
- added joint FL_calf_joint: type revolute, parent FL_thigh, child FL_calf, origin xyz=0 0 -0.245 rpy=0 0 0, axis 0 1 0, limit lower=-2.775073510670984 upper=-0.6457718232379019 effort=44.4 velocity=15.89
- added joint FL_hip_joint: type revolute, parent base, child FL_hip, origin xyz=0.2515 0.0605 0 rpy=0 0 0, axis 1 0 0, limit lower=-1.2217304763960306 upper=1.2217304763960306 effort=35.278 velocity=20
- added joint FL_thigh_joint: type revolute, parent FL_hip, child FL_thigh, origin xyz=0 0.11475 0 rpy=0 0 0, axis 0 1 0, limit lower=-1.5708 upper=3.4907 effort=35.278 velocity=20
- added joint FR_calf_joint: type revolute, parent FR_thigh, child FR_calf, origin xyz=0 0 -0.245 rpy=0 0 0, axis 0 1 0, limit lower=-2.775073510670984 upper=-0.6457718232379019 effort=44.4 velocity=15.89
- added joint FR_hip_joint: type revolute, parent base, child FR_hip, origin xyz=0.2515 -0.0605 0 rpy=0 0 0, axis 1 0 0, limit lower=-1.2217304763960306 upper=1.2217304763960306 effort=35.278 velocity=20
- added joint FR_thigh_joint: type revolute, parent FR_hip, child FR_thigh, origin xyz=0 -0.11475 0 rpy=0 0 0, axis 0 1 0, limit lower=-1.5708 upper=3.4907 effort=35.278 velocity=20
- added joint RL_calf_joint: type revolute, parent RL_thigh, child RL_calf, origin xyz=0 0 -0.245 rpy=0 0 0, axis 0 1 0, limit lower=-2.775073510670984 upper=-0.6457718232379019 effort=44.4 velocity=15.89
- added joint RL_hip_joint: type revolute, parent base, child RL_hip, origin xyz=-0.2515 0.0605 0 rpy=0 0 0, axis 1 0 0, limit lower=-1.2217304763960306 upper=1.2217304763960306 effort=35.278 velocity=20
- added joint RL_thigh_joint: type revolute, parent RL_hip, child RL_thigh, origin xyz=0 0.11475 0 rpy=0 0 0, axis 0 1 0, limit lower=-1.5708 upper=3.4907 effort=35.278 velocity=20
- added joint RR_calf_joint: type revolute, parent RR_thigh, child RR_calf, origin xyz=0 0 -0.245 rpy=0 0 0, axis 0 1 0, limit lower=-2.775073510670984 upper=-0.6457718232379019 effort=44.4 velocity=15.89
- added joint RR_hip_joint: type revolute, parent base, child RR_hip, origin xyz=-0.2515 -0.0605 0 rpy=0 0 0, axis 1 0 0, limit lower=-1.2217304763960306 upper=1.2217304763960306 effort=35.278 velocity=20
- added joint RR_thigh_joint: type revolute, parent RR_hip, child RR_thigh, origin xyz=0 -0.11475 0 rpy=0 0 0, axis 0 1 0, limit lower=-1.5708 upper=3.4907 effort=35.278 velocity=20

Commit message: recover urdf, nothing happened

File: robot_description/arcdog_description/urdf/arcdog_test.urdf (robot description, URDF)
Before this commit: robot arcdog_description, 19 links, 18 joints
Joints:
- removed joint FL_calf_joint
- removed joint FL_hip_joint
- removed joint FL_thigh_joint
- removed joint FR_calf_joint
- removed joint FR_hip_joint
- removed joint FR_thigh_joint
- removed joint RL_calf_joint
- removed joint RL_hip_joint
- removed joint RL_thigh_joint
- removed joint RR_calf_joint
- removed joint RR_hip_joint
- removed joint RR_thigh_joint
- added joint FL_HAA: type revolute, parent base, child FL_hip, origin xyz=0.2515 0.0605 0 rpy=0 0 0, axis 1 0 0, limit lower=-1.2217304763960306 upper=1.2217304763960306 effort=35.278 velocity=20
- added joint FL_HFE: type revolute, parent FL_hip, child FL_thigh, origin xyz=0 0.11475 0 rpy=0 0 0, axis 0 1 0, limit lower=-1.5708 upper=3.4907 effort=35.278 velocity=20
- added joint FL_KFE: type revolute, parent FL_thigh, child FL_calf, origin xyz=0 0 -0.245 rpy=0 0 0, axis 0 1 0, limit lower=-2.775073510670984 upper=-0.6457718232379019 effort=44.4 velocity=15.89
- added joint FR_HAA: type revolute, parent base, child FR_hip, origin xyz=0.2515 -0.0605 0 rpy=0 0 0, axis 1 0 0, limit lower=-1.2217304763960306 upper=1.2217304763960306 effort=35.278 velocity=20
- added joint FR_HFE: type revolute, parent FR_hip, child FR_thigh, origin xyz=0 -0.11475 0 rpy=0 0 0, axis 0 1 0, limit lower=-1.5708 upper=3.4907 effort=35.278 velocity=20
- added joint FR_KFE: type revolute, parent FR_thigh, child FR_calf, origin xyz=0 0 -0.245 rpy=0 0 0, axis 0 1 0, limit lower=-2.775073510670984 upper=-0.6457718232379019 effort=44.4 velocity=15.89
- added joint RL_HAA: type revolute, parent base, child RL_hip, origin xyz=-0.2515 0.0605 0 rpy=0 0 0, axis 1 0 0, limit lower=-1.2217304763960306 upper=1.2217304763960306 effort=35.278 velocity=20
- added joint RL_HFE: type revolute, parent RL_hip, child RL_thigh, origin xyz=0 0.11475 0 rpy=0 0 0, axis 0 1 0, limit lower=-1.5708 upper=3.4907 effort=35.278 velocity=20
- added joint RL_KFE: type revolute, parent RL_thigh, child RL_calf, origin xyz=0 0 -0.245 rpy=0 0 0, axis 0 1 0, limit lower=-2.775073510670984 upper=-0.6457718232379019 effort=44.4 velocity=15.89
- added joint RR_HAA: type revolute, parent base, child RR_hip, origin xyz=-0.2515 -0.0605 0 rpy=0 0 0, axis 1 0 0, limit lower=-1.2217304763960306 upper=1.2217304763960306 effort=35.278 velocity=20
- added joint RR_HFE: type revolute, parent RR_hip, child RR_thigh, origin xyz=0 -0.11475 0 rpy=0 0 0, axis 0 1 0, limit lower=-1.5708 upper=3.4907 effort=35.278 velocity=20
- added joint RR_KFE: type revolute, parent RR_thigh, child RR_calf, origin xyz=0 0 -0.245 rpy=0 0 0, axis 0 1 0, limit lower=-2.775073510670984 upper=-0.6457718232379019 effort=44.4 velocity=15.89
