Commit message: update arcdog_description (arcdog_test.urdf is the newest model)

File: robot_description/arcdog_description/urdf/arcdog_test1209.urdf (robot description, URDF)
Before this commit: robot arcdog, 19 links, 18 joints
Links:
- link FL_thigh: geometry collision box size=0.245 0.04 0.06797; collision cylinder length=0.03826 radius=0.0495
- link FR_thigh: geometry collision box size=0.245 0.04 0.06797; collision cylinder length=0.03826 radius=0.0495
- link RL_thigh: geometry collision box size=0.245 0.04 0.06797; collision cylinder length=0.03826 radius=0.0495
- link RR_thigh: geometry collision box size=0.245 0.04 0.06797; collision cylinder length=0.03826 radius=0.0495
- link imu_link: geometry visual box size=0.015 0.015 0.004
- link trunk: geometry collision box size=0.361 0.25 0.114; visual mesh filename=file:///home/lxq/colcon_ws/install/arcdog_description/share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 scale=1 1 1
Joints:
- joint FL_hip_joint: parent trunk -> base
- joint FR_hip_joint: parent trunk -> base
- joint RL_hip_joint: parent trunk -> base
- joint RR_hip_joint: parent trunk -> base

File: robot_description/arcdog_description/urdf/arcdog_test_backup.urdf (robot description, URDF)
Before this commit: robot arcdog, 19 links, 18 joints
Links:
- removed link imu_link
- removed link trunk
- added link body; visual box size=0.001 0.001 0.001
- added link unitree_imu, mass 0.01; visual box size=0.015 0.015 0.004
- link FL_calf: mass 0.213 -> 0.18; geometry collision box size=0.19534 0.02 0.05; visual mesh filename=package://arclab_robot_description/meshes/quadrupedal_robot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 scale=1 1 1
- link FL_hip: mass 0.8365 -> 1.108; geometry collision cylinder length=0.0834 radius=0.0495; visual mesh filename=package://arclab_robot_description/meshes/quadrupedal_robot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 scale=1 1 1
- link FL_thigh: mass 1.987 -> 1.636; geometry collision box size=0.245 0.04 0.06797; collision cylinder length=0.03826 radius=0.0495
- link FR_calf: mass 0.213 -> 0.18; geometry collision box size=0.19534 0.02 0.05; visual mesh filename=package://arclab_robot_description/meshes/quadrupedal_robot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 scale=1 1 1
- link FR_hip: mass 0.8365 -> 1.108; geometry collision cylinder length=0.0834 radius=0.0495; visual mesh filename=package://arclab_robot_description/meshes/quadrupedal_robot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 scale=1 1 1
- link FR_thigh: mass 1.987 -> 1.636; geometry collision box size=0.245 0.04 0.06797; collision cylinder length=0.03826 radius=0.0495
- link RL_calf: mass 0.213 -> 0.18; geometry collision box size=0.19534 0.02 0.05; visual mesh filename=package://arclab_robot_description/meshes/quadrupedal_robot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 scale=1 1 1
- link RL_hip: mass 0.8365 -> 1.108; geometry collision cylinder length=0.0834 radius=0.0495; visual mesh filename=package://arclab_robot_description/meshes/quadrupedal_robot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 scale=1 1 1
- link RL_thigh: mass 1.987 -> 1.636; geometry collision box size=0.245 0.04 0.06797; collision cylinder length=0.03826 radius=0.0495
- link RR_calf: mass 0.213 -> 0.18; geometry collision box size=0.19534 0.02 0.05; visual mesh filename=package://arclab_robot_description/meshes/quadrupedal_robot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 scale=1 1 1
- link RR_hip: mass 0.8365 -> 1.108; geometry collision cylinder length=0.0834 radius=0.0495; visual mesh filename=package://arclab_robot_description/meshes/quadrupedal_robot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 scale=1 1 1
- link RR_thigh: mass 1.987 -> 1.636; geometry collision box size=0.245 0.04 0.06797; collision cylinder length=0.03826 radius=0.0495
- link base: mass None -> 5.742; geometry collision box size=0.361 0.25 0.114; visual mesh filename=package://arclab_robot_description/meshes/quadrupedal_robot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 scale=1 1 1
Joints:
- removed joint FL_calf_joint
- removed joint FL_hip_joint
- removed joint FL_thigh_joint
- removed joint FR_calf_joint
- removed joint FR_hip_joint
- removed joint FR_thigh_joint
- removed joint RL_calf_joint
- removed joint RL_hip_joint
- removed joint RL_thigh_joint
- removed joint RR_calf_joint
- removed joint RR_hip_joint
- removed joint RR_thigh_joint
- removed joint imu_joint
- added joint FL_HAA: type revolute, parent base, child FL_hip, origin xyz=0.2515 0.0605 0 rpy=0 0 0, axis 1 0 0, limit lower=-1.2217304763960306 upper=1.2217304763960306 effort=35.278 velocity=20
- added joint FL_HFE: type revolute, parent FL_hip, child FL_thigh, origin xyz=0 0.11475 0 rpy=0 0 0, axis 0 1 0, limit lower=-1.5708 upper=3.4907 effort=35.278 velocity=20
- added joint FL_KFE: type revolute, parent FL_thigh, child FL_calf, origin xyz=0 0 -0.245 rpy=0 0 0, axis 0 1 0, limit lower=-2.775073510670984 upper=-0.6457718232379019 effort=44.4 velocity=15.89
- added joint FR_HAA: type revolute, parent base, child FR_hip, origin xyz=0.2515 -0.0605 0 rpy=0 0 0, axis 1 0 0, limit lower=-1.2217304763960306 upper=1.2217304763960306 effort=35.278 velocity=20
- added joint FR_HFE: type revolute, parent FR_hip, child FR_thigh, origin xyz=0 -0.11475 0 rpy=0 0 0, axis 0 1 0, limit lower=-1.5708 upper=3.4907 effort=35.278 velocity=20
- added joint FR_KFE: type revolute, parent FR_thigh, child FR_calf, origin xyz=0 0 -0.245 rpy=0 0 0, axis 0 1 0, limit lower=-2.775073510670984 upper=-0.6457718232379019 effort=44.4 velocity=15.89
- added joint RL_HAA: type revolute, parent base, child RL_hip, origin xyz=-0.2515 0.0605 0 rpy=0 0 0, axis 1 0 0, limit lower=-1.2217304763960306 upper=1.2217304763960306 effort=35.278 velocity=20
- added joint RL_HFE: type revolute, parent RL_hip, child RL_thigh, origin xyz=0 0.11475 0 rpy=0 0 0, axis 0 1 0, limit lower=-1.5708 upper=3.4907 effort=35.278 velocity=20
- added joint RL_KFE: type revolute, parent RL_thigh, child RL_calf, origin xyz=0 0 -0.245 rpy=0 0 0, axis 0 1 0, limit lower=-2.775073510670984 upper=-0.6457718232379019 effort=44.4 velocity=15.89
- added joint RR_HAA: type revolute, parent base, child RR_hip, origin xyz=-0.2515 -0.0605 0 rpy=0 0 0, axis 1 0 0, limit lower=-1.2217304763960306 upper=1.2217304763960306 effort=35.278 velocity=20
- added joint RR_HFE: type revolute, parent RR_hip, child RR_thigh, origin xyz=0 -0.11475 0 rpy=0 0 0, axis 0 1 0, limit lower=-1.5708 upper=3.4907 effort=35.278 velocity=20
- added joint RR_KFE: type revolute, parent RR_thigh, child RR_calf, origin xyz=0 0 -0.245 rpy=0 0 0, axis 0 1 0, limit lower=-2.775073510670984 upper=-0.6457718232379019 effort=44.4 velocity=15.89
- added joint unitree_imu_joint: type fixed, parent base, child unitree_imu, origin xyz=0. 0. 0. rpy=0. 0. 0.
- joint FL_foot_fixed: origin xyz=0 0 -0.23704 rpy=0 0 0 -> xyz=0 0 -0.19534 rpy=0 0 0
- joint FR_foot_fixed: origin xyz=0 0 -0.23704 rpy=0 0 0 -> xyz=0 0 -0.19534 rpy=0 0 0
- joint RL_foot_fixed: origin xyz=0 0 -0.23704 rpy=0 0 0 -> xyz=0 0 -0.19534 rpy=0 0 0
- joint RR_foot_fixed: origin xyz=0 0 -0.23704 rpy=0 0 0 -> xyz=0 0 -0.19534 rpy=0 0 0
- joint floating_base: child trunk -> base; parent base -> body

File: robot_description/arcdog_description/xacro/const.xacro (robot description, xacro)
@@ -2,7 +2,8 @@
 <robot xmlns:xacro="http://www.ros.org/wiki/xacro" name="arcdog_description">
     <!-- Constants for robot dimensions -->
+    <xacro:property name="PI" value="3.1415926535897931"/>
     <xacro:property name="stick_mass" value="0.00001"/>
     <!-- simplified collision value -->
-    <xacro:property name="trunk_width" value="0.250"/>
+    <xacro:property name="trunk_width" value="0.121"/>
     <xacro:property name="trunk_length" value="0.361"/>
     <xacro:property name="trunk_height" value="0.114"/>
@@ -11,12 +12,11 @@
     <xacro:property name="thigh_shoulder_radius" value="0.0495"/>
     <xacro:property name="thigh_shoulder_length" value="0.03826"/>
-    <xacro:property name="thigh_shoulder_y_offset" value="0.0"/>
-    <xacro:property name="thigh_width" value="0.040"/> //little larger than real value
+    <xacro:property name="thigh_width" value="0.040"/>
     <xacro:property name="thigh_height" value="0.06797"/>
-    <xacro:property name="thigh_x_offset" value="0.000"/>
     <xacro:property name="calf_width" value="0.02"/>
     <xacro:property name="calf_height" value="0.05"/>
-    <xacro:property name="calf_x_offset" value="0.000"/>
     <xacro:property name="foot_radius" value="0.0265"/>
+    <xacro:property name="stick_radius" value="?"/> //TODO
+	<xacro:property name="stick_length" value="?"/> //TODO
     <!-- kinematic value -->
     <xacro:property name="thigh_offset" value="0.11475"/>
@@ -27,18 +27,28 @@
     <xacro:property name="leg_offset_y" value="0.0605"/>
     <xacro:property name="trunk_offset_z" value="0.01675"/> //TODO
-    <xacro:property name="hip_offset" value="0.0001"/> //TODO
+    <xacro:property name="hip_offset" value="0.11475"/> //go2 special point, puting hip collision model at thigh position
+    <!-- offset of link locations (left front) -->
+    <xacro:property name="hip_offset_x" value="?"/> //TODO
+	<xacro:property name="hip_offset_y" value="?"/> //TODO
+	<xacro:property name="hip_offset_z" value="?"/> //TODO
+	<xacro:property name="thigh_offset_x" value="?"/> //TODO
+	<xacro:property name="thigh_offset_y" value="?"/> //TODO
+	<xacro:property name="thigh_offset_z" value="?"/> //TODO
+	<xacro:property name="calf_offset_x" value="?"/> //TODO
+	<xacro:property name="calf_offset_y" value="?"/> //TODO
+	<xacro:property name="calf_offset_z" value="?"/> //TODO
     <!-- joint limits -->
     <xacro:property name="damping" value="0.05"/>
     <xacro:property name="friction" value="0.01"/>
-    <xacro:property name="hip_max" value="${70*pi/180.0}"/>
-    <xacro:property name="hip_min" value="${-70*pi/180.0}"/>
+    <xacro:property name="hip_position_max" value="${70*pi/180.0}"/>
+    <xacro:property name="hip_position_min" value="${-70*pi/180.0}"/>
     <xacro:property name="hip_velocity_max" value="20"/>
     <xacro:property name="hip_torque_max" value="35.278"/>
-    <xacro:property name="thigh_max" value="3.4907"/>
-    <xacro:property name="thigh_min" value="-1.5708"/>
+    <xacro:property name="thigh_position_max" value="3.4907"/>
+    <xacro:property name="thigh_position_min" value="-1.5708"/>
     <xacro:property name="thigh_velocity_max" value="20"/>
     <xacro:property name="thigh_torque_max" value="35.278"/>
-    <xacro:property name="calf_max" value="${-37*pi/180.0}"/>
-    <xacro:property name="calf_min" value="${-159*pi/180.0}"/>
+    <xacro:property name="calf_position_max" value="${-37*pi/180.0}"/>
+    <xacro:property name="calf_position_min" value="${-159*pi/180.0}"/>
     <xacro:property name="calf_velocity_max" value="15.89"/>
     <xacro:property name="calf_torque_max" value="44.4"/>

File: robot_description/arcdog_description/xacro/robot.xacro (robot description, xacro)
@@ -4,8 +4,4 @@
 	<xacro:arg name="GAZEBO" default="false"/>
 	<xacro:arg name="CLASSIC" default="false"/>
-    <xacro:arg name="robot_type" default="arcdog"/>
-    <xacro:property name="robot_type" value="$(arg robot_type)"/>
-	<xacro:arg name="simulator" default="test"/>
-    <xacro:property name="simulator" value="$(arg simulator)"/>
 	<xacro:include filename="$(find arcdog_description)/xacro/const.xacro"/>
 	<xacro:include filename="$(find arcdog_description)/xacro/materials.xacro"/>
@@ -79,24 +75,49 @@
 			<mass value="0.001"/>
 			<origin rpy="0 0 0" xyz="0 0 0"/>
-			<inertia ixx="0.000001" ixy="0" ixz="0" iyy="0.000001" iyz="0" izz="0.000001"/>
+			<inertia ixx="0.0001" ixy="0" ixz="0" iyy="0.0001" iyz="0" izz="0.0001"/>
 		</inertial>
 		<visual>
 			<origin rpy="0 0 0" xyz="0 0 0"/>
-            <geometry>
-			<box size="0.015 0.015 0.004"/>
-            </geometry>
+			<geometry>
+				<box size="0.001 0.001 0.001"/>
+			</geometry>
+			<!-- <material name="red"/> -->
 		</visual>
+		<collision>
+			<origin rpy="0 0 0" xyz="0 0 0"/>
+			<geometry>
+				<box size=".001 .001 .001"/>
+			</geometry>
+		</collision>
 		</link>
-    <xacro:leg prefix="FR" mirror="-1" mirror_dae="False" front_hind="1" front_hind_dae="True" simulator="${simulator}" robot_type="${robot_type}">
-        <origin rpy="0 0 0" xyz="${leg_offset_x} ${-leg_offset_y} 0"/>
-    </xacro:leg>
-    <xacro:leg prefix="FL" mirror="1" mirror_dae="True" front_hind="1" front_hind_dae="True" simulator="${simulator}" robot_type="${robot_type}">
-        <origin rpy="0 0 0" xyz="${leg_offset_x} ${leg_offset_y} 0"/>
-    </xacro:leg>
-    <xacro:leg prefix="RR" mirror="-1" mirror_dae="False" front_hind="-1" front_hind_dae="False" simulator="${simulator}" robot_type="${robot_type}">
-        <origin rpy="0 0 0" xyz="${-leg_offset_x} ${-leg_offset_y} 0"/>
-    </xacro:leg>
-    <xacro:leg prefix="RL" mirror="1" mirror_dae="True" front_hind="-1" front_hind_dae="False" simulator="${simulator}" robot_type="${robot_type}">
-        <origin rpy="0 0 0" xyz="${-leg_offset_x} ${leg_offset_y} 0"/>
-    </xacro:leg>
+		<!--
+	<joint name="load_joint" type="fixed">
+			<parent link="trunk"/>
+			<child link="load_link"/>
+			<origin rpy="0 0 0" xyz="0 0 0"/>
+	</joint>
+	<link name="load_link">
+			<inertial>
+					<mass value="5"/>
+					<origin rpy="0 0 0" xyz="0 0 0"/>
+					<inertia ixx="0.01" ixy="0" ixz="0" iyy="0.01" iyz="0" izz="0.01"/>
+			</inertial>
+			<visual>
+					<origin rpy="0 0 0" xyz="0 0 0.2"/>
+					<geometry>
+							<box size="0.5 0.3 0.2"/>
+					</geometry>
+			</visual>
+			<collision>
+					<origin rpy="0 0 0" xyz="0 0 0"/>
+					<geometry>
+							<box size=".001 .001 .001"/>
+					</geometry>
+			</collision>
+	</link>
+-->
+	<xacro:leg name="FR" mirror="-1" mirror_dae="False" front_hind="1" front_hind_dae="True"/>
+	<xacro:leg name="FL" mirror="1" mirror_dae="True" front_hind="1" front_hind_dae="True"/>
+	<xacro:leg name="RR" mirror="-1" mirror_dae="False" front_hind="-1" front_hind_dae="False"/>
+	<xacro:leg name="RL" mirror="1" mirror_dae="True" front_hind="-1" front_hind_dae="False"/>
 </robot>
