Commit message: update arcdog_adjustable leg xml xacro and urdf model

File: robot_description/arcdog_adjustable_leg_description/urdf/arcdog_adjustable_leg_test.urdf (robot description, URDF)
Before this commit: robot robot, 23 links, 22 joints
Links:
- link FL_box: geometry collision box size=0.1691 0.02 0.05; visual mesh filename=package://arcdog_adjustable_leg_description/assets/adjustab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 scale=1 1 1
- link FL_calf: geometry collision box size=0.193 0.02 0.05; visual mesh filename=package://arcdog_adjustable_leg_description/meshes/calf.stl scale=1 1 1
- link FL_hip: mass 1.162 -> 1.108; geometry collision cylinder length=0.0834 radius=0.0495; visual mesh filename=package://arcdog_adjustable_leg_description/meshes/hip.stl scale=1 1 1
- link FL_thigh: mass 1.528 -> 1.636; geometry collision box size=0.245 0.04 0.06797; visual mesh filename=package://arcdog_adjustable_leg_description/meshes/thigh.stl scale=1 1 1
- link FR_box: geometry collision box size=0.1691 0.02 0.05; visual mesh filename=package://arcdog_adjustable_leg_description/assets/adjustab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 scale=1 1 1
- link FR_calf: geometry collision box size=0.193 0.02 0.05; visual mesh filename=package://arcdog_adjustable_leg_description/meshes/calf.stl scale=1 1 1
- link FR_hip: mass 1.162 -> 1.108; geometry collision cylinder length=0.0834 radius=0.0495; visual mesh filename=package://arcdog_adjustable_leg_description/meshes/hip.stl scale=1 1 1
- link FR_thigh: mass 1.528 -> 1.636; geometry collision box size=0.245 0.04 0.06797; visual mesh filename=package://arcdog_adjustable_leg_description/meshes/thigh_mi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 scale=1 1 1
- link RL_box: geometry collision box size=0.1691 0.02 0.05; visual mesh filename=package://arcdog_adjustable_leg_description/assets/adjustab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 scale=1 1 1
- link RL_calf: geometry collision box size=0.193 0.02 0.05; visual mesh filename=package://arcdog_adjustable_leg_description/meshes/calf.stl scale=1 1 1
- link RL_hip: mass 1.162 -> 1.108; geometry collision cylinder length=0.0834 radius=0.0495; visual mesh filename=package://arcdog_adjustable_leg_description/meshes/hip.stl scale=1 1 1
- link RL_thigh: mass 1.528 -> 1.636; geometry collision box size=0.245 0.04 0.06797; visual mesh filename=package://arcdog_adjustable_leg_description/meshes/thigh.stl scale=1 1 1
- link RR_box: geometry collision box size=0.1691 0.02 0.05; visual mesh filename=package://arcdog_adjustable_leg_description/assets/adjustab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 scale=1 1 1
- link RR_calf: geometry collision box size=0.193 0.02 0.05; visual mesh filename=package://arcdog_adjustable_leg_description/meshes/calf.stl scale=1 1 1
- link RR_hip: mass 1.162 -> 1.108; geometry collision cylinder length=0.0834 radius=0.0495; visual mesh filename=package://arcdog_adjustable_leg_description/meshes/hip.stl scale=1 1 1
- link RR_thigh: mass 1.528 -> 1.636; geometry collision box size=0.245 0.04 0.06797; visual mesh filename=package://arcdog_adjustable_leg_description/meshes/thigh_mi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 scale=1 1 1
- link trunk: mass 7.021 -> 5.742; geometry collision box size=0.361 0.121 0.114; visual mesh filename=file:///home/lxq/colcon_ws/install/arcdog_adjustable_leg_de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 scale=1 1 1
Joints:
- joint FL_box_joint: limit lower=0 upper=0.193 effort=50 velocity=50 -> lower=0 upper=-0.193 effort=50 velocity=50
- joint FL_calf_joint: origin xyz=0 0 -0.2445 rpy=0 0 0 -> xyz=0 0 -0.245 rpy=0 0 0
- joint FL_hip_joint: origin xyz=0.269 0.0605 0 rpy=0 0 0 -> xyz=0.2515 0.0605 0 rpy=0 0 0
- joint FL_thigh_joint: origin xyz=0 0.09426 0 rpy=0 0 0 -> xyz=0 0.11475 0 rpy=0 0 0
- joint FR_box_joint: limit lower=0 upper=0.193 effort=50 velocity=50 -> lower=0 upper=-0.193 effort=50 velocity=50
- joint FR_calf_joint: origin xyz=0 0 -0.2445 rpy=0 0 0 -> xyz=0 0 -0.245 rpy=0 0 0
- joint FR_hip_joint: origin xyz=0.269 -0.0605 0 rpy=0 0 0 -> xyz=0.2515 -0.0605 0 rpy=0 0 0
- joint FR_thigh_joint: origin xyz=0 -0.09426 0 rpy=0 0 0 -> xyz=0 -0.11475 0 rpy=0 0 0
- joint RL_box_joint: limit lower=0 upper=0.193 effort=50 velocity=50 -> lower=0 upper=-0.193 effort=50 velocity=50
- joint RL_calf_joint: origin xyz=0 0 -0.2445 rpy=0 0 0 -> xyz=0 0 -0.245 rpy=0 0 0
- joint RL_hip_joint: origin xyz=-0.269 0.0605 0 rpy=0 0 0 -> xyz=-0.2515 0.0605 0 rpy=0 0 0
- joint RL_thigh_joint: origin xyz=0 0.09426 0 rpy=0 0 0 -> xyz=0 0.11475 0 rpy=0 0 0
- joint RR_box_joint: limit lower=0 upper=0.193 effort=50 velocity=50 -> lower=0 upper=-0.193 effort=50 velocity=50
- joint RR_calf_joint: origin xyz=0 0 -0.2445 rpy=0 0 0 -> xyz=0 0 -0.245 rpy=0 0 0
- joint RR_hip_joint: origin xyz=-0.269 -0.0605 0 rpy=0 0 0 -> xyz=-0.2515 -0.0605 0 rpy=0 0 0
- joint RR_thigh_joint: origin xyz=0 -0.09426 0 rpy=0 0 0 -> xyz=0 -0.11475 0 rpy=0 0 0

File: robot_description/arcdog_adjustable_leg_description/xacro/const.xacro (robot description, xacro)
@@ -1,4 +1,4 @@
 <?xml version="1.0"?>
-<robot xmlns:xacro="http://www.ros.org/wiki/xacro">
+<robot xmlns:xacro="http://www.ros.org/wiki/xacro" name="arcdog_adjustable_leg_description">
 	<!-- Constants for robot dimensions -->
 	<xacro:property name="PI" value="3.1415926535897931"/>
@@ -6,89 +6,85 @@
 	<!-- simplified collision value -->
     <xacro:property name="trunk_width" value="0.121"/>
-    <xacro:property name="trunk_length" value="0.548"/>
-    <xacro:property name="trunk_height" value="0.116"/>
-    <xacro:property name="hip_radius" value="0.041"/>
-    <xacro:property name="hip_length" value=" 0.1095"/>
-    <xacro:property name="thigh_shoulder_radius" value="0.044"/>
-    <xacro:property name="thigh_shoulder_length" value="0.0985"/>
-    <xacro:property name="thigh_shoulder_y_offset" value="0.0"/> //TODO
-    <xacro:property name="thigh_width" value="0.088"/>
+    <xacro:property name="trunk_length" value="0.361"/>
+    <xacro:property name="trunk_height" value="0.114"/>
+    <xacro:property name="hip_radius" value="0.0495"/>
+    <xacro:property name="hip_length" value=" 0.0834"/>
+    <xacro:property name="thigh_shoulder_radius" value="0.0495"/>
+    <xacro:property name="thigh_shoulder_length" value="0.03826"/>
+    <xacro:property name="thigh_width" value="0.040"/>
     <xacro:property name="thigh_height" value="0.06797"/>
-    <xacro:property name="thigh_x_offset" value="0.000"/> //TODO
     <xacro:property name="calf_width" value="0.02"/>
     <xacro:property name="calf_height" value="0.05"/>
-    <xacro:property name="calf_x_offset" value="0.000"/> //TODO
-	<xacro:property name="foot_radius" value="0.0265"/>
-	<xacro:property name="stick_radius" value="0.01"/>
-	<xacro:property name="stick_length" value="0.2"/>
+    <xacro:property name="foot_radius" value="0.0265"/>
+    <xacro:property name="stick_radius" value="?"/> //TODO
+	<xacro:property name="stick_length" value="?"/> //TODO
     <!-- kinematic value -->
-    <xacro:property name="thigh_offset" value="0.09426"/>
-    <xacro:property name="thigh_length" value="0.2445"/>
+    <xacro:property name="thigh_offset" value="0.11475"/>
+    <xacro:property name="thigh_length" value="0.245"/>
     <xacro:property name="calf_length" value="0.1930"/>
     <!-- leg offset from trunk center value -->
-    <xacro:property name="leg_offset_x" value="0.269"/>
+    <xacro:property name="leg_offset_x" value="0.2515"/>
     <xacro:property name="leg_offset_y" value="0.0605"/>
     <xacro:property name="trunk_offset_z" value="0.01675"/> //TODO
-    <xacro:property name="hip_offset" value="0.0001"/> //TODO
+    <xacro:property name="hip_offset" value="0.11475"/> //go2 special point, puting hip collision model at thigh position
 	<!-- offset of link locations (left front) -->
-	<xacro:property name="hip_offset_x" value="0.1934"/>
-	<xacro:property name="hip_offset_y" value="0.0465"/>
-	<xacro:property name="hip_offset_z" value="0.0"/>
-    <!-- kinematic value -->
-    <!-- <xacro:property name="thigh_offset" value="0.1095"/>
-    <xacro:property name="thigh_length" value="0.2445"/>
-    <xacro:property name="calf_length" value="0.23704"/>  -->
-	<xacro:property name="calf_offset_x" value="0.0"/>
-	<xacro:property name="calf_offset_y" value="0.0"/>
-	<xacro:property name="calf_offset_z" value="-0.213"/>
+    <xacro:property name="hip_offset_x" value="?"/> //TODO
+	<xacro:property name="hip_offset_y" value="?"/> //TODO
+	<xacro:property name="hip_offset_z" value="?"/> //TODO
+	<xacro:property name="thigh_offset_x" value="?"/> //TODO
+	<xacro:property name="thigh_offset_y" value="?"/> //TODO
+	<xacro:property name="thigh_offset_z" value="?"/> //TODO
+	<xacro:property name="calf_offset_x" value="?"/> //TODO
+	<xacro:property name="calf_offset_y" value="?"/> //TODO
+	<xacro:property name="calf_offset_z" value="?"/> //TODO
     <!-- joint limits -->
     <xacro:property name="damping" value="0.05"/>
     <xacro:property name="friction" value="0.01"/>
-    <xacro:property name="hip_max" value="${70*pi/180.0}"/>
-    <xacro:property name="hip_min" value="${-70*pi/180.0}"/>
+    <xacro:property name="hip_position_max" value="${70*pi/180.0}"/>
+    <xacro:property name="hip_position_min" value="${-70*pi/180.0}"/>
     <xacro:property name="hip_velocity_max" value="20"/>
     <xacro:property name="hip_torque_max" value="35.278"/>
-    <xacro:property name="thigh_max" value="3.4907"/>
-    <xacro:property name="thigh_min" value="-1.5708"/>
+    <xacro:property name="thigh_position_max" value="3.4907"/>
+    <xacro:property name="thigh_position_min" value="-1.5708"/>
     <xacro:property name="thigh_velocity_max" value="20"/>
     <xacro:property name="thigh_torque_max" value="35.278"/>
-    <xacro:property name="calf_max" value="${-37*pi/180.0}"/>
-    <xacro:property name="calf_min" value="${-159*pi/180.0}"/>
+    <xacro:property name="calf_position_max" value="${-37*pi/180.0}"/>
+    <xacro:property name="calf_position_min" value="${-159*pi/180.0}"/>
     <xacro:property name="calf_velocity_max" value="15.89"/>
     <xacro:property name="calf_torque_max" value="44.4"/>
     <!-- dynamics inertial value    total 22.0kg-->
     <!-- trunk -->
-    <xacro:property name="trunk_mass" value="7.021"/>
-    <xacro:property name="trunk_com_x" value="0.00575"/>
-    <xacro:property name="trunk_com_y" value="0.00126"/>
-    <xacro:property name="trunk_com_z" value="-0.00469"/>
-    <xacro:property name="trunk_ixx" value="0.03769023916"/>
-    <xacro:property name="trunk_ixy" value="0.00001433761"/>
-    <xacro:property name="trunk_ixz" value="0.00051349975"/>
-    <xacro:property name="trunk_iyy" value="0.05008788073"/>
-    <xacro:property name="trunk_iyz" value="0.00015851764"/>
-    <xacro:property name="trunk_izz" value="0.07146322696"/>
+    <xacro:property name="trunk_mass" value="5.742"/>
+    <xacro:property name="trunk_com_x" value="-0.002250"/>
+    <xacro:property name="trunk_com_y" value="0.000116"/>
+    <xacro:property name="trunk_com_z" value="-0.001452"/>
+    <xacro:property name="trunk_ixx" value="0.037914363"/>
+    <xacro:property name="trunk_ixy" value="0.000098848"/>
+    <xacro:property name="trunk_ixz" value="-0.000073338"/>
+    <xacro:property name="trunk_iyy" value="0.119267297"/>
+    <xacro:property name="trunk_iyz" value="0.000013463"/>
+    <xacro:property name="trunk_izz" value="0.142804844"/>
     <!-- hip (left front) -->
-    <xacro:property name="hip_mass" value="1.162"/>
-    <xacro:property name="hip_com_x" value="-0.00758"/>
-    <xacro:property name="hip_com_y" value="-0.00359"/>
-    <xacro:property name="hip_com_z" value="-0.00029"/>
-    <xacro:property name="hip_ixx" value="0.00095157705"/>
-    <xacro:property name="hip_ixy" value="0.00001109670"/>
-    <xacro:property name="hip_ixz" value="-0.00000266665"/>
-    <xacro:property name="hip_iyy" value="0.00159323348"/>
-    <xacro:property name="hip_iyz" value="-0.00001267180"/>
-    <xacro:property name="hip_izz" value="0.00125451931"/>
+    <xacro:property name="hip_mass" value="1.108"/>
+    <xacro:property name="hip_com_x" value="-0.0082"/>
+    <xacro:property name="hip_com_y" value="0.000984"/>
+    <xacro:property name="hip_com_z" value="0.000162"/>
+    <xacro:property name="hip_ixx" value="0.000972670"/>
+    <xacro:property name="hip_ixy" value="0.000004550"/>
+    <xacro:property name="hip_ixz" value="0.000000139"/>
+    <xacro:property name="hip_iyy" value="0.001754403"/>
+    <xacro:property name="hip_iyz" value="0.000001705"/>
+    <xacro:property name="hip_izz" value="0.001311138"/>
     <!-- thigh -->
-    <xacro:property name="thigh_mass" value="1.528"/>
-    <xacro:property name="thigh_com_x" value="0.00033"/>
-    <xacro:property name="thigh_com_y" value="0.03334"/>
-    <xacro:property name="thigh_com_z" value="-0.02983"/>
-    <xacro:property name="thigh_ixx" value="0.00884041519"/>
-    <xacro:property name="thigh_ixy" value="-0.00003381758"/>
-    <xacro:property name="thigh_ixz" value="-0.00005336860"/>
-    <xacro:property name="thigh_iyy" value="0.00784145389"/>
-    <xacro:property name="thigh_iyz" value="0.00128350622"/>
-    <xacro:property name="thigh_izz" value="0.00260045020"/>
+    <xacro:property name="thigh_mass" value="1.636"/>
+    <xacro:property name="thigh_com_x" value="-0.004484"/>
+    <xacro:property name="thigh_com_y" value="-0.033084"/>
+    <xacro:property name="thigh_com_z" value="-0.030728"/>
+    <xacro:property name="thigh_ixx" value="0.009596889"/>
+    <xacro:property name="thigh_ixy" value="-0.000241414"/>
+    <xacro:property name="thigh_ixz" value="0.000789459"/>
+    <xacro:property name="thigh_iyy" value="0.009201469"/>
+    <xacro:property name="thigh_iyz" value="-0.001676085"/>
+    <xacro:property name="thigh_izz" value="0.002385568"/>
     <!-- calf -->
     <xacro:property name="calf_mass" value="0.132"/>
