Commit message: update arcdog_adjustable leg xml xacro and urdf model

File: robot_description/arcdog_adjustable_leg_description/xacro/leg.xacro (robot description, xacro)
@@ -2,57 +2,32 @@
 <robot xmlns:xacro="http://www.ros.org/wiki/xacro">
     <xacro:include filename="$(find arcdog_adjustable_leg_description)/xacro/transmission.xacro"/>
-    <xacro:macro name="leg" params="prefix mirror mirror_dae front_hind front_hind_dae simulator robot_type *origin">
-        <xacro:if value="${simulator == 'ocs2'}">
-            <joint name="${prefix}_HAA" type="revolute">
-                <xacro:insert_block name="origin"/>
-                <parent link="trunk"/>
-                <child link="${prefix}_hip"/>
+    <xacro:macro name="leg" params="name mirror mirror_dae front_hind front_hind_dae">
+        <joint name="${name}_hip_joint" type="revolute">
+			<xacro:if value="${(mirror_dae == False) and (front_hind_dae == True)}">
+				<origin rpy="0 0 0" xyz="${leg_offset_x} ${-leg_offset_y} 0"/>
+			</xacro:if>
+			<xacro:if value="${(mirror_dae == True) and (front_hind_dae == True)}">
+				<origin rpy="0 0 0" xyz="${leg_offset_x} ${leg_offset_y} 0"/>
+			</xacro:if>
+			<xacro:if value="${(mirror_dae == False) and (front_hind_dae == False)}">
+				<origin rpy="0 0 0" xyz="${-leg_offset_x} ${-leg_offset_y} 0"/>
+			</xacro:if>
+			<xacro:if value="${(mirror_dae == True) and (front_hind_dae == False)}">
+				<origin rpy="0 0 0" xyz="${-leg_offset_x} ${leg_offset_y} 0"/>
+			</xacro:if>
+			<parent link="trunk"/>
+			<child link="${name}_hip"/>
                 <axis xyz="1 0 0"/>
                 <dynamics damping="${damping}" friction="${friction}"/>
-                <xacro:if value="${(mirror_dae == True)}">
-                    <limit effort="${hip_torque_max}" velocity="${hip_velocity_max}" lower="${hip_min}"
-                        upper="${hip_max}"/>
-                </xacro:if>
-                <xacro:if value="${(mirror_dae == False)}">
-                    <limit effort="${hip_torque_max}" velocity="${hip_velocity_max}" lower="${-hip_max}"
-                        upper="${-hip_min}"/>
+			<xacro:if value="${(mirror_dae == True)}">
+				<limit effort="${hip_torque_max}" velocity="${hip_velocity_max}" lower="${hip_position_min}"
+							 upper="${hip_position_max}"/>
+			</xacro:if>
+			<xacro:if value="${(mirror_dae == False)}">
+				<limit effort="${hip_torque_max}" velocity="${hip_velocity_max}" lower="${-hip_position_max}"
+							 upper="${-hip_position_min}"/>
                 </xacro:if>
             </joint>
-        </xacro:if>
-        <xacro:if value="${simulator == 'test'}">
-            <joint name="${prefix}_hip_joint" type="revolute">
-                <xacro:insert_block name="origin"/>
-                <parent link="trunk"/>
-                <child link="${prefix}_hip"/>
-                <axis xyz="1 0 0"/>
-                <dynamics damping="${damping}" friction="${friction}"/>
-                <xacro:if value="${(mirror_dae == True)}">
-                    <limit effort="${hip_torque_max}" velocity="${hip_velocity_max}" lower="${hip_min}"
-                        upper="${hip_max}"/>
-                </xacro:if>
-                <xacro:if value="${(mirror_dae == False)}">
-                    <limit effort="${hip_torque_max}" velocity="${hip_velocity_max}" lower="${-hip_max}"
-                        upper="${-hip_min}"/>
-                </xacro:if>
-            </joint>
-        </xacro:if>
-        <xacro:if value="${simulator == 'mujoco'}">
-            <joint name="${prefix}_hip_joint" type="revolute">
-                <xacro:insert_block name="origin"/>
-                <parent link="trunk"/>
-                <child link="${prefix}_hip"/>
-                <axis xyz="1 0 0"/>
-                <dynamics damping="${damping}" friction="${friction}"/>
-                <xacro:if value="${(mirror_dae == True)}">
-                    <limit effort="${hip_torque_max}" velocity="${hip_velocity_max}" lower="${hip_min}"
-                        upper="${hip_max}"/>
-                </xacro:if>
-                <xacro:if value="${(mirror_dae == False)}">
-                    <limit effort="${hip_torque_max}" velocity="${hip_velocity_max}" lower="${-hip_max}"
-                        upper="${-hip_min}"/>
-                </xacro:if>
-            </joint>
-        </xacro:if>
-        <link name="${prefix}_hip">
+        <link name="${name}_hip">
             <visual>
                 <xacro:if value="${(mirror_dae == True) and (front_hind_dae == True)}">
@@ -60,20 +35,19 @@
                 </xacro:if>
                 <xacro:if value="${(mirror_dae == False) and (front_hind_dae == True)}">
-                    <origin rpy="${pi} 0 0" xyz="0 0 0"/>
+                    <origin rpy="${PI} 0 0" xyz="0 0 0"/>
                 </xacro:if>
                 <xacro:if value="${(mirror_dae == True) and (front_hind_dae == False)}">
-                    <origin rpy="0 ${pi} 0" xyz="0 0 0"/>
+                    <origin rpy="0 ${PI} 0" xyz="0 0 0"/>
                 </xacro:if>
                 <xacro:if value="${(mirror_dae == False) and (front_hind_dae == False)}">
-                    <origin rpy="${pi} ${pi} 0" xyz="0 0 0"/>
+                    <origin rpy="${PI} ${PI} 0" xyz="0 0 0"/>
                 </xacro:if>
                 <geometry>
-                    <mesh filename="package://arcdog_adjustable_leg_description/assets/hip.stl"
+                    <mesh filename="package://arcdog_adjustable_leg_description/meshes/hip.stl"
                           scale="1 1 1"/>
                 </geometry>
-                <material name="orange"/>
             </visual>
             <collision>
-                <origin rpy="${pi/2.0} 0 0" xyz="0 0 0"/>
+                <origin rpy="${PI/2.0} 0 0" xyz="0 ${hip_offset*mirror} 0"/>
                 <geometry>
                     <cylinder length="${hip_length}" radius="${hip_radius}"/>
@@ -89,62 +63,29 @@
             </inertial>
         </link>
-        <xacro:if value="${simulator == 'ocs2'}">
-            <joint name="${prefix}_HFE" type="revolute">
-                <origin rpy="0 0 0" xyz="0 ${thigh_offset*mirror} 0"/>
-                <parent link="${prefix}_hip"/>
-                <child link="${prefix}_thigh"/>
-                <axis xyz="0 1 0"/>
-                <dynamics damping="${damping}" friction="${friction}"/>
-                <limit effort="${thigh_torque_max}" velocity="${thigh_velocity_max}" lower="${thigh_min}"
-                    upper="${thigh_max}"/>
-            </joint>
-        </xacro:if>
-        <xacro:if value="${simulator == 'test'}">
-            <joint name="${prefix}_thigh_joint" type="revolute">
-                <origin rpy="0 0 0" xyz="0 ${thigh_offset*mirror} 0"/>
-                <parent link="${prefix}_hip"/>
-                <child link="${prefix}_thigh"/>
-                <axis xyz="0 1 0"/>
-                <dynamics damping="${damping}" friction="${friction}"/>
-                <limit effort="${thigh_torque_max}" velocity="${thigh_velocity_max}" lower="${thigh_min}"
-                    upper="${thigh_max}"/>
-            </joint>
-        </xacro:if>
-        <xacro:if value="${simulator == 'mujoco'}">
-            <joint name="${prefix}_thigh_joint" type="revolute">
-                <origin rpy="0 0 0" xyz="0 ${thigh_offset*mirror} 0"/>
-                <parent link="${prefix}_hip"/>
-                <child link="${prefix}_thigh"/>
-                <axis xyz="0 1 0"/>
-                <dynamics damping="${damping}" friction="${friction}"/>
-                <limit effort="${thigh_torque_max}" velocity="${thigh_velocity_max}" lower="${thigh_min}"
-                    upper="${thigh_max}"/>
-            </joint>
-        </xacro:if>
-        <link name="${prefix}_thigh">
+		<joint name="${name}_thigh_joint" type="revolute">
+			<origin rpy="0 0 0" xyz="0 ${thigh_offset*mirror} 0"/>
+			<parent link="${name}_hip"/>
+			<child link="${name}_thigh"/>
+			<axis xyz="0 1 0"/>
+			<dynamics damping="${damping}" friction="${friction}"/>
+			<limit effort="${thigh_torque_max}" velocity="${thigh_velocity_max}" lower="${thigh_position_min}"
+						 upper="${thigh_position_max}"/>
+		</joint>
+        <link name="${name}_thigh">
             <visual>
                 <origin rpy="0 0 0" xyz="0 0 0"/>
                 <geometry>
                     <xacro:if value="${mirror_dae == True}">
-                        <mesh filename="package://arcdog_adjustable_leg_description/assets/thigh.stl"
-                              scale="1 1 1"/>
+                        <mesh filename="package://arcdog_adjustable_leg_description/meshes/thigh.stl" scale="1 1 1"/>
                     </xacro:if>
                     <xacro:if value="${mirror_dae == False}">
-                        <mesh filename="package://arcdog_adjustable_leg_description/assets/thigh_mirror.stl"
-                              scale="1 1 1"/>
+                        <mesh filename="package://arcdog_adjustable_leg_description/meshes/thigh_mirror.stl" scale="1 1 1"/>
                     </xacro:if>
                 </geometry>
-                <material name="orange"/>
             </visual>
             <collision>
-                <origin rpy="0 ${pi/2.0+0.1} 0" xyz="${thigh_x_offset} 0 ${-thigh_length/2.0}"/>
+                <origin rpy="0 ${PI/2.0} 0" xyz="0 0 ${-thigh_length/2.0}"/>
                 <geometry>
                     <box size="${thigh_length} ${thigh_width} ${thigh_height}"/>
-                </geometry>
-            </collision>
-            <collision>
-                <origin rpy="${pi/2.0} 0 0" xyz="0 ${mirror*thigh_shoulder_y_offset} 0"/>
-                <geometry>
-                    <cylinder length="${thigh_shoulder_length}" radius="${thigh_shoulder_radius}"/>
                 </geometry>
             </collision>
@@ -158,45 +99,22 @@
             </inertial>
         </link>
-        <xacro:if value="${simulator == 'ocs2'}">
-            <joint name="${prefix}_KFE" type="revolute">
-                <origin rpy="0 0 0" xyz="0 0 ${-thigh_length}"/>
-                <parent link="${prefix}_thigh"/>
-                <child link="${prefix}_calf"/>
-                <axis xyz="0 1 0"/>
-                <dynamics damping="${damping}" friction="${friction}"/>
-                <limit effort="${calf_torque_max}" velocity="${calf_velocity_max}" lower="${calf_min}" upper="${calf_max}"/>
-            </joint>
-        </xacro:if>
-        <xacro:if value="${simulator == 'test'}">
-            <joint name="${prefix}_calf_joint" type="revolute">
-                <origin rpy="0 0 0" xyz="0 0 ${-thigh_length}"/>
-                <parent link="${prefix}_thigh"/>
-                <child link="${prefix}_calf"/>
-                <axis xyz="0 1 0"/>
-                <dynamics damping="${damping}" friction="${friction}"/>
-                <limit effort="${calf_torque_max}" velocity="${calf_velocity_max}" lower="${calf_min}" upper="${calf_max}"/>
-            </joint>
-        </xacro:if>
-        <xacro:if value="${simulator == 'mujoco'}">
-            <joint name="${prefix}_calf_joint" type="revolute">
-                <origin rpy="0 0 0" xyz="0 0 ${-thigh_length}"/>
-                <parent link="${prefix}_thigh"/>
-                <child link="${prefix}_calf"/>
-                <axis xyz="0 1 0"/>
-                <dynamics damping="${damping}" friction="${friction}"/>
-                <limit effort="${calf_torque_max}" velocity="${calf_velocity_max}" lower="${calf_min}" upper="${calf_max}"/>
-            </joint>
-        </xacro:if>
-        <link name="${prefix}_calf">
+		<joint name="${name}_calf_joint" type="revolute">
+			<origin rpy="0 0 0" xyz="0 0 ${-thigh_length}"/>
+			<parent link="${name}_thigh"/>
+			<child link="${name}_calf"/>
+			<axis xyz="0 1 0"/>
+			<dynamics damping="${damping}" friction="${friction}"/>
+			<limit effort="${calf_torque_max}" velocity="${calf_velocity_max}" lower="${calf_position_min}"
+						 upper="${calf_position_max}"/>
+		</joint>
+        <link name="${name}_calf">
             <visual>
                 <origin rpy="0 0 0" xyz="0 0 0"/>
                 <geometry>
-                    <mesh filename="package://arcdog_adjustable_leg_description/assets/calf.stl"
-                          scale="1 1 1"/>
+                    <mesh filename="package://arcdog_adjustable_leg_description/meshes/calf.stl" scale="1 1 1"/>
                 </geometry>
-                <material name="orange"/>
             </visual>
             <collision>
-                <origin rpy="0 ${pi/2.0} 0" xyz="${calf_x_offset} 0 ${-calf_length/2.0}"/>
+                <origin rpy="0 ${PI/2.0} 0" xyz="0 0 ${-calf_length/2.0}"/>
                 <geometry>
                     <box size="${calf_length} ${calf_width} ${calf_height}"/>
@@ -213,5 +131,5 @@
         </link>
         <!-- 在 calf 和 foot 之间添加 box link -->
-        <link name="${prefix}_box">
+        <link name="${name}_box">
             <visual>
                 <origin rpy="0 0 0" xyz="0 0 0"/>
@@ -223,5 +141,5 @@
             </visual>
             <collision>
-                <origin rpy="0 0 0" xyz="0 0 0"/>
+                <origin rpy="0 ${PI/2.0} 0" xyz="0 0 ${-box_length/2.0}"/>
                 <geometry>
                     <box size="${box_length} ${box_width} ${box_height}"/>
@@ -229,5 +147,5 @@
             </collision>
             <inertial>
-                <origin rpy="0 0 0" xyz="0 0 0"/>
+                <origin rpy="0 0 0" xyz="0 0 ${-box_length/2.0}"/>
                 <mass value="${box_mass}"/> <!-- 定义 box 的质量 -->
                 <inertia
@@ -238,18 +156,18 @@
         </link>
         <!-- 添加 prismatic joint -->
-        <joint name="${prefix}_box_joint" type="prismatic">
+        <joint name="${name}_box_joint" type="prismatic">
             <origin rpy="0 0 0" xyz="0 0 ${-calf_length}"/> <!-- 根据 calf 的长度调整位置 -->
-            <parent link="${prefix}_calf"/>
-            <child link="${prefix}_box"/>
+            <parent link="${name}_calf"/>
+            <child link="${name}_box"/>
             <axis xyz="0 0 1"/> <!-- 定义滑动轴 -->
             <dynamics damping="${damping}" friction="${friction}"/>
             <limit effort="${box_effort_max}" velocity="${box_velocity_max}" lower="0" upper="${-calf_length}"/> <!-- 定义限制条件 -->
         </joint>
-        <joint name="${prefix}_foot_fixed" type="fixed" dont_collapse="true">
+        <joint name="${name}_foot_fixed" type="fixed">
             <origin rpy="0 0 0" xyz="0 0 ${-box_length}"/> <!-- 连接到 box 的底部 -->
-            <parent link="${prefix}_box"/>
-            <child link="${prefix}_foot"/>
+            <parent link="${name}_box"/>
+            <child link="${name}_foot"/>
         </joint>
-        <link name="${prefix}_foot">
+        <link name="${name}_foot">
             <visual>
                 <origin rpy="0 0 0" xyz="0 0 0"/>
@@ -257,5 +175,4 @@
                     <sphere radius="${foot_radius-0.01}"/>
                 </geometry>
-                <material name="orange"/>
             </visual>
             <collision>
@@ -273,44 +190,5 @@
             </inertial>
         </link>
-        <gazebo reference="${prefix}_foot_fixed">
-            <disableFixedJointLumping>true</disableFixedJointLumping>
-        </gazebo>
-        <gazebo reference="${prefix}_hip">
-            <mu1>0.2</mu1>
-            <mu2>0.2</mu2>
-            <material>Gazebo/DarkGrey</material>
-        </gazebo>
-        <gazebo reference="${prefix}_thigh">
-            <mu1>0.2</mu1>
-            <mu2>0.2</mu2>
-            <self_collide>0</self_collide>
-            <material>Gazebo/DarkGrey</material>
-            <kp value="1000000.0"/>
-            <kd value="100.0"/>
-        </gazebo>
-        <gazebo reference="${prefix}_calf">
-            <mu1>0.6</mu1>
-            <mu2>0.6</mu2>
-            <self_collide>1</self_collide>
-        </gazebo>
-        <gazebo reference="${prefix}_box">
-            <mu1>0.4</mu1>  <!-- 根据需要设置静摩擦系数 -->
-            <mu2>0.4</mu2>  <!-- 根据需要设置动摩擦系数 -->
-            <self_collide>0</self_collide>
-            <material>Gazebo/DarkGrey</material>  <!-- 可根据需要更改材料 -->
-        </gazebo>
-        <gazebo reference="${prefix}_FOOT">
-            <mu1>0.6</mu1>
-            <mu2>0.6</mu2>
-            <self_collide>1</self_collide>
-            <material>Gazebo/DarkGrey</material>
-            <kp value="1000000.0"/>
-            <kd value="100.0"/>
-        </gazebo>
-        <gazebo reference="${prefix}_box_joint">
-            <mu1>0.4</mu1>  <!-- 设置滑动关节的摩擦系数 -->
-            <mu2>0.4</mu2>
-        </gazebo>
-        <xacro:leg_transmission name="${prefix}"/>
+        <xacro:leg_transmission name="${name}"/>
     </xacro:macro>
 </robot>

File: robot_description/arcdog_adjustable_leg_description/xacro/real_robot.xacro (robot description, xacro)
@@ -1,24 +1,20 @@
 <?xml version="1.0"?>
 <robot name="arcdog" xmlns:xacro="http://www.ros.org/wiki/xacro">
-	<xacro:arg name="DEBUG" default="false"/>
+	<xacro:arg name="DEBUG" default="true"/>
 	<xacro:arg name="GAZEBO" default="false"/>
 	<xacro:arg name="CLASSIC" default="false"/>
-    <xacro:arg name="robot_type" default="arcdog"/>
-    <xacro:property name="robot_type" value="$(arg robot_type)"/>
-	<xacro:arg name="simulator" default="test"/>
-    <xacro:property name="simulator" value="$(arg simulator)"/>
-	<xacro:include filename="$(find arcdog_description)/xacro/const.xacro"/>
-	<xacro:include filename="$(find arcdog_description)/xacro/materials.xacro"/>
-	<xacro:include filename="$(find arcdog_description)/xacro/leg.xacro"/>
+	<xacro:include filename="$(find arcdog_adjustable_leg_description)/xacro/const.xacro"/>
+	<xacro:include filename="$(find arcdog_adjustable_leg_description)/xacro/materials.xacro"/>
+	<xacro:include filename="$(find arcdog_adjustable_leg_description)/xacro/leg.xacro"/>
 	<xacro:if value="$(arg GAZEBO)">
 		<xacro:if value="$(arg CLASSIC)">
-			<xacro:include filename="$(find arcdog_description)/xacro/gazebo_classic.xacro"/>
+			<xacro:include filename="$(find arcdog_adjustable_leg_description)/xacro/gazebo_classic.xacro"/>
 		</xacro:if>
 		<xacro:unless value="$(arg CLASSIC)">
-			<xacro:include filename="$(find arcdog_description)/xacro/gazebo.xacro"/>
+			<xacro:include filename="$(find arcdog_adjustable_leg_description)/xacro/gazebo.xacro"/>
 		</xacro:unless>
 	</xacro:if>
 	<xacro:unless value="$(arg GAZEBO)">
-		<xacro:include filename="$(find arcdog_description)/xacro/ros2_control_real_robot.xacro"/>
+		<xacro:include filename="$(find arcdog_adjustable_leg_description)/xacro/ros2_control_real_robot.xacro"/>
 	</xacro:unless>
 	<!-- <xacro:stairs stairs="15" xpos="0" ypos="0" zpos="0" /> -->
@@ -51,5 +47,5 @@
 			<origin rpy="0 0 0" xyz="0 0 0"/>
 			<geometry>
-				<mesh filename="file://$(find arcdog_description)/meshes/trunk.dae" scale="1 1 1"/>
+				<mesh filename="file://$(find arcdog_adjustable_leg_description)/meshes/trunk.stl" scale="1 1 1"/>
 			</geometry>
 			<!-- <material name="orange"/> -->
@@ -59,22 +55,4 @@
 			<geometry>
 				<box size="${trunk_length} ${trunk_width} ${trunk_height}"/>
-			</geometry>
-		</collision>
-		<collision>
-			<origin rpy="0 0 0" xyz="0 0 0"/>
-			<geometry>
-				<box size="0.1881 0.04675 0.057"/>
-			</geometry>
-		</collision>
-		<collision>
-			<origin rpy="0 0 0" xyz="0.285 0 0.01"/>
-			<geometry>
-				<cylinder length="0.05" radius="0.045"/>
-			</geometry>
-		</collision>
-		<collision>
-			<origin rpy="0 0 0" xyz="0.293 0 -0.06"/>
-			<geometry>
-				<box size="0.047 0.047 0.047"/>
 			</geometry>
 		</collision>
@@ -139,15 +117,7 @@
 	</link>
 -->
-    <xacro:leg prefix="FR" mirror="-1" mirror_dae="False" front_hind="1" front_hind_dae="True" simulator="${simulator}" robot_type="${robot_type}">
-        <origin rpy="0 0 0" xyz="${leg_offset_x} ${-leg_offset_y} 0"/>
-    </xacro:leg>
-    <xacro:leg prefix="FL" mirror="1" mirror_dae="True" front_hind="1" front_hind_dae="True" simulator="${simulator}" robot_type="${robot_type}">
-        <origin rpy="0 0 0" xyz="${leg_offset_x} ${leg_offset_y} 0"/>
-    </xacro:leg>
-    <xacro:leg prefix="RR" mirror="-1" mirror_dae="False" front_hind="-1" front_hind_dae="False" simulator="${simulator}" robot_type="${robot_type}">
-        <origin rpy="0 0 0" xyz="${-leg_offset_x} ${-leg_offset_y} 0"/>
-    </xacro:leg>
-    <xacro:leg prefix="RL" mirror="1" mirror_dae="True" front_hind="-1" front_hind_dae="False" simulator="${simulator}" robot_type="${robot_type}">
-        <origin rpy="0 0 0" xyz="${-leg_offset_x} ${leg_offset_y} 0"/>
-    </xacro:leg>
+	<xacro:leg name="FR" mirror="-1" mirror_dae="False" front_hind="1" front_hind_dae="True"/>
+	<xacro:leg name="FL" mirror="1" mirror_dae="True" front_hind="1" front_hind_dae="True"/>
+	<xacro:leg name="RR" mirror="-1" mirror_dae="False" front_hind="-1" front_hind_dae="False"/>
+	<xacro:leg name="RL" mirror="1" mirror_dae="True" front_hind="-1" front_hind_dae="False"/>
 </robot>
