Commit message: update arcdog_adjustable leg xml xacro and urdf model

File: robot_description/arcdog_adjustable_leg_description/xacro/robot.xacro (robot description, xacro)
@@ -4,8 +4,4 @@
 	<xacro:arg name="GAZEBO" default="false"/>
 	<xacro:arg name="CLASSIC" default="false"/>
-    <xacro:arg name="robot_type" default="arcdog_adjustable_leg"/>
-    <xacro:property name="robot_type" value="$(arg robot_type)"/>
-	<xacro:arg name="simulator" default="test"/>
-    <xacro:property name="simulator" value="$(arg simulator)"/>
 	<xacro:include filename="$(find arcdog_adjustable_leg_description)/xacro/const.xacro"/>
 	<xacro:include filename="$(find arcdog_adjustable_leg_description)/xacro/materials.xacro"/>
@@ -51,5 +47,5 @@
 			<origin rpy="0 0 0" xyz="0 0 0"/>
 			<geometry>
-				<mesh filename="file://$(find arcdog_adjustable_leg_description)/assets/trunk.stl" scale="1 1 1"/>
+				<mesh filename="file://$(find arcdog_adjustable_leg_description)/meshes/trunk1.dae" scale="1 1 1"/>
 			</geometry>
 			<!-- <material name="orange"/> -->
@@ -59,22 +55,4 @@
 			<geometry>
 				<box size="${trunk_length} ${trunk_width} ${trunk_height}"/>
-			</geometry>
-		</collision>
-		<collision>
-			<origin rpy="0 0 0" xyz="0 0 0"/>
-			<geometry>
-				<box size="0.1881 0.04675 0.057"/>
-			</geometry>
-		</collision>
-		<collision>
-			<origin rpy="0 0 0" xyz="0.285 0 0.01"/>
-			<geometry>
-				<cylinder length="0.05" radius="0.045"/>
-			</geometry>
-		</collision>
-		<collision>
-			<origin rpy="0 0 0" xyz="0.293 0 -0.06"/>
-			<geometry>
-				<box size="0.047 0.047 0.047"/>
 			</geometry>
 		</collision>
@@ -139,15 +117,7 @@
 	</link>
 -->
-    <xacro:leg prefix="FR" mirror="-1" mirror_dae="False" front_hind="1" front_hind_dae="True" simulator="${simulator}" robot_type="${robot_type}">
-        <origin rpy="0 0 0" xyz="${leg_offset_x} ${-leg_offset_y} 0"/>
-    </xacro:leg>
-    <xacro:leg prefix="FL" mirror="1" mirror_dae="True" front_hind="1" front_hind_dae="True" simulator="${simulator}" robot_type="${robot_type}">
-        <origin rpy="0 0 0" xyz="${leg_offset_x} ${leg_offset_y} 0"/>
-    </xacro:leg>
-    <xacro:leg prefix="RR" mirror="-1" mirror_dae="False" front_hind="-1" front_hind_dae="False" simulator="${simulator}" robot_type="${robot_type}">
-        <origin rpy="0 0 0" xyz="${-leg_offset_x} ${-leg_offset_y} 0"/>
-    </xacro:leg>
-    <xacro:leg prefix="RL" mirror="1" mirror_dae="True" front_hind="-1" front_hind_dae="False" simulator="${simulator}" robot_type="${robot_type}">
-        <origin rpy="0 0 0" xyz="${-leg_offset_x} ${leg_offset_y} 0"/>
-    </xacro:leg>
+	<xacro:leg name="FR" mirror="-1" mirror_dae="False" front_hind="1" front_hind_dae="True"/>
+	<xacro:leg name="FL" mirror="1" mirror_dae="True" front_hind="1" front_hind_dae="True"/>
+	<xacro:leg name="RR" mirror="-1" mirror_dae="False" front_hind="-1" front_hind_dae="False"/>
+	<xacro:leg name="RL" mirror="1" mirror_dae="True" front_hind="-1" front_hind_dae="False"/>
 </robot>

File: robot_description/arcdog_adjustable_leg_description/xacro/ros2_control_real_robot.xacro (robot description, xacro)
@@ -3,5 +3,6 @@
 	<ros2_control name="ArcdogSystem" type="system">
 		<hardware>
-			<plugin>hardware_arcdog/HardwareArcdog</plugin>
+			<plugin>hardware_arcdog_adjustable_leg/HardwareArcdog_adjustable_leg</plugin>
+			<!-- <plugin>hardware_arcdog/HardwareArcdog</plugin> -->
 		</hardware>
 		<joint name="FR_hip_joint">
@@ -26,4 +27,14 @@
 		</joint>
 		<joint name="FR_calf_joint">
+			<command_interface name="position"/>
+			<command_interface name="velocity"/>
+			<command_interface name="effort"/>
+			<command_interface name="kp"/>
+			<command_interface name="kd"/>
+			<state_interface name="position"/>
+			<state_interface name="velocity"/>
+			<state_interface name="effort"/>
+		</joint>
+		<joint name="FR_box_joint">
 			<command_interface name="position"/>
 			<command_interface name="velocity"/>
@@ -65,4 +76,14 @@
 			<state_interface name="effort"/>
 		</joint>
+		<joint name="FL_box_joint">
+			<command_interface name="position"/>
+			<command_interface name="velocity"/>
+			<command_interface name="effort"/>
+			<command_interface name="kp"/>
+			<command_interface name="kd"/>
+			<state_interface name="position"/>
+			<state_interface name="velocity"/>
+			<state_interface name="effort"/>
+		</joint>
 		<joint name="RR_hip_joint">
 			<command_interface name="position"/>
@@ -86,4 +107,14 @@
 		</joint>
 		<joint name="RR_calf_joint">
+			<command_interface name="position"/>
+			<command_interface name="velocity"/>
+			<command_interface name="effort"/>
+			<command_interface name="kp"/>
+			<command_interface name="kd"/>
+			<state_interface name="position"/>
+			<state_interface name="velocity"/>
+			<state_interface name="effort"/>
+		</joint>
+		<joint name="RR_box_joint">
 			<command_interface name="position"/>
 			<command_interface name="velocity"/>
@@ -125,4 +156,14 @@
 			<state_interface name="effort"/>
 		</joint>
+		<joint name="RL_box_joint">
+			<command_interface name="position"/>
+			<command_interface name="velocity"/>
+			<command_interface name="effort"/>
+			<command_interface name="kp"/>
+			<command_interface name="kd"/>
+			<state_interface name="position"/>
+			<state_interface name="velocity"/>
+			<state_interface name="effort"/>
+		</joint>
 		<sensor name="imu_sensor">
 			<state_interface name="orientation.w"/>

Commit message: modify leg.xacro and urdf

File: robot_description/arcdog_adjustable_leg_description/urdf/arcdog_adjustable_leg_test.urdf (robot description, URDF)
Before this commit: robot arcdog_adjustable_leg, 23 links, 22 joints
Joints:
- joint FL_box_joint: limit lower=0 upper=-0.193 effort=50 velocity=50 -> lower=0 upper=0.193 effort=50 velocity=50
- joint FR_box_joint: limit lower=0 upper=-0.193 effort=50 velocity=50 -> lower=0 upper=0.193 effort=50 velocity=50
- joint RL_box_joint: limit lower=0 upper=-0.193 effort=50 velocity=50 -> lower=0 upper=0.193 effort=50 velocity=50
- joint RR_box_joint: limit lower=0 upper=-0.193 effort=50 velocity=50 -> lower=0 upper=0.193 effort=50 velocity=50

File: robot_description/arcdog_adjustable_leg_description/xacro/leg.xacro (robot description, xacro)
@@ -162,5 +162,5 @@
             <axis xyz="0 0 1"/> <!-- 定义滑动轴 -->
             <dynamics damping="${damping}" friction="${friction}"/>
-            <limit effort="${box_effort_max}" velocity="${box_velocity_max}" lower="0" upper="${-calf_length}"/> <!-- 定义限制条件 -->
+            <limit effort="${box_effort_max}" velocity="${box_velocity_max}" lower="0" upper="${calf_length}"/> <!-- 定义限制条件 -->
         </joint>
         <joint name="${name}_foot_fixed" type="fixed">
